File: Board Dev/Gen2/Power_Distribution/_autosave-Power_Distribution.kicad_sch (KiCad schematic)
At the start: 27 parts, among them IC1 ACS713ELCTR-30A-T, IC2 ACS713ELCTR-30A-T, IC3 ACS713ELCTR-30A-T, IC4 ACS713ELCTR-30A-T, IC5 ACS713ELCTR-30A-T, IC6 ACS713ELCTR-30A-T, IC7 ACS713ELCTR-30A-T, IC8 ACS713ELCTR-30A-T, J1 8TERM_VERT_1719370, J2 8TERM_VERT_1719370, J3 Conn_01x02_Socket

Commit message: draft of connecting board with current sensors
I'm still waiting to get an email back for the footprint of the connector pins but i have a good one saved.
Parts:
- C_byp1, C_byp2, C_byp3, C_byp4, C_byp5, C_byp6, C_byp7, C_byp8: footprint (none) -> Capacitor_SMD:C_0805_2012Metric_Pad1.18x1.45mm_HandSolder
- C_filter1, C_filter2, C_filter3, C_filter4, C_filter5, C_filter6, C_filter7, C_filter8: footprint 0802 cap:0802 Cap -> Capacitor_SMD:C_0805_2012Metric_Pad1.18x1.45mm_HandSolder
Changed lines of the file:
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@@
 			)
 		)
-		(property "Footprint" ""
+		(property "Footprint" "Capacitor_SMD:C_0805_2012Metric_Pad1.18x1.45mm_HandSolder"
 			(at 327.2007 191.6377 0)
 			(effects
@@
 			)
 		)
-		(property "Footprint" "0802 cap:0802 Cap"
+		(property "Footprint" "Capacitor_SMD:C_0805_2012Metric_Pad1.18x1.45mm_HandSolder"
 			(at 387.065 195.8556 0)
 			(effects
@@
 			)
 		)
-		(property "Footprint" "0802 cap:0802 Cap"
+		(property "Footprint" "Capacitor_SMD:C_0805_2012Metric_Pad1.18x1.45mm_HandSolder"
 			(at 386.1763 165.5607 0)
 			(effects
@@
 			)
 		)
-		(property "Footprint" ""
+		(property "Footprint" "Capacitor_SMD:C_0805_2012Metric_Pad1.18x1.45mm_HandSolder"
 			(at 401.9285 191.3965 0)
 			(effects
@@
 			)
 		)
-		(property "Footprint" ""
+		(property "Footprint" "Capacitor_SMD:C_0805_2012Metric_Pad1.18x1.45mm_HandSolder"
 			(at 183.8147 191.9041 0)
 			(effects
@@
 			)
 		)
-		(property "Footprint" "0802 cap:0802 Cap"
+		(property "Footprint" "Capacitor_SMD:C_0805_2012Metric_Pad1.18x1.45mm_HandSolder"
 			(at 311.2517 163.6342 0)
 			(effects
@@
 			)
 		)
-		(property "Footprint" "0802 cap:0802 Cap"
+		(property "Footprint" "Capacitor_SMD:C_0805_2012Metric_Pad1.18x1.45mm_HandSolder"
 			(at 238.4999 163.1161 0)
 			(effects
@@
 			)
 		)
-		(property "Footprint" ""
+		(property "Footprint" "Capacitor_SMD:C_0805_2012Metric_Pad1.18x1.45mm_HandSolder"
 			(at 182.7292 159.4415 0)
 			(effects
@@
 			)
 		)
-		(property "Footprint" ""
+		(property "Footprint" "Capacitor_SMD:C_0805_2012Metric_Pad1.18x1.45mm_HandSolder"
 			(at 326.1152 159.1751 0)
 			(effects
@@
 			)
 		)
-		(property "Footprint" ""
+		(property "Footprint" "Capacitor_SMD:C_0805_2012Metric_Pad1.18x1.45mm_HandSolder"
 			(at 253.3634 158.657 0)
 			(effects
@@
 			)
 		)
-		(property "Footprint" "0802 cap:0802 Cap"
+		(property "Footprint" "Capacitor_SMD:C_0805_2012Metric_Pad1.18x1.45mm_HandSolder"
 			(at 239.5854 195.5787 0)
 			(effects
@@
 			)
 		)
-		(property "Footprint" ""
+		(property "Footprint" "Capacitor_SMD:C_0805_2012Metric_Pad1.18x1.45mm_HandSolder"
 			(at 254.4489 191.1196 0)
 			(effects
@@
 			)
 		)
-		(property "Footprint" "0802 cap:0802 Cap"
+		(property "Footprint" "Capacitor_SMD:C_0805_2012Metric_Pad1.18x1.45mm_HandSolder"
 			(at 168.9512 196.3632 0)
 			(effects
@@
 			)
 		)
-		(property "Footprint" ""
+		(property "Footprint" "Capacitor_SMD:C_0805_2012Metric_Pad1.18x1.45mm_HandSolder"
 			(at 401.0398 161.1016 0)
 			(effects
@@
 			)
 		)
-		(property "Footprint" "0802 cap:0802 Cap"
+		(property "Footprint" "Capacitor_SMD:C_0805_2012Metric_Pad1.18x1.45mm_HandSolder"
 			(at 167.8657 163.9006 0)
 			(effects
@@
 			)
 		)
-		(property "Footprint" "0802 cap:0802 Cap"
+		(property "Footprint" "Capacitor_SMD:C_0805_2012Metric_Pad1.18x1.45mm_HandSolder"
 			(at 312.3372 196.0968 0)
 			(effects
