File: Board Dev/Gen2/Power_Distribution/Power_Distribution.kicad_pcb (KiCad board)
At the start: 2 copper layers, 156.7 x 60.7 mm, 37 parts, among them IC1 ACS713ELCTR-30A-T, IC2 ACS713ELCTR-30A-T, IC3 ACS713ELCTR-30A-T, IC4 ACS713ELCTR-30A-T, IC5 ACS713ELCTR-30A-T, IC6 ACS713ELCTR-30A-T, IC7 ACS713ELCTR-30A-T, IC8 ACS713ELCTR-30A-T, J1 8TERM_VERT_1719370, J2 8TERM_VERT_1719370, J3 Conn_01x04_Socket, J4 1986660-2, J5 Conn_01x04_Socket

Commit message: pcb to fit dimensions
Parts:
- removed the ? at (150.1, 128.8) (x2)
- removed the ? at (298.6, 128.8)
- removed the REF** at (298.6, 128.8)
- removed the REF** at (150.1, 128.8)
- removed the REF** at (298.6, 93.8)
- removed the REF** at (150.1, 93.8)
- added ? (x2): , , F.Cu at (67.0, 110.2)
- added ?: , , F.Cu at (196.5, 108.4)
- added REF**: MountingHole_2.2mm_M2_Pad_TopBottom, MountingHole:MountingHole_2.2mm_M2_Pad_TopBottom, F.Cu at (66.5, 72.7)
- added REF**: MountingHole_2.2mm_M2_Pad_TopBottom, MountingHole:MountingHole_2.2mm_M2_Pad_TopBottom, F.Cu at (67.0, 110.2)
- added REF**: MountingHole_2.2mm_M2_Pad_TopBottom, MountingHole:MountingHole_2.2mm_M2_Pad_TopBottom, F.Cu at (196.5, 108.4)
- added REF**: MountingHole_2.2mm_M2_Pad_TopBottom, MountingHole:MountingHole_2.2mm_M2_Pad_TopBottom, F.Cu at (196.4, 72.7)
- moved C_byp5 156.5 mm to (68.8, 102.0), turned to -90 degrees
- moved C_byp6 142.0 mm to (83.5, 99.2), turned to -90 degrees
- moved C_byp7 125.3 mm to (100.3, 102.5), turned to -90 degrees
- moved J5 113.9 mm to (186.5, 115.4)
- moved C_byp8 111.6 mm to (114.3, 102.0), turned to -90 degrees
- moved C_filter5 104.1 mm to (138.2, 103.2)
- moved C_filter6 104.1 mm to (153.2, 103.2)
- moved IC5 104.1 mm to (138.2, 95.2)
- moved IC6 104.1 mm to (153.2, 95.2)
- moved REF** 104.1 mm to (196.9, 100.0)
- moved C_filter7 104.1 mm to (168.2, 103.2)
- moved C_filter8 104.1 mm to (183.2, 103.2)
- moved IC7 104.1 mm to (168.2, 95.2)
- moved IC8 104.1 mm to (183.2, 95.2)
- moved J4 95.5 mm to (125.1, 111.2)
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Routing:
- net PWR8: track 23.7 -> 75.2 mm
- net PWR1: track 23.1 -> 67.1 mm
- net PWR5: track 22.9 -> 56.6 mm
- net PWR4: track 24.1 -> 54.0 mm
- net PWR2: track 23.5 -> 47.4 mm
- net +BATT: track 299.0 -> 318.5 mm
- net VIout5: track 84.5 -> 71.5 mm
- net PWR7: track 23.5 -> 36.3 mm
- net VIout7: track 51.7 -> 41.1 mm
- net VIout6: track 66.6 -> 56.1 mm
- net GND: track 383.5 -> 373.1 mm, vias 9 -> 17
- net VIout8: track 36.9 -> 26.7 mm
- net 5V: track 271.4 -> 281.7 mm, vias 9 -> 21
- net PWR3: track 24.3 -> 19.7 mm
- net PWR6: track 24.6 -> 20.2 mm
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Other:
- board size 156.7 x 60.7 mm -> 135.6 x 59 mm
- board text added: "Stanford RoboSub 2024-2025 Stay Wavyyy"
- board text removed: "Stanford RoboSub 2025 Stay Wavyyy"
