File: Board Dev/Gen2/Power_Distribution/Power_Distribution.kicad_pcb (KiCad board)
At the start: 2 copper layers, 155 x 59 mm, 26 parts, among them IC1 ACS713ELCTR-30A-T, IC2 ACS713ELCTR-30A-T, IC3 ACS713ELCTR-30A-T, IC4 ACS713ELCTR-30A-T, IC5 ACS713ELCTR-30A-T, IC6 ACS713ELCTR-30A-T, IC7 ACS713ELCTR-30A-T, IC8 ACS713ELCTR-30A-T, J1 8TERM_VERT_1719370, J2 8TERM_VERT_1719370

Commit message: Final Power Dist Board
Parts:
- removed the REF** at (150.1, 120.4)
- added C_byp1: 0.1 µF, Capacitor_SMD:C_0805_2012Metric_Pad1.18x1.45mm_HandSolder, F.Cu at (225.3, 92.4)
- added C_byp2: 0.1 µF, Capacitor_SMD:C_0805_2012Metric_Pad1.18x1.45mm_HandSolder, F.Cu at (225.3, 95.4)
- added C_byp3: 0.1 µF, Capacitor_SMD:C_0805_2012Metric_Pad1.18x1.45mm_HandSolder, F.Cu at (225.3, 98.4)
- added C_byp4: 0.1 µF, Capacitor_SMD:C_0805_2012Metric_Pad1.18x1.45mm_HandSolder, F.Cu at (225.3, 101.4)
- added C_byp5: 0.1 µF, Capacitor_SMD:C_0805_2012Metric_Pad1.18x1.45mm_HandSolder, F.Cu at (225.3, 104.4)
- added C_byp6: 0.1 µF, Capacitor_SMD:C_0805_2012Metric_Pad1.18x1.45mm_HandSolder, F.Cu at (225.3, 107.4)
- added C_byp7: 0.1 µF, Capacitor_SMD:C_0805_2012Metric_Pad1.18x1.45mm_HandSolder, F.Cu at (225.3, 110.5)
- added C_byp8: 0.1 µF, Capacitor_SMD:C_0805_2012Metric_Pad1.18x1.45mm_HandSolder, F.Cu at (225.3, 113.5)
- added J3: Conn_01x04_Socket, Connector_PinHeader_2.54mm:PinHeader_1x04_P2.54mm_Vertical, F.Cu at (150.3, 143.8)
- added J4: 1986660-2, HighPowerRoboConnector:CONN2_1986660-2_TEC, F.Cu at (218.4, 131.7)
- added J5: Conn_01x04_Socket, Connector_PinHeader_2.54mm:PinHeader_1x04_P2.54mm_Vertical, F.Cu at (298.6, 135.8)
- added REF**: PinSocket_1x02_P2.54mm_Vertical, Connector_PinSocket_2.54mm:PinSocket_1x02_P2.54mm_Vertical, F.Cu at (298.9, 120.4)
- C_filter1, C_filter2, C_filter3, C_filter4, C_filter5, C_filter6, C_filter7, C_filter8: footprint 0802 cap:0802 Cap -> Capacitor_SMD:C_0805_2012Metric_Pad1.18x1.45mm_HandSolder
- IC2, IC3, IC4, IC5, IC6, IC7: footprint Imported_Footprints:ACS711ELCTR25ABT -> Imported_Footprints:MyHalleffectSensor
Routing:
- net +BATT: track 4.54 -> 299.0 mm
- net 5V: track 0.00 -> 227.2 mm, vias 0 -> 1
- net VIout5: track 0.00 -> 84.5 mm, vias 0 -> 1
- net VIout4: track 0.00 -> 77.5 mm, vias 0 -> 1
- net VIout6: track 0.00 -> 66.6 mm, vias 0 -> 1
- net GND: track 303.4 -> 367.9 mm, vias 0 -> 1
- net VIout3: track 0.00 -> 60.5 mm, vias 0 -> 1
- net VIout7: track 0.00 -> 51.8 mm, vias 0 -> 1
- net VIout2: track 0.00 -> 41.8 mm, vias 0 -> 1
- net VIout8: track 0.00 -> 37.0 mm, vias 0 -> 1
- net VIout1: track 0.00 -> 32.2 mm
- net PWR5: track 28.4 -> 22.9 mm
- net PWR2: track 21.7 -> 23.5 mm
- net PWR6: track 22.9 -> 24.6 mm
- net Net-(IC8-FILTER): track 12.9 -> 11.3 mm
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
Commit message: Finished and Tested
Routing:
- net 5V: track 227.2 -> 271.4 mm, vias 1 -> 9
- net GND: track 367.9 -> 383.5 mm, vias 1 -> 9
Other:
- board size 155 x 59 mm -> 156.7 x 60.7 mm
- board text added: "Stanford RoboSub 2025 Stay Wavyyy"

Commit message: good spot
Parts:
- moved C_byp5 74.1 mm to (153.4, 122.4), turned to -90 degrees
- moved C_byp1 73.6 mm to (291.9, 123.6), turned to -90 degrees
- moved C_byp2 59.0 mm to (277.2, 123.5), turned to -90 degrees
- moved C_byp6 58.4 mm to (168.1, 119.7), turned to -90 degrees
- moved C_byp3 43.1 mm to (259.8, 124.2), turned to -90 degrees
- moved C_byp7 42.3 mm to (184.9, 122.9), turned to -90 degrees
- moved C_byp4 29.2 mm to (246.4, 121.7), turned to -90 degrees
- moved C_byp8 27.9 mm to (198.9, 122.4), turned to -90 degrees
Routing:
- net +BATT: track 299.0 -> 353.0 mm
- net GND: track 383.5 -> 354.7 mm, vias 9 -> 14
- net 5V: track 271.4 -> 298.4 mm, vias 9 -> 22
- net PWR7: track 23.5 -> 31.0 mm
- net PWR8: track 23.7 -> 31.1 mm
- net VIout5: track 84.5 -> 80.1 mm
- net PWR6: track 24.6 -> 22.9 mm
- net VIout3: track 60.5 -> 59.0 mm
- net PWR3: track 24.3 -> 22.9 mm
- net PWR2: track 23.5 -> 22.3 mm
- net PWR4: track 24.1 -> 22.9 mm
- net VIout4: track 77.5 -> 76.5 mm
- net PWR1: track 23.1 -> 22.3 mm
- net VIout8: track 36.9 -> 36.3 mm
- net VIout7: track 51.7 -> 51.1 mm
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Other:
- board text added: "Stanford RoboSub 2024-2025 Stay Wavyyy"
- board text removed: "Stanford RoboSub 2025 Stay Wavyyy"

Commit message: tweaking board
Parts:
- removed ? (x3): , 
- removed REF** (x4): MountingHole_2.2mm_M2_Pad_TopBottom, MountingHole:MountingHole_2.2mm_M2_Pad_TopBottom
- removed REF**: PinSocket_1x02_P2.54mm_Vertical, Connector_PinSocket_2.54mm:PinSocket_1x02_P2.54mm_Vertical
- added J6: 1098169, Imported_Footprints:PHOENIX_1098169, F.Cu at (210.6, 54.0)
- added J7: 1098169, Imported_Footprints:PHOENIX_1098169, F.Cu at (113.5, 53.8)
- J1, J2: value 8TERM_VERT_1719370 -> 1098169; footprint Imported_Footprints:PHOENIX_1719370 -> Imported_Footprints:PHOENIX_1098169
- J4: footprint HighPowerRoboConnector:CONN2_1986660-2_TEC -> Imported_Footprints:TE_1986660-2
- moved C_byp1 238.3 mm to (69.5, 38.0), turned to 0 degrees
- moved J5 231.4 mm to (88.5, 38.8)
- moved C_byp2 223.5 mm to (69.5, 41.0), turned to 0 degrees
- moved C_filter8 219.9 mm to (79.1, 47.0)
- moved IC7 209.0 mm to (79.1, 31.2), turned to 0 degrees
- moved C_filter7 207.1 mm to (79.1, 44.0)
- moved C_byp3 206.5 mm to (69.5, 44.0), turned to 0 degrees
- moved IC6 202.6 mm to (71.1, 31.2), turned to 0 degrees
- moved IC8 196.6 mm to (91.4, 82.8)
- moved C_filter6 194.6 mm to (79.1, 41.0)
- moved C_byp4 192.0 mm to (69.5, 47.0), turned to 0 degrees
- moved C_filter5 182.5 mm to (79.1, 38.0)
- moved IC5 166.8 mm to (103.1, 20.8), turned to 0 degrees
- moved C_filter4 149.0 mm to (74.3, 53.0)
- moved C_byp8 148.8 mm to (74.3, 41.0), turned to 0 degrees
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Connections:
- C_filter3 pad 1: Net-(IC3-FILTER) -> Net-(IC6-FILTER)
- C_filter4 pad 1: Net-(IC4-FILTER) -> Net-(IC7-FILTER)
- C_filter6 pad 1: Net-(IC6-FILTER) -> Net-(IC3-FILTER)
- C_filter7 pad 1: Net-(IC7-FILTER) -> Net-(IC4-FILTER)
- J1 pad 1: PWR1 -> PWR3
- J1 pad 3: PWR2 -> PWR4
Routing:
- net GND: track 354.7 -> 0.00 mm, vias 14 -> 0
- net +BATT: track 353.0 -> 0.00 mm
- net 5V: track 298.4 -> 0.00 mm, vias 22 -> 0
- net VIout5: track 80.1 -> 0.00 mm, vias 1 -> 0
- net VIout4: track 76.5 -> 0.00 mm, vias 1 -> 0
- net VIout6: track 66.0 -> 0.00 mm, vias 1 -> 0
- net VIout3: track 59.0 -> 0.00 mm, vias 1 -> 0
- net VIout7: track 51.1 -> 0.00 mm, vias 1 -> 0
- net VIout2: track 41.3 -> 0.00 mm, vias 1 -> 0
- net VIout8: track 36.3 -> 0.00 mm, vias 1 -> 0
- net VIout1: track 31.8 -> 0.00 mm
- net PWR8: track 31.1 -> 0.00 mm
- net PWR7: track 31.0 -> 0.00 mm
- net PWR6: track 22.9 -> 0.00 mm
- net PWR5: track 22.9 -> 0.00 mm
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- removed copper zone on B.Cu, net -BATT
Other:
- board size 156.7 x 60.7 mm -> 130 x 60 mm
- board text removed: "Stanford RoboSub 2024-2025 Stay Wavyyy"

Commit message: Rev2 on Power Distribution Complete
Parts:
- removed C_byp1, C_byp2, C_byp3, C_byp4, C_byp5, C_byp6, C_byp7, C_byp8: 0.1 µF, Capacitor_SMD:C_0805_2012Metric_Pad1.18x1.45mm_HandSolder
- removed C_filter1, C_filter2, C_filter3, C_filter4, C_filter5, C_filter6, C_filter7, C_filter8: 100 µF, Capacitor_SMD:C_0805_2012Metric_Pad1.18x1.45mm_HandSolder
- added Cb1: 0.1 µF, Capacitor_SMD:C_0805_2012Metric_Pad1.18x1.45mm_HandSolder, F.Cu at (196.8, 84.6)
- added Cb2: 0.1 µF, Capacitor_SMD:C_0805_2012Metric_Pad1.18x1.45mm_HandSolder, F.Cu at (181.2, 84.4)
- added Cb3: 0.1 µF, Capacitor_SMD:C_0805_2012Metric_Pad1.18x1.45mm_HandSolder, F.Cu at (116.9, 84.4)
- added Cb4: 0.1 µF, Capacitor_SMD:C_0805_2012Metric_Pad1.18x1.45mm_HandSolder, F.Cu at (99.8, 85.0)
- added Cb5: 0.1 µF, Capacitor_SMD:C_0805_2012Metric_Pad1.18x1.45mm_HandSolder, F.Cu at (132.1, 84.4)
- added Cb6: 0.1 µF, Capacitor_SMD:C_0805_2012Metric_Pad1.18x1.45mm_HandSolder, F.Cu at (164.4, 84.5)
- added Cb7: 0.1 µF, Capacitor_SMD:C_0805_2012Metric_Pad1.18x1.45mm_HandSolder, F.Cu at (149.1, 84.4)
- added Cb8: 0.1 µF, Capacitor_SMD:C_0805_2012Metric_Pad1.18x1.45mm_HandSolder, F.Cu at (84.6, 84.4)
- added Cf1: 100 µF, Capacitor_SMD:C_0805_2012Metric_Pad1.18x1.45mm_HandSolder, F.Cu at (196.8, 82.3)
- added Cf2: 100 µF, Capacitor_SMD:C_0805_2012Metric_Pad1.18x1.45mm_HandSolder, F.Cu at (181.2, 82.2)
- added Cf3: 100 µF, Capacitor_SMD:C_0805_2012Metric_Pad1.18x1.45mm_HandSolder, F.Cu at (116.9, 82.1)
- added Cf4: 100 µF, Capacitor_SMD:C_0805_2012Metric_Pad1.18x1.45mm_HandSolder, F.Cu at (99.8, 82.9)
- added Cf5: 100 µF, Capacitor_SMD:C_0805_2012Metric_Pad1.18x1.45mm_HandSolder, F.Cu at (132.1, 82.1)
- added Cf6: 100 µF, Capacitor_SMD:C_0805_2012Metric_Pad1.18x1.45mm_HandSolder, F.Cu at (164.3, 82.1)
- added Cf7: 100 µF, Capacitor_SMD:C_0805_2012Metric_Pad1.18x1.45mm_HandSolder, F.Cu at (149.0, 82.0)
- added Cf8: 100 µF, Capacitor_SMD:C_0805_2012Metric_Pad1.18x1.45mm_HandSolder, F.Cu at (84.6, 82.1)
- added H1: MountingHole, MountingHole:MountingHole_3.2mm_M3, F.Cu at (186.9, 107.4)
- added H2: MountingHole, MountingHole:MountingHole_3.2mm_M3, F.Cu at (171.9, 107.4)
- added H3: MountingHole, MountingHole:MountingHole_3.2mm_M3, F.Cu at (201.9, 107.4)
- added H4: MountingHole, MountingHole:MountingHole_3.2mm_M3, F.Cu at (96.9, 107.4)
- added J8: Conn_01x02, Connector_PinHeader_2.54mm:PinHeader_1x02_P2.54mm_Vertical, F.Cu at (95.2, 97.6)
- added J9: Conn_01x08, Connector_PinHeader_2.54mm:PinHeader_1x08_P2.54mm_Vertical, F.Cu at (105.0, 97.5)
- J3: value Conn_01x04_Socket -> Conn_01x08; footprint Connector_PinHeader_2.54mm:PinHeader_1x04_P2.54mm_Vertical -> Connector_PinHeader_2.54mm:PinHeader_1x08_P2.54mm_Vertical
- J5: value Conn_01x04_Socket -> Conn_01x06; footprint Connector_PinHeader_2.54mm:PinHeader_1x04_P2.54mm_Vertical -> Connector_PinHeader_2.54mm:PinHeader_1x06_P2.54mm_Vertical
- moved IC1 146.3 mm to (203.7, 82.7), turned to 90 degrees
- moved IC2 125.7 mm to (188.6, 82.6), turned to 90 degrees
- moved IC3 104.4 mm to (171.2, 82.6), turned to 90 degrees
- moved IC4 86.9 mm to (156.3, 82.6), turned to 90 degrees
- moved J3 74.5 mm to (105.0, 110.2), turned to 90 degrees
- moved IC6 73.5 mm to (123.8, 82.5), turned to 90 degrees
- moved J5 71.4 mm to (89.6, 110.2), turned to 180 degrees
- moved IC5 71.3 mm to (138.9, 82.5), turned to 90 degrees
- moved IC7 58.1 mm to (106.6, 82.5), turned to 90 degrees
- moved IC8 0.36 mm to (91.4, 82.4)
Connections:
- J3 pad 1: VIout4 -> 5V
- J3 pad 2: VIout3 -> GND
- J3 pad 3: VIout2 -> SCL
- J3 pad 4: VIout1 -> SDA
- J5 pad 1: VIout8 -> SCL
- J5 pad 2: VIout7 -> SDA
- J5 pad 3: VIout6 -> REF
- J5 pad 4: VIout5 -> COM
Routing:
- net GND: track 0.00 -> 284.8 mm, vias 0 -> 11
- net -BATT: track 0.00 -> 270.5 mm
- net +BATT: track 0.00 -> 241.0 mm
- net 5V: track 0.00 -> 207.1 mm, vias 0 -> 11
- net VIout1: track 0.00 -> 89.6 mm, vias 0 -> 3
- net VIout2: track 0.00 -> 77.9 mm, vias 0 -> 3
- net VIout3: track 0.00 -> 63.3 mm, vias 0 -> 3
- net VIout4: track 0.00 -> 55.0 mm, vias 0 -> 1
- net AD1: track 0.00 -> 41.1 mm, vias 0 -> 1
- net AD0: track 0.00 -> 36.9 mm, vias 0 -> 1
- net COM: track 0.00 -> 33.1 mm, vias 0 -> 1
- net VIout5: track 0.00 -> 33.1 mm, vias 0 -> 1
- net REF: track 0.00 -> 29.9 mm, vias 0 -> 1
- net SDA: track 0.00 -> 27.4 mm, vias 0 -> 1
- net VIout8: track 0.00 -> 24.7 mm, vias 0 -> 1
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Other:
- board text added: "+BATT"
- board text added: "-BATT"
- board text added: "1"
- board text added: "2"
- board text added: "3"
- board text added: "4"
- board text added: "5"
- board text added: "5V"
- board text added: "6"
- board text added: "7"
- board text added: "8"
- board text added: "AD0"
- board text added: "AD1"
- board text added: "Analog In"
- board text added: "COM"
- board text added: "GND"
- board text added: "PWR1"
- board text added: "PWR2"
- board text added: "PWR3"
- board text added: "PWR4"
- board text added: "PWR5"
- board text added: "PWR6"
- board text added: "PWR7"
- board text added: "PWR8"
- board text added: "REF"
- board text added: "SCL"
- board text added: "SDA"
- board text added: "Stanford Robosub, Thruster Power {dblquote}The sea, once it casts its spell, holds one in its net of wonder forever.{dblquote} - Jacques Cousteau"
- board text added: "__ |__ __L L_|L L__ ...[+(____________) C_________/"
