File: Board Dev/Gen2/Power_Distribution/Power_Distribution.kicad_sch (KiCad schematic)
At the start: 27 parts, among them IC1 ACS713ELCTR-30A-T, IC2 ACS713ELCTR-30A-T, IC3 ACS713ELCTR-30A-T, IC4 ACS713ELCTR-30A-T, IC5 ACS713ELCTR-30A-T, IC6 ACS713ELCTR-30A-T, IC7 ACS713ELCTR-30A-T, IC8 ACS713ELCTR-30A-T, J1 8TERM_VERT_1719370, J2 8TERM_VERT_1719370, J3 Conn_01x02_Socket

Commit message: Final Power Dist Board
Parts:
- removed J3: Conn_01x02_Socket, symbol Connector:Conn_01x02_Socket
- added J3, J5: Conn_01x04_Socket, Connector_PinHeader_2.54mm:PinHeader_1x04_P2.54mm_Vertical, symbol Connector:Conn_01x04_Socket
- added J4: 1986660-2, CONN2_1986660-2_TEC, symbol HighPowerRoboConnector:1986660-2
- C_byp1, C_byp2, C_byp3, C_byp4, C_byp5, C_byp6, C_byp7, C_byp8: footprint (none) -> Capacitor_SMD:C_0805_2012Metric_Pad1.18x1.45mm_HandSolder
- C_filter1, C_filter2, C_filter3, C_filter4, C_filter5, C_filter6, C_filter7, C_filter8: footprint 0802 cap:0802 Cap -> Capacitor_SMD:C_0805_2012Metric_Pad1.18x1.45mm_HandSolder
- IC2, IC3, IC4, IC5, IC6, IC7: footprint Imported_Footprints:ACS711ELCTR25ABT -> Imported_Footprints:MyHalleffectSensor
Connections:
- net +BATT: now also J4.1A, J4.1B
- net -BATT: now also J4.2A, J4.2B
- net VIout1: now also J3.4 (Pin_4)
- net VIout2: now also J3.3 (Pin_3)
- net VIout3: now also J3.2 (Pin_2)
- net VIout4: now also J3.1 (Pin_1)
- net VIout5: now also J5.4 (Pin_4)
- net VIout6: now also J5.3 (Pin_3)
- net VIout7: now also J5.2 (Pin_2)
- net VIout8: now also J5.1 (Pin_1)
Other:
- note added: "Connectors To ESCs"
- note added: "Hall Effect Sensors"
- note added: "High Power Connector Socket For Bat in and Gnd"
- note added: "One by Four Pin Headers"
- moved on the sheet: J1, J2

Commit message: good spot
Other:
- moved on the sheet: C_byp2, C_filter1, C_filter2, IC1, IC2

Commit message: BOM changes
Parts:
- C_byp1, C_byp2, C_byp3, C_byp4, C_byp5, C_byp6, C_byp7, C_byp8: Supplier 1 (none) -> https://www.digikey.com/en/products/detail/yageo/CC0805KRX7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; Supplier 1 S/N (none) -> 311-1140-1-ND
- C_filter1, C_filter2, C_filter3, C_filter4, C_filter5, C_filter6, C_filter7, C_filter8: Supplier 1 (none) -> https://www.digikey.com/en/products/detail/murata-electroni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; Supplier 1 S/N (none) -> 490-13980-1-ND
- J4: Supplier 1 (none) -> https://www.digikey.com/en/products/detail/te-connectivity-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; Supplier 1 S/N (none) -> A107722-ND
Connections:
- net at C_filter6.1: now also IC3.6 (FILTER); no longer IC6.6 (FILTER)
- net at IC4.6 (FILTER): now also C_filter7.1; no longer C_filter4.1
- net at C_filter3.1: now also IC6.6 (FILTER); no longer IC3.6 (FILTER)
- net at IC7.6 (FILTER): now also C_filter4.1; no longer C_filter7.1

Commit message: tweaking board
Parts:
- removed J1, J2: 8TERM_VERT_1719370, Imported_Footprints:PHOENIX_1719370, symbol Imported_Symbols:8TERM_VERT_1719370
- added J1, J2, J6, J7: 1098169, Imported_Footprints:PHOENIX_1098169, symbol Imported_Symbols:1098169
- J4: footprint CONN2_1986660-2_TEC -> Imported_Footprints:TE_1986660-2
Connections:
- net -BATT: now also J1.2, J1.4, J2.2, J2.4, J6.2, J6.4, J7.2, J7.4
- net PWR1: now also J6.1
- net PWR2: now also J6.3
- net PWR3: now also J1.1
- net PWR4: now also J1.3
- net PWR5: now also J2.1
- net PWR6: now also J2.3
- net PWR7: now also J7.1
- net PWR8: now also J7.3

Commit message: Rev2 on Power Distribution Complete
Parts:
- removed J3, J5: Conn_01x04_Socket, Connector_PinHeader_2.54mm:PinHeader_1x04_P2.54mm_Vertical, symbol Connector:Conn_01x04_Socket
- added J3, J9: Conn_01x08, Connector_PinHeader_2.54mm:PinHeader_1x08_P2.54mm_Vertical, symbol Connector_Generic:Conn_01x08
- added J5: Conn_01x06, Connector_PinHeader_2.54mm:PinHeader_1x06_P2.54mm_Vertical, symbol Connector_Generic:Conn_01x06
- added J8: Conn_01x02, Connector_PinHeader_2.54mm:PinHeader_1x02_P2.54mm_Vertical, symbol Connector_Generic:Conn_01x02
- renumbered C_byp1 to Cb1, C_byp2 to Cb2, C_byp3 to Cb3, C_byp4 to Cb4, C_byp5 to Cb5, C_byp6 to Cb6, C_byp7 to Cb7, C_byp8 to Cb8, C_filter1 to Cf1, C_filter2 to Cf2, C_filter3 to Cf3, C_filter4 to Cf4, C_filter5 to Cf5, C_filter6 to Cf6, C_filter7 to Cf7, C_filter8 to Cf8
Connections:
- net +BATT: now also J4.1_1 (1), J4.1_2 (1); no longer J4.1A, J4.1B
- net -BATT: now also J4.2_1 (2), J4.2_2 (2); no longer J4.2A, J4.2B
- net 5V: now also J3.1 (Pin_1), J8.1 (Pin_1)
- net GND: now also J3.2 (Pin_2), J8.2 (Pin_2)
- net VIout1: now also J9.8 (Pin_8)
- net VIout2: now also J9.7 (Pin_7)
- net VIout3: now also J9.6 (Pin_6)
- net VIout4: now also J9.5 (Pin_5)
- net VIout5: now also J9.4 (Pin_4)
- net VIout6: now also J9.3 (Pin_3)
- net VIout7: now also J9.2 (Pin_2)
- net VIout8: now also J9.1 (Pin_1)
- new net AD0: J3.7 (Pin_7), J5.5 (Pin_5)
- new net AD1: J3.8 (Pin_8), J5.6 (Pin_6)
- new net COM: J3.6 (Pin_6), J5.4 (Pin_4)
- new net REF: J3.5 (Pin_5), J5.3 (Pin_3)
- new net SCL: J3.3 (Pin_3), J5.1 (Pin_1)
- new net SDA: J3.4 (Pin_4), J5.2 (Pin_2)
Other:
- note added: "Adafruit ADS7830 Interconnect"
- note removed: "One by Four Pin Headers"
