File: Board Dev/Gen2/Power_Management/Power_Management.kicad_sch (KiCad schematic)
At the start: 31 parts, among them IC1 MC33063AQDRQ1, J1 Conn_01x02_Pin, J2 Conn_01x02_Pin, J3 Conn_01x02_Pin, K1 G5V-1 DC3, Q1 MCTL160N15Y-TP, Q2 MCTL160N15Y-TP, Q3 MCTL160N15Y-TP, U1 ACS758ECB-200U-PFF-T

Commit message: done with management
Parts:
- removed C1: 0.1u, symbol Device:C
- removed C2: 1.5nF, symbol Device:C
- removed C3: 330mF, symbol Device:C
- removed C4, C5: 100mF, symbol Device:C
- removed C7, C8: 1u (electrolytic), Imported_Footprints:U2-D_NCH, symbol Device:C
- removed CR1: SBRT15U50SP5-13, Imported_Footprints:POWERDI5_DIO, symbol SBRT15U50SP5_13:SBRT15U50SP5-13
- removed D1: 1N5819, Diode_THT:D_DO-41_SOD81_P10.16mm_Horizontal, symbol Diode:1N5819
- removed D2: LED, LED_SMD:LED_0805_2012Metric_Pad1.15x1.40mm_HandSolder, symbol Device:LED
- removed IC1: MC33063AQDRQ1, Imported_Footprints:SOIC127P600X175-8N, symbol Imported_Symbols:MC33063AQDRQ1
- removed J3: Conn_01x02_Pin, symbol Connector:Conn_01x02_Pin
- removed JP1: SolderJumper_2_Open, Jumper:SolderJumper-2_P1.3mm_Open_RoundedPad1.0x1.5mm, symbol Jumper:SolderJumper_2_Open
- removed JP2, JP3: SolderJumper_3_Bridged12, Jumper:SolderJumper-3_P1.3mm_Bridged2Bar12_RoundedPad1.0x1.5mm, symbol Jumper:SolderJumper_3_Bridged12
- removed K1: G5V-1 DC3, Imported_Footprints:RELAY_G5V-1_OMR, symbol Imported_Symbols:G5V-1_DC3
- removed L1: 170mH, symbol Device:L
- removed L2: 1mH, symbol Device:L
- removed Q1, Q2, Q3: MCTL160N15Y-TP, Imported_Footprints:TOLL-8L_MCC, symbol Imported_Symbols:MCTL160N15Y-TP
- removed R1: 18k, symbol Device:R_US
- removed R2: 180k, symbol Device:R_US
- removed R3: 180, symbol Device:R_US
- removed R4: 0.22, symbol Device:R_US
- removed R5: 100k, symbol Device:R_US
- removed R6: 600k, symbol Device:R_US
- removed U1: ACS758ECB-200U-PFF-T, PFF_ACS758ECB-200U-PFF-T_ALM, symbol Imported_Symbols:ACS758ECB-200U-PFF-T
- added H1, H3, H4: MountingHole, MountingHole:MountingHole_3.2mm_M3, symbol Mechanical:MountingHole
- added J10, J6: Conn_01x02_Pin, Connector_PinHeader_2.54mm:PinHeader_1x02_P2.54mm_Vertical, symbol Connector:Conn_01x02_Pin
- added J9: Conn_01x03_Pin, Connector_PinHeader_2.54mm:PinHeader_1x03_P2.54mm_Vertical, symbol Connector:Conn_01x03_Pin
- C6: footprint (none) -> Capacitor_SMD:C_0805_2012Metric_Pad1.18x1.45mm_HandSolder; MFR (none) -> Samsung Electro-Mechanics; MFR S/N (none) -> CL21A106KOQNNNE; Supplier 1 (none) -> https://www.digikey.com/en/products/detail/samsung-electro-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; Supplier 1 S/N (none) -> 1276-1096-1-ND
- J1, J2: footprint (none) -> Connector_PinHeader_2.54mm:PinHeader_1x02_P2.54mm_Vertical
Connections:
- net GND: now also J10.2 (Pin_2), J6.2 (Pin_2), J9.3 (Pin_3); no longer J1.2 (Pin_2)
- net ISENSE_ANALOG renamed OCP_UVP_detect/ISENSE_ANALOG
- new net +3.3V: J6.1 (Pin_1)
- new net FET_control_logic/Kill_Switch: J10.1 (Pin_1)
- new net OCP_UVP_detect/BATT_SAMPLE: J1.2 (Pin_2)
- new net OCP_UVP_detect/LE_Teensy: J9.1 (Pin_1)
- new net OCP_UVP_detect/OE_Teensy: J9.2 (Pin_2)
Other:
- added sheet Battery_input (Battery_interfaces.kicad_sch)
- added sheet FET_control_logic (AND_GATES.kicad_sch)
- added sheet FETs (FETs.kicad_sch)
- added sheet OCP_UVP_detect (OCP_UVP_detect.kicad_sch)
- added sheet Thruster_output (Thruster_output.kicad_sch)
- added sheet V_I_sample (V_I_sample.kicad_sch)
- added sheet buck_boost (buck_boost.kicad_sch)
- note removed: "10 mV/A at 25C 9.88 mV/A above 25C"
- note removed: "160A at 25C, 100A at 100C"
- note removed: "25V Buck-Boost (Gate Driver)"
- note removed: "Able to swap between the two"
- note removed: "Flyback diode - 50V/15A w/ 290A surge eliminates reverse voltage from inductive loads (*place close to logic*)"
- note removed: "Hall Effect Current Sensor"
- note removed: "Input decoupling capacitors must be located as close as possible to the MC33063-Q1. In addition, the voltage set-point resistor divider components must also be kept close to the IC to eliminate any noise pick-up into the feedback loop"
- note removed: "Make sure to put IP+ and IP- contacts as close to the power trace as possible"
- note removed: "NC --> system is off NO --> need to drive power to turn on motors"
- note removed: "Need Vdiv at least = ~0.19 and on the order of kohm Let R2 = 100k, R1 = 600k, Vdiv = 0.142 Meaning that V_batt,max = 2.38V and V_batt,min = 1.8176V P = V^2 / R, with R_eff = 700k = 403uW"
- note removed: "POWER FETS"
- note removed: "Relay FET Driver (3.3V to 24V isolated interface)"
- note removed: "Teensy 4.1 Analog Pin Range is 0-3.3V -- 10 bit ADC, 1023 levels"
- note removed: "Vgs = +/- 25V"
- note removed: "Voltage reference (1.25V) used to set the output voltage: -->V_out = 1.25(R2/R1 + 1), choose R2 = 180k and R1 = 18k to get 23.75V Current limit peak current set by Ipk = 330mV/Rsense, with Rsense min at 0.2 Ohm -->(1.5A at 0.22 Ohm)"
- note removed: "Vth = 3V"
- note removed: "optional filter"
- note removed: "slap a heat sink on it"
- note removed: "slap heat sinks on them"
- moved on the sheet: C6, J2
