File: Board Dev/Gen2/Power_Management/buck_boost.kicad_sch (KiCad schematic)
At the start: 13 parts, among them J5 Conn_01x02_Pin, K2 G5V-1 DC3, U6 LTC1255CS8-PBF

Commit message: BOM changes
Parts:
- TH1, TH2: Supplier 1 (none) -> https://www.digikey.com/en/products/detail/yageo/RC0805FR-0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; Supplier 1 S/N (none) -> 311-150CRCT-ND
Changed lines of the file:
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@@
 			)
 		)
-		(property "Supplier 1" ""
+		(property "Supplier 1" "https://www.digikey.com/en/products/detail/yageo/RC0805FR-07150RL/727613"
 			(at 94.996 41.91 0)
 			(effects
@@
 			)
 		)
-		(property "Supplier 1 S/N" ""
+		(property "Supplier 1 S/N" "311-150CRCT-ND"
 			(at 94.996 41.91 0)
 			(effects
@@
 			)
 		)
-		(property "Supplier 1" ""
+		(property "Supplier 1" "https://www.digikey.com/en/products/detail/yageo/RC0805FR-07150RL/727613"
 			(at 202.692 41.91 0)
 			(effects
@@
 			)
 		)
-		(property "Supplier 1 S/N" ""
+		(property "Supplier 1 S/N" "311-150CRCT-ND"
 			(at 202.692 41.91 0)
 			(effects
