File: Gen2/MLU_Breakout/MLU_Breakout.kicad_pcb (KiCad board)
At the start: 2 copper layers, 63 x 71.6 mm, 7 parts, among them J1 Conn_02x24_Odd_Even, J10 Conn_02x09_Odd_Even, J25 PixHawk PM02, U4 Teensy4.1

Commit message: MLU progress
Parts:
- added C1: 135p, Capacitor_SMD:C_0603_1608Metric_Pad1.08x0.95mm_HandSolder, F.Cu at (85.3, 108.9)
- added C2: 135p, Capacitor_SMD:C_0603_1608Metric_Pad1.08x0.95mm_HandSolder, F.Cu at (85.3, 111.4)
- added C3: 10uF, Capacitor_SMD:C_0805_2012Metric_Pad1.18x1.45mm_HandSolder, F.Cu at (85.5, 103.2)
- added C4: 10uF, Capacitor_SMD:C_0805_2012Metric_Pad1.18x1.45mm_HandSolder, F.Cu at (85.5, 106.2)
- added H2: MountingHole, MountingHole:MountingHole_3.2mm_M3, F.Cu at (87.2, 127.1)
- added J2: Conn_01x03_Pin, Connector_PinHeader_2.54mm:PinHeader_1x03_P2.54mm_Vertical, F.Cu at (81.0, 133.5)
- added J26: 3.3V Power, Connector_PinSocket_2.54mm:PinSocket_2x08_P2.54mm_Vertical, F.Cu at (78.8, 81.6)
- added J27: 5V Power, Connector_PinSocket_2.54mm:PinSocket_2x08_P2.54mm_Vertical, F.Cu at (85.9, 81.6)
- added J3: PixHawk PM02, Connector_PinSocket_2.54mm:PinSocket_1x06_P2.54mm_Vertical, F.Cu at (81.0, 116.2)
- added J4: BUS1, Connector_PinSocket_2.54mm:PinSocket_1x04_P2.54mm_Vertical, F.Cu at (76.2, 104.0)
- added J5: BUS2, Connector_PinSocket_2.54mm:PinSocket_1x04_P2.54mm_Vertical, F.Cu at (80.8, 104.0)
- added J7: Conn_01x24_Pin, Connector_PinHeader_2.54mm:PinHeader_1x24_P2.54mm_Horizontal, F.Cu at (62.9, 81.6)
- added J8: UART, Connector_PinSocket_2.54mm:PinSocket_1x02_P2.54mm_Vertical, F.Cu at (76.2, 136.9)
- added J9: Conn_01x09_Pin, Connector_PinHeader_1.00mm:PinHeader_1x09_P1.00mm_Vertical, F.Cu at (85.0, 132.7)
- added JP3: Jumper_2_Open, Jumper:SolderJumper-2_P1.3mm_Open_RoundedPad1.0x1.5mm, F.Cu at (101.8, 100.8)
- added R1: 10k, Resistor_SMD:R_0805_2012Metric_Pad1.20x1.40mm_HandSolder, F.Cu at (76.3, 115.4)
- added R2: 10k, Resistor_SMD:R_0805_2012Metric_Pad1.20x1.40mm_HandSolder, F.Cu at (76.3, 118.3)
- added R3: 10k, Resistor_SMD:R_0805_2012Metric_Pad1.20x1.40mm_HandSolder, F.Cu at (76.3, 121.3)
- added R4: 10k, Resistor_SMD:R_0805_2012Metric_Pad1.20x1.40mm_HandSolder, F.Cu at (76.3, 124.2)
- added R5: 10k, Resistor_SMD:R_0805_2012Metric_Pad1.20x1.40mm_HandSolder, F.Cu at (76.3, 127.2)
- added R6: 10k, Resistor_SMD:R_0805_2012Metric_Pad1.20x1.40mm_HandSolder, F.Cu at (76.3, 130.1)
- added R7: 10k, Resistor_SMD:R_0805_2012Metric_Pad1.20x1.40mm_HandSolder, F.Cu at (76.3, 133.1)
- added RN1: 10kΩ, Resistor_SMD:R_Array_Convex_4x0612, F.Cu at (88.5, 137.7)
- added U1: MCP23008-xP, Package_DIP:DIP-18_W7.62mm, F.Cu at (185.8, 68.6)
- added U2: MCP9808_MSOP, Package_SO:MSOP-8_3x3mm_P0.65mm, F.Cu at (87.0, 116.2)
- added U3: BME280, Imported Footprints:BME280, F.Cu at (88.8, 133.3)
- added U5: MCP9808_MSOP, Package_SO:MSOP-8_3x3mm_P0.65mm, F.Cu at (87.0, 120.8)
- J10: value Conn_02x09_Odd_Even -> Conn_02x08_Odd_Even; footprint Connector_PinHeader_2.54mm:PinHeader_2x09_P2.54mm_Vertical -> Connector_PinSocket_2.54mm:PinSocket_2x08_P2.54mm_Vertical
- moved H1 1.56 mm to (184.2, 112.6)
- moved H3 1.56 mm to (154.2, 112.6)
- moved H4 1.56 mm to (154.2, 67.6)
Connections:
- net SPI_CS2 renamed D10
- J1 pad 10: unconnected-(J1-Pin_10-Pad10) -> A3
- J1 pad 12: PWM1 -> GND
- J1 pad 13: D4 -> Dswitch2
- J1 pad 14: GND -> A4
- J1 pad 16: unconnected-(J1-Pin_16-Pad16) -> GND
- J1 pad 18: PWM2 -> +3.3V
- J1 pad 2: GND -> A1
- J1 pad 22: unconnected-(J1-Pin_22-Pad22) -> I2C1_SCL
- J1 pad 24: PWM3 -> I2C1_SDA
- J1 pad 25: unconnected-(J1-Pin_25-Pad25) -> UART_TX3
- J1 pad 26: GND -> unconnected-(J1-Pin_26-Pad26)
- J1 pad 27: unconnected-(J1-Pin_27-Pad27) -> UART_RX3
- J1 pad 29: unconnected-(J1-Pin_29-Pad29) -> GND
- J1 pad 3: D1 -> Dled1
- J1 pad 30: PWM4 -> unconnected-(J1-Pin_30-Pad30)
- J1 pad 31: unconnected-(J1-Pin_31-Pad31) -> UART_TX2
- J1 pad 32: GND -> unconnected-(J1-Pin_32-Pad32)
- J1 pad 33: unconnected-(J1-Pin_33-Pad33) -> UART_RX2
- J1 pad 35: unconnected-(J1-Pin_35-Pad35) -> +3.3V
- J1 pad 36: PWM5 -> unconnected-(J1-Pin_36-Pad36)
- J1 pad 37: unconnected-(J1-Pin_37-Pad37) -> GND
- J1 pad 38: GND -> unconnected-(J1-Pin_38-Pad38)
- J1 pad 4: unconnected-(J1-Pin_4-Pad4) -> GND
- J1 pad 41: unconnected-(J1-Pin_41-Pad41) -> PWM9
- J1 pad 42: PWM6 -> unconnected-(J1-Pin_42-Pad42)
- J1 pad 44: GND -> unconnected-(J1-Pin_44-Pad44)
- J1 pad 48: PWM7 -> unconnected-(J1-Pin_48-Pad48)
- J1 pad 6: PWM0 -> A2
- J1 pad 7: D2 -> Dled2
- J1 pad 9: D3 -> Dswitch1
- J10 pad 10: D5 -> xD4
- J10 pad 12: D6 -> xD5
- J10 pad 14: D7 -> xD6
- J10 pad 16: D8 -> xD7
- J10 pad 2: unconnected-(J10-Pin_2-Pad2) -> xD0
- J10 pad 4: unconnected-(J10-Pin_4-Pad4) -> xD1
- J10 pad 6: unconnected-(J10-Pin_6-Pad6) -> xD2
- J10 pad 8: unconnected-(J10-Pin_8-Pad8) -> xD3
- U4 pad 16: I2C3_SCL -> UART_TX3
- U4 pad 17: I2C3_SDA -> UART_RX3
- U4 pad 18: D1 -> Dswitch1
- U4 pad 19: D2 -> Dswitch2
- U4 pad 25: D9 -> Dleak
- U4 pad 28: SPI_CS4 -> Dled2
- U4 pad 29: SPI_CS3 -> Dled1
- U4 pad 36: D3 -> Dreset
- U4 pad 37: D8 -> Dint

Commit message: layout done
Parts:
- removed H2: MountingHole, MountingHole:MountingHole_3.2mm_M3
- removed J25: PixHawk PM02, Connector_PinSocket_2.54mm:PinSocket_1x06_P2.54mm_Vertical
- removed J26: 3.3V Power, Connector_PinSocket_2.54mm:PinSocket_2x08_P2.54mm_Vertical
- removed J27: 5V Power, Connector_PinSocket_2.54mm:PinSocket_2x08_P2.54mm_Vertical
- added J17: Conn_02x03_Odd_Even, Connector_PinHeader_2.54mm:PinHeader_2x03_P2.54mm_Vertical, F.Cu at (146.4, 122.0)
- added J18: Conn_02x03_Odd_Even, Connector_PinHeader_2.54mm:PinHeader_2x03_P2.54mm_Vertical, F.Cu at (158.8, 122.0)
- added J19: Conn_02x03_Odd_Even, Connector_PinHeader_2.54mm:PinHeader_2x03_P2.54mm_Vertical, F.Cu at (152.6, 122.0)
- added J20: Conn_02x03_Odd_Even, Connector_PinHeader_2.54mm:PinHeader_2x03_P2.54mm_Vertical, F.Cu at (165.0, 122.0)
- added J6: Conn_01x02_Pin, Connector_PinHeader_2.54mm:PinHeader_1x02_P2.54mm_Vertical, B.Cu at (193.8, 123.8)
- added JP1: Jumper_3_Bridged12, Jumper:SolderJumper-3_P1.3mm_Bridged2Bar12_RoundedPad1.0x1.5mm, F.Cu at (183.3, 121.2)
- added JP2: Jumper_3_Bridged12, Jumper:SolderJumper-3_P1.3mm_Bridged2Bar12_RoundedPad1.0x1.5mm, F.Cu at (183.3, 125.4)
- J10: value Conn_02x08_Odd_Even -> Conn_01x17_Pin; footprint Connector_PinSocket_2.54mm:PinSocket_2x08_P2.54mm_Vertical -> Connector_PinHeader_2.54mm:PinHeader_1x17_P2.54mm_Horizontal
- J3, J4, J8: moved to B.Cu
- J7: value Conn_01x24_Pin -> Conn_02x02_Odd_Even; footprint Connector_PinHeader_2.54mm:PinHeader_1x24_P2.54mm_Horizontal -> Connector_PinHeader_2.54mm:PinHeader_2x02_P2.54mm_Vertical
- J9: footprint Connector_PinHeader_1.00mm:PinHeader_1x09_P1.00mm_Vertical -> Connector_PinHeader_2.54mm:PinHeader_1x09_P2.54mm_Vertical; moved to B.Cu
- JP3: value Jumper_2_Open -> Jumper_3_Bridged12; footprint Jumper:SolderJumper-2_P1.3mm_Open_RoundedPad1.0x1.5mm -> Jumper:SolderJumper-3_P1.3mm_Bridged2Bar12_RoundedPad1.0x1.5mm
- U1: value MCP23008-xP -> MCP23008-E_P; footprint Package_DIP:DIP-18_W7.62mm -> Imported Footprints:MCP3008
- moved J7 132.1 mm to (193.9, 64.9)
- moved J3 126.6 mm to (199.8, 72.6), turned to 180 degrees
- moved J4 123.7 mm to (199.9, 99.4)
- moved R4 123.2 mm to (193.4, 85.8), turned to -90 degrees
- moved R5 122.0 mm to (191.1, 85.8), turned to -90 degrees
- moved J8 120.7 mm to (193.4, 107.8), turned to 90 degrees
- moved R3 120.0 mm to (192.4, 91.0)
- moved J9 118.0 mm to (199.9, 105.8), turned to 180 degrees
- moved C4 111.1 mm to (190.4, 69.4), turned to -90 degrees
- moved U5 108.4 mm to (192.4, 95.6), turned to 90 degrees
- moved R2 101.5 mm to (177.6, 124.4), turned to -90 degrees
- moved R1 99.5 mm to (175.4, 124.4), turned to -90 degrees
- moved R7 96.3 mm to (167.0, 100.6)
- moved R6 93.1 mm to (163.4, 97.2), turned to -90 degrees
- moved U3 86.2 mm to (167.0, 97.1)
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Connections:
- J1 pad 10: A3 -> +3.3V
- J1 pad 14: A4 -> I2C1_SCL
- J1 pad 16: GND -> I2C1_SDA
- J1 pad 19: I2C1_SCL -> Net-(J1-Pin_19)
- J1 pad 2: A1 -> A3
- J1 pad 21: I2C1_SDA -> Net-(J1-Pin_21)
- J1 pad 26: unconnected-(J1-Pin_26-Pad26) -> D5
- J1 pad 28: unconnected-(J1-Pin_28-Pad28) -> GND
- J1 pad 30: unconnected-(J1-Pin_30-Pad30) -> xD7
- J1 pad 32: unconnected-(J1-Pin_32-Pad32) -> GND
- J1 pad 34: unconnected-(J1-Pin_34-Pad34) -> xD6
- J1 pad 36: unconnected-(J1-Pin_36-Pad36) -> GND
- J1 pad 38: unconnected-(J1-Pin_38-Pad38) -> +5V
- J1 pad 40: unconnected-(J1-Pin_40-Pad40) -> GND
- J1 pad 42: unconnected-(J1-Pin_42-Pad42) -> +5V
- J1 pad 44: unconnected-(J1-Pin_44-Pad44) -> GND
- J1 pad 46: unconnected-(J1-Pin_46-Pad46) -> +3.3V
- J1 pad 48: unconnected-(J1-Pin_48-Pad48) -> GND
- J1 pad 6: A2 -> A4
- J10 pad 1: GND -> xD0
- J10 pad 10: xD4 -> Ab_s
- J10 pad 11: GND -> Ai_s
- J10 pad 12: xD5 -> Dkill_out
- J10 pad 13: GND -> D3.3v_GE
- J10 pad 14: xD6 -> I2C1_SDA
- J10 pad 15: GND -> I2C1_SCL
- J10 pad 16: xD7 -> GND
- J10 pad 2: xD0 -> xD1
- J10 pad 3: GND -> xD2
- J10 pad 4: xD1 -> xD3
- J10 pad 5: GND -> xD4
- J10 pad 6: xD2 -> xD5
- J10 pad 8: xD3 -> +3.3V
- J10 pad 9: GND -> +5V
- J7 pad 1: GND -> +5V
- J7 pad 2: unconnected-(J7-Pin_2-Pad2) -> I2C2_SCL
- J7 pad 3: PWM0 -> GND
- J7 pad 4: GND -> I2C2_SDA
- JP3 pad 1: +5V -> Net-(JP3-A)
- JP3 pad 2: Net-(JP3-B) -> Net-(JP3-C)
- RN1 pad 1: Dreset -> Net-(JP3-A)
- U1 pad 1: unconnected-(U1-SCL-Pad1) -> I2C2_SCL
- U1 pad 10: unconnected-(U1-GP0-Pad10) -> xD0
- U1 pad 11: unconnected-(U1-GP1-Pad11) -> xD1
- U1 pad 12: unconnected-(U1-GP2-Pad12) -> xD2
- U1 pad 13: unconnected-(U1-GP3-Pad13) -> xD3
- U1 pad 14: unconnected-(U1-GP4-Pad14) -> xD4
- U1 pad 15: unconnected-(U1-GP5-Pad15) -> xD5
- U1 pad 16: unconnected-(U1-GP6-Pad16) -> xD6
- U1 pad 17: unconnected-(U1-GP7-Pad17) -> xD7
- U1 pad 18: unconnected-(U1-VDD-Pad18) -> +5V
- U1 pad 2: unconnected-(U1-SDA-Pad2) -> I2C2_SDA
- U1 pad 3: unconnected-(U1-A2-Pad3) -> GND
- U1 pad 4: unconnected-(U1-A1-Pad4) -> GND
- U1 pad 5: unconnected-(U1-A0-Pad5) -> GND
- U1 pad 6: unconnected-(U1-~{RESET}-Pad6) -> Net-(JP3-C)
- U1 pad 8: unconnected-(U1-INT-Pad8) -> Dint
- U1 pad 9: unconnected-(U1-VSS-Pad9) -> GND
- U4 pad 30: D10 -> Dkill_out
- U4 pad 31: D4 -> D3.3v_GE
- U4 pad 36: Dreset -> D5
- U4 pad 44: A2 -> Ab_s
- U4 pad 45: A1 -> Ai_s
Routing:
- net +5V: track 0.00 -> 179.6 mm, vias 0 -> 2
- net I2C1_SCL: track 0.00 -> 168.0 mm, vias 0 -> 15
- net I2C1_SDA: track 0.00 -> 167.6 mm, vias 0 -> 9
- net I2C2_SCL: track 0.00 -> 104.4 mm, vias 0 -> 2
- net +3.3V: track 0.00 -> 100.4 mm, vias 0 -> 6
- net I2C2_SDA: track 0.00 -> 96.0 mm, vias 0 -> 2
- net A3: track 0.00 -> 91.6 mm, vias 0 -> 3
- net A4: track 0.00 -> 89.5 mm, vias 0 -> 3
- net PWM0: track 0.00 -> 79.9 mm, vias 0 -> 3
- net PWM1: track 0.00 -> 74.9 mm, vias 0 -> 3
- net Dkill_out: track 0.00 -> 71.0 mm, vias 0 -> 4
- net xD6: track 0.00 -> 70.2 mm, vias 0 -> 3
- net PWM2: track 0.00 -> 69.6 mm, vias 0 -> 3
- net D3.3v_GE: track 0.00 -> 67.4 mm, vias 0 -> 2
- net PWM3: track 0.00 -> 65.4 mm, vias 0 -> 3
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- added copper zone on In1.Cu, net +3.3V
- added copper zone on In2.Cu, net GND
Other:
- board size 63 x 71.6 mm -> 65.6 x 74.8 mm
- copper layers 2 -> 4
- board text added: "3.3V"
- board text added: "BAR30"
- board text added: "CS"
- board text added: "ESC Temperature (splits into two)"
- board text added: "Leak Detect"
- board text added: "MISO"
- board text added: "MOSI"
- board text added: "Orin/IMU Temp"
- board text added: "PWM1"
- board text added: "RX1"
- board text added: "SCK"
- board text added: "SCL"
- board text added: "SDA"
- board text added: "Stanford Robosub '25"
- board text added: "TX1"
- board text added: "We are tied to the ocean. And when we go back to the sea, whether it is to sail or to watch it we are going back from whence we came -- John F. Kennedy"
- board text removed: "D1"
- board text removed: "D2"
- board text removed: "D3"
- board text removed: "D4"
- board text removed: "D5"
- board text removed: "D6"
- board text removed: "D7"
- board text removed: "D8"
- board text removed: "D9"
- board text removed: "GND NC PWM"
- board text removed: "T1"
- board text removed: "T2"
- board text removed: "T3"
- board text removed: "T4"
- board text removed: "T5"
- board text removed: "T6"
- board text removed: "T7"
- board text removed: "T8"

Commit message: done with MLU
Parts:
- U3: value BME280 -> PSON65P250X250X100-8N
Connections:
- J1 pad 26: D5 -> Dunused
- U4 pad 22: D5 -> Dunused
Routing:
- net I2C1_SDA: track 167.6 -> 208.9 mm, vias 9 -> 14
- net I2C1_SCL: track 168.0 -> 199.8 mm, vias 15 -> 16
- net UART_RX2: track 8.95 -> 24.9 mm, vias 2 -> 5
- net Dunused: track 0.00 -> 13.1 mm
- net D5: track 32.7 -> 20.3 mm
- net UART_TX2: track 10.6 -> 20.4 mm, vias 2 -> 4
- net BAR_SCL: track 12.5 -> 13.5 mm
- net PWM8: track 64.2 -> 63.1 mm
- net BAR_SDA: track 16.4 -> 17.1 mm
- net D7: track 32.8 -> 33.4 mm
