File: Gen2/MLU_Breakout/MLU_Breakout.kicad_sch (KiCad schematic)
At the start: 31 parts, among them J1 Conn_02x24_Odd_Even, J10 Conn_02x09_Odd_Even, J17 UART, J2 Conn_01x03_Pin, J26 3.3V Power, J27 5V Power, J28 BUS1, J29 BUS2, J3 PixHawk PM02, J30 BUS3, J35 I2C_2, J36 I2C_3, J37 SPI1, J38 SPI2, J39 SPI3, J4 BUS4, J40 SPI4, J5 BUS4, J6 Conn_02x04_Odd_Even, U4 Teensy4.1

Commit message: MLU progress
Parts:
- removed J10: Conn_02x09_Odd_Even, Connector_PinHeader_2.54mm:PinHeader_2x09_P2.54mm_Vertical, symbol Connector_Generic:Conn_02x09_Odd_Even
- removed J17: UART, Connector_PinSocket_2.54mm:PinSocket_1x02_P2.54mm_Vertical, symbol Connector:Conn_01x02_Pin
- removed J28: BUS1, Connector_PinSocket_2.54mm:PinSocket_1x04_P2.54mm_Vertical, symbol Connector:Conn_01x04_Pin
- removed J29: BUS2, Connector_PinSocket_2.54mm:PinSocket_1x04_P2.54mm_Vertical, symbol Connector:Conn_01x04_Pin
- removed J30: BUS3, Connector_PinSocket_2.54mm:PinSocket_1x04_P2.54mm_Vertical, symbol Connector:Conn_01x04_Pin
- removed J35: I2C_2, Connector_PinSocket_2.54mm:PinSocket_1x04_P2.54mm_Vertical, symbol Connector:Conn_01x04_Pin
- removed J36: I2C_3, Connector_PinSocket_2.54mm:PinSocket_1x04_P2.54mm_Vertical, symbol Connector:Conn_01x04_Pin
- removed J37: SPI1, Connector_PinSocket_2.54mm:PinSocket_1x06_P2.54mm_Vertical, symbol Connector:Conn_01x06_Pin
- removed J38: SPI2, Connector_PinSocket_2.54mm:PinSocket_1x06_P2.54mm_Vertical, symbol Connector:Conn_01x06_Pin
- removed J39: SPI3, Connector_PinSocket_2.54mm:PinSocket_1x06_P2.54mm_Vertical, symbol Connector:Conn_01x06_Pin
- removed J40: SPI4, Connector_PinSocket_2.54mm:PinSocket_1x06_P2.54mm_Vertical, symbol Connector:Conn_01x06_Pin
- removed J6: Conn_02x04_Odd_Even, symbol Connector_Generic:Conn_02x04_Odd_Even
- removed JP5: I2C2_PWR, Jumper:SolderJumper-3_P1.3mm_Open_RoundedPad1.0x1.5mm, symbol Jumper:Jumper_3_Bridged12
- removed JP6: I2C3_PWR, Jumper:SolderJumper-3_P1.3mm_Open_RoundedPad1.0x1.5mm, symbol Jumper:Jumper_3_Bridged12
- removed JP7: SPI1_PWR, Jumper:SolderJumper-3_P1.3mm_Open_RoundedPad1.0x1.5mm, symbol Jumper:Jumper_3_Bridged12
- removed JP8: SPI2_PWR, Jumper:SolderJumper-3_P1.3mm_Open_RoundedPad1.0x1.5mm, symbol Jumper:Jumper_3_Bridged12
- added C1, C2: 135p, Capacitor_SMD:C_0603_1608Metric_Pad1.08x0.95mm_HandSolder, symbol Device:C
- added C3, C4: 10uF, Capacitor_SMD:C_0805_2012Metric_Pad1.18x1.45mm_HandSolder, symbol Device:C
- added J10: Conn_02x08_Odd_Even, Connector_PinSocket_2.54mm:PinSocket_2x08_P2.54mm_Vertical, symbol Connector_Generic:Conn_02x08_Odd_Even
- added J6: Conn_01x02_Pin, Connector_PinHeader_2.54mm:PinHeader_1x02_P2.54mm_Vertical, symbol Connector:Conn_01x02_Pin
- added J7: Conn_01x24_Pin, Connector_PinHeader_2.54mm:PinHeader_1x24_P2.54mm_Horizontal, symbol Connector:Conn_01x24_Pin
- added J8: UART, Connector_PinSocket_2.54mm:PinSocket_1x02_P2.54mm_Vertical, symbol Connector:Conn_01x02_Pin
- added J9: Conn_01x09_Pin, Connector_PinHeader_1.00mm:PinHeader_1x09_P1.00mm_Vertical, symbol Connector:Conn_01x09_Pin
- added R2, R3, R4, R5, R6, R7: 10k, Resistor_SMD:R_0805_2012Metric_Pad1.20x1.40mm_HandSolder, symbol Device:R_US
- added RN1: 10kΩ, Resistor_SMD:R_Array_Convex_4x0612, symbol Lab_3:R_Pack04_Split
- added U1: MCP23008-E_P, MCP23008-E_P:DIP254P762X533-18, symbol Imported:MCP23008-E_P
- added U2, U5: MCP9808_MSOP, Package_SO:MSOP-8_3x3mm_P0.65mm, symbol Sensor_Temperature:MCP9808_MSOP
- added U3: BME280, Imported Footprints:BME280, symbol Sensor:BME280
- J4: value BUS4 -> BUS1
- J5: value BUS4 -> BUS2
- JP1: value BUS1_PWR -> Jumper_3_Bridged12; footprint Jumper:SolderJumper-3_P1.3mm_Open_RoundedPad1.0x1.5mm -> Jumper:SolderJumper-3_P1.3mm_Bridged2Bar12_RoundedPad1.0x1.5mm
- JP2: value BUS2_PWR -> Jumper_3_Bridged12; footprint Jumper:SolderJumper-3_P1.3mm_Open_RoundedPad1.0x1.5mm -> Jumper:SolderJumper-3_P1.3mm_Bridged2Bar12_RoundedPad1.0x1.5mm
- R1: value R_US -> 10k; footprint (none) -> Resistor_SMD:R_0805_2012Metric_Pad1.20x1.40mm_HandSolder; Supplier 1 (none) -> https://www.digikey.com/en/products/detail/panasonic-electr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; Supplier 1 S/N (none) -> P10KACT-ND
Connections:
- net I2C3_SCL is gone; now on net UART_TX3: U4.16 (24_A10_TX6_SCL2)
- net I2C3_SDA is gone; now on net UART_RX3: U4.17 (25_A11_RX6_SDA2)
- net SPI_CS3 is gone; now on net Dled1: U4.29 (37_CS)
- net SPI_CS4 is gone; now on net Dled2: U4.28 (36_CS)
- net +3.3V: now also J1.18 (Pin_18), J1.35 (Pin_35), R1.1, R2.1, R3.1, R4.1, R5.1, R6.1, R7.1, U2.8 (V_{DD}), U3.6 (VDDIO), U3.8 (VDD), U5.7 (A0), U5.8 (V_{DD}); no longer JP1.1 (A), JP2.1 (A)
- net +5V: now also C3.1, C4.1, J9.1 (Pin_1), RN1.5 (R4.2), RN1.6 (R3.2), RN1.7 (R2.2), RN1.8 (R1.2), U1.18 (VDD); no longer JP1.3 (B), JP2.3 (B)
- net A1: now also J1.2 (Pin_2)
- net A2: now also J1.6 (Pin_6)
- net A3: now also J1.10 (Pin_10)
- net A4: now also J1.14 (Pin_14)
- net D4: no longer J1.13 (Pin_13)
- net D5: now also J9.4 (Pin_4)
- net D6: now also J9.5 (Pin_5)
- net D7: now also J9.8 (Pin_8)
- net GND: now also J1.12 (Pin_12), J1.16 (Pin_16), J1.29 (Pin_29), J1.37 (Pin_37), J1.4 (Pin_4), C1.2, C2.2, C3.2, C4.2, J10.1 (Pin_1), J10.11 (Pin_11), J10.13 (Pin_13), J10.15 (Pin_15), J10.3 (Pin_3), J10.5 (Pin_5), J10.7 (Pin_7), J10.9 (Pin_9), J7.1 (Pin_1), J7.10 (Pin_10), J7.13 (Pin_13), J7.16 (Pin_16), J7.19 (Pin_19), J7.22 (Pin_22), J7.4 (Pin_4), J7.7 (Pin_7), J9.2 (Pin_2), R3.2, U1.3 (A2), U1.4 (A1), U1.5 (A0), U1.9 (VSS), U2.4 (GND), U2.5 (A2), U2.6 (A1), U2.7 (A0), U3.1 (GND), U3.7 (GND), U5.4 (GND), U5.5 (A2), U5.6 (A1); no longer J1.14 (Pin_14), J1.2 (Pin_2), J1.26 (Pin_26), J1.32 (Pin_32), J1.38 (Pin_38), J1.44 (Pin_44)
- net I2C1_SCL: now also J1.22 (Pin_22), JP1.2 (C), R5.2, U2.2 (SCL), U3.4 (SCK), U5.2 (SCL); no longer J1.19 (Pin_19)
- net I2C1_SDA: now also J1.24 (Pin_24), JP2.2 (C), R4.2, U2.1 (SDA), U3.3 (SDI), U5.1 (SDA); no longer J1.21 (Pin_21)
- net I2C2_SCL: now also C2.1, RN1.3 (R3.1), U1.1 (SCL)
- net I2C2_SDA: now also C1.1, RN1.4 (R4.1), U1.2 (SDA)
- net PWM0: now also J7.3 (Pin_3); no longer J1.6 (Pin_6)
- net PWM1: now also J7.6 (Pin_6); no longer J1.12 (Pin_12)
- net PWM2: now also J7.9 (Pin_9); no longer J1.18 (Pin_18)
- net PWM3: now also J7.12 (Pin_12); no longer J1.24 (Pin_24)
- net PWM4: now also J7.15 (Pin_15); no longer J1.30 (Pin_30)
- net PWM5: now also J7.18 (Pin_18); no longer J1.36 (Pin_36)
- net PWM6: now also J7.21 (Pin_21); no longer J1.42 (Pin_42)
- net PWM7: now also J7.24 (Pin_24); no longer J1.48 (Pin_48)
- net PWM9: now also J1.41 (Pin_41)
- net SPI_CS1: now also J9.3 (Pin_3)
- net SPI_MISO: now also J9.9 (Pin_9)
- net SPI_MOSI: now also J9.6 (Pin_6)
- net SPI_SCK: now also J9.7 (Pin_7)
- net UART_RX1: now also J8.1 (Pin_1)
- net UART_RX2: now also J1.33 (Pin_33), R2.2
- net UART_TX1: now also J8.2 (Pin_2)
- net UART_TX2: now also J1.31 (Pin_31), R1.2
- net UART_TX3: now reaches J1.25 (Pin_25)
- net UART_RX3: now reaches J1.27 (Pin_27)
- net D1 renamed Dled1
- net Dled1: no longer U4.18 (26_A12_MOSI1)
- net D2 renamed Dled2
- net Dled2: no longer U4.19 (27_A13_SCK1)
- net D3 renamed Dreset
- net Dreset: now also RN1.1 (R1.1), U1.6 (*RESET); no longer J1.9 (Pin_9)
- net D8 renamed Dint
- net Dint: now also RN1.2 (R2.1), U1.8 (INT)
- net D9 renamed Dleak
- net SPI_CS2 renamed D10
- new net: J1.21 (Pin_21), JP2.1 (A)
- new net: R7.2, U3.2 (CSB)
- new net: R6.2, U3.5 (SDO)
- new net: J1.19 (Pin_19), JP1.1 (A)
- new net BAR_SCL: J6.2 (Pin_2), JP1.3 (B)
- new net BAR_SDA: J6.1 (Pin_1), JP2.3 (B)
- new net Dswitch1: J1.9 (Pin_9), U4.18 (26_A12_MOSI1)
- new net Dswitch2: J1.13 (Pin_13), U4.19 (27_A13_SCK1)
- new net xD0: J10.2 (Pin_2), U1.10 (GP0)
- new net xD1: J10.4 (Pin_4), U1.11 (GP1)
- new net xD2: J10.6 (Pin_6), U1.12 (GP2)
- new net xD3: J10.8 (Pin_8), U1.13 (GP3)
- new net xD4: J10.10 (Pin_10), U1.14 (GP4)
- new net xD5: J10.12 (Pin_12), U1.15 (GP5)
- new net xD6: J10.14 (Pin_14), U1.16 (GP6)
- new net xD7: J10.16 (Pin_16), U1.17 (GP7)
- no-connect marks 28 -> 32
Other:
- note added: "0x76"
- note added: "2.2" TFT Screen"
- note added: "Address Select"
- note added: "Analog Inputs"
- note added: "Analog Inputs Sonar Localization"
- note added: "Arm"
- note added: "Center leak detector to be mounted on lower board"
- note added: "Display"
- note added: "Display Interface"
- note added: "Downstream pull-up"
- note added: "External LEDs"
- note added: "Extra I2C"
- note added: "For Sonar"
- note added: "GPIO Expander"
- note added: "I2C @ 0x18 format: 0011(A2)(A1)(A0)"
- note added: "I2C @ 0x19 format: 0011(A2)(A1)(A0)"
- note added: "I2C @ 0x20 format: 0100(A2)(A1)(A0)"
- note added: "I2C @ 0x76 when SDO low I2C @ 0x77 when SDO high"
- note added: "Integrated BME280"
- note added: "Integrated MCP9808 #1"
- note added: "Integrated MCP9808 #2"
- note added: "Low Speed Digital Pins"
- note added: "Main I2C Bus"
- note added: "Orin Passthrough"
- note added: "Pixhawk IN"
- note added: "Thruster Interface"
- note added: "UART Arm"
- note added: "UART CTD"
- note added: "UART Main"
- note added: "UART Main Teensy Comms"
- note removed: "4x SPI Bus"
- note removed: "8x I2C Bus"
- note removed: "Analog Pins"
- note removed: "Digital Pins"
- moved on the sheet: H1, H2, H3, H4, J1, J2, J3, J4, J5, U4

Commit message: layout done
Parts:
- removed H2: MountingHole, MountingHole:MountingHole_3.2mm_M3, symbol Mechanical:MountingHole
- removed J10: Conn_02x08_Odd_Even, Connector_PinSocket_2.54mm:PinSocket_2x08_P2.54mm_Vertical, symbol Connector_Generic:Conn_02x08_Odd_Even
- removed J26: 3.3V Power, Connector_PinSocket_2.54mm:PinSocket_2x08_P2.54mm_Vertical, symbol Connector_Generic:Conn_02x08_Odd_Even
- removed J27: 5V Power, Connector_PinSocket_2.54mm:PinSocket_2x08_P2.54mm_Vertical, symbol Connector_Generic:Conn_02x08_Odd_Even
- removed J7: Conn_01x24_Pin, Connector_PinHeader_2.54mm:PinHeader_1x24_P2.54mm_Horizontal, symbol Connector:Conn_01x24_Pin
- added J10: Conn_01x17_Pin, Connector_PinHeader_2.54mm:PinHeader_1x17_P2.54mm_Horizontal, symbol Connector:Conn_01x17_Pin
- added J17, J18, J19, J20: Conn_02x03_Odd_Even, Connector_PinHeader_2.54mm:PinHeader_2x03_P2.54mm_Vertical, symbol Connector_Generic:Conn_02x03_Odd_Even
- added J7: Conn_02x02_Odd_Even, Connector_PinHeader_2.54mm:PinHeader_2x02_P2.54mm_Vertical, symbol Connector_Generic:Conn_02x02_Odd_Even
- added JP3: Jumper_3_Bridged12, Jumper:SolderJumper-3_P1.3mm_Bridged2Bar12_RoundedPad1.0x1.5mm, symbol Jumper:Jumper_3_Bridged12
- J9: footprint Connector_PinHeader_1.00mm:PinHeader_1x09_P1.00mm_Vertical -> Connector_PinHeader_2.54mm:PinHeader_1x09_P2.54mm_Vertical
- U1: footprint MCP23008-E_P:DIP254P762X533-18 -> Imported Footprints:MCP3008
Connections:
- net +3.3V: now also J1.10 (Pin_10), J1.46 (Pin_46), J10.17 (Pin_17), J10.8 (Pin_8)
- net +5V: now also J1.38 (Pin_38), J1.42 (Pin_42), J10.9 (Pin_9), J7.1 (Pin_1)
- net A3: now also J1.2 (Pin_2); no longer J1.10 (Pin_10)
- net A4: now also J1.6 (Pin_6); no longer J1.14 (Pin_14)
- net D5: now also J1.26 (Pin_26), U4.36 (14_A0_TX3_SPDIF_OUT)
- net GND: now also J1.28 (Pin_28), J1.32 (Pin_32), J1.36 (Pin_36), J1.40 (Pin_40), J1.44 (Pin_44), J1.48 (Pin_48), J10.16 (Pin_16), J10.7 (Pin_7), J17.1 (Pin_1), J17.2 (Pin_2), J18.1 (Pin_1), J18.2 (Pin_2), J19.1 (Pin_1), J19.2 (Pin_2), J20.1 (Pin_1), J20.2 (Pin_2), J7.3 (Pin_3), JP3.3 (B); no longer J1.16 (Pin_16)
- net I2C1_SCL: now also J1.14 (Pin_14), J10.15 (Pin_15)
- net I2C1_SDA: now also J1.16 (Pin_16), J10.14 (Pin_14)
- net I2C2_SCL: now also J7.2 (Pin_2)
- net I2C2_SDA: now also J7.4 (Pin_4)
- net PWM0: now also J17.5 (Pin_5)
- net PWM1: now also J17.6 (Pin_6)
- net PWM2: now also J19.5 (Pin_5)
- net PWM3: now also J19.6 (Pin_6)
- net PWM4: now also J18.5 (Pin_5)
- net PWM5: now also J18.6 (Pin_6)
- net PWM6: now also J20.5 (Pin_5)
- net PWM7: now also J20.6 (Pin_6)
- net xD0: now also J10.1 (Pin_1)
- net xD1: now also J10.2 (Pin_2)
- net xD2: now also J10.3 (Pin_3)
- net xD3: now also J10.4 (Pin_4)
- net xD4: now also J10.5 (Pin_5)
- net xD5: now also J10.6 (Pin_6)
- net xD6: now also J1.34 (Pin_34)
- net xD7: now also J1.30 (Pin_30)
- net A1 renamed Ai_s
- net Ai_s: now also J10.11 (Pin_11); no longer J1.2 (Pin_2)
- net A2 renamed Ab_s
- net Ab_s: now also J10.10 (Pin_10); no longer J1.6 (Pin_6)
- net D10 renamed Dkill_out
- net Dkill_out: now also J10.12 (Pin_12)
- net D4 renamed D3.3v_GE
- net D3.3v_GE: now also J10.13 (Pin_13)
- removed net Dreset: RN1.1 (R1.1), U1.6 (*RESET), U4.36 (14_A0_TX3_SPDIF_OUT)
- new net: JP3.1 (A), RN1.1 (R1.1)
- new net: JP3.2 (C), U1.6 (*RESET)
Other:
- note added: "Battery sampling"
- note added: "ESCs"
- note added: "Extra Temp Sensors"
- note added: "FET Temp"
- note added: "Intermediate Signals"
- note added: "Interrupts"
- note added: "Low Speed"
- note added: "Orin/IMU"
- note added: "Power"
- note added: "Power Distrbution Interface"
- note added: "Power Management"
- note added: "Power Management Interface"
- note added: "Sampling"
- note added: "Towards the bulkhead"
- note added: "through the bottom plate"
- note removed: "BME280"
- note removed: "Low Speed Digital Pins"
- moved on the sheet: C1, C2, C3, C4, H1, H3, H4, J1, J2, J3, J4, J5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

Commit message: done with MLU
Connections:
- net D5: no longer J1.26 (Pin_26), U4.22 (30_CRX3)
- new net Dunused: J1.26 (Pin_26), U4.22 (30_CRX3)
Other:
- note added: "ESCs Temp"
- note added: "Orin/IMU Temp"
- note removed: "Address Select"
- note removed: "ESCs"
- note removed: "Extra Temp Sensors"
- note removed: "Orin/IMU"
- moved on the sheet: C1, C2, C3, H1, H3, H4, J10, J17, J18, J19, J2, J20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

Commit message: syncing data
Parts:
- RN1: Supplier 1 P/N CAY16-103J4LFCT-ND -> (none); Supplier 1 S/N (none) -> CAY16-103J4LFCT-ND
Changed lines of the file:
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@@
 			)
 		)
-		(property "Supplier 1 P/N" "CAY16-103J4LFCT-ND"
+		(property "Supplier 1 P/N" ""
 			(at 58.928 121.92 0)
 			(effects
@@
 			)
 		)
-		(property "Supplier 1 S/N" ""
+		(property "Supplier 1 S/N" "CAY16-103J4LFCT-ND"
 			(at 58.928 121.92 0)
 			(effects
@@
 			)
 		)
-		(property "Supplier 1 P/N" "CAY16-103J4LFCT-ND"
+		(property "Supplier 1 P/N" ""
 			(at 51.054 121.92 0)
 			(effects
@@
 			)
 		)
-		(property "Supplier 1 S/N" ""
+		(property "Supplier 1 S/N" "CAY16-103J4LFCT-ND"
 			(at 51.054 121.92 0)
 			(effects
@@
 			)
 		)
-		(property "Supplier 1 P/N" "CAY16-103J4LFCT-ND"
+		(property "Supplier 1 P/N" ""
 			(at 35.052 121.92 0)
 			(effects
@@
 			)
 		)
-		(property "Supplier 1 S/N" ""
+		(property "Supplier 1 S/N" "CAY16-103J4LFCT-ND"
 			(at 35.052 121.92 0)
 			(effects
@@
 			)
 		)
-		(property "Supplier 1 P/N" "CAY16-103J4LFCT-ND"
+		(property "Supplier 1 P/N" ""
 			(at 42.926 121.92 0)
 			(effects
@@
 			)
 		)
-		(property "Supplier 1 S/N" ""
+		(property "Supplier 1 S/N" "CAY16-103J4LFCT-ND"
 			(at 42.926 121.92 0)
 			(effects
