File: 0-Gen2/1-PCBs/MLU_BreakoutV2/MLU_BreakoutV2.kicad_pcb (KiCad board)
At the start: 4 copper layers, 65.6 x 74.8 mm, 45 parts, among them J1 Conn_02x24_Odd_Even, J10 Conn_01x17_Pin, J11 430450228, J12 430450228, J13 430450228, J14 430450228, J15 430450228, J16 430450228, J17 Conn_02x03_Odd_Even, J18 Conn_02x03_Odd_Even, J19 Conn_02x03_Odd_Even, J2 Conn_01x03_Pin, J20 Conn_02x03_Odd_Even, J21 430450228, J22 430450228, J3 PixHawk PM02, J4 BUS1, J5 BUS2, J6 Conn_01x02_Pin, J7 Conn_02x02_Odd_Even, J8 UART, J9 Conn_01x09_Pin, U1 MCP23008-E_P, U2 MCP9808_MSOP, U3 BME280, U4 Teensy4.1, U5 MCP9808_MSOP

Commit message: [add] MLU2 progress, [bugfix] depth sensor
Parts:
- removed J15, J16, J21, J22: 430450228, ImportedV2:CONN_SD-43045-010_02_MOL
- removed JP1, JP2: Jumper_3_Bridged12, Jumper:SolderJumper-3_P1.3mm_Bridged2Bar12_RoundedPad1.0x1.5mm
- removed U1: MCP23008-E_P, Imported Footprints:MCP3008
- added C5: 10uF, Capacitor_SMD:C_0805_2012Metric_Pad1.18x1.45mm_HandSolder, F.Cu at (65.0, 180.7)
- added C6: 0.1uF, ImportedV2:K104K15X7RF5TL2_VIS, F.Cu at (162.3, 85.6)
- added D1: LED, LED_THT:LED_D3.0mm, F.Cu at (63.0, 154.5)
- added D2: LED, LED_THT:LED_D3.0mm, F.Cu at (63.0, 160.0)
- added D3: 1N5817, Diode_THT:D_5W_P12.70mm_Horizontal, F.Cu at (41.9, 149.1)
- added H12: MountingHole, MountingHole:MountingHole_3.2mm_M3, F.Cu at (250.2, 56.9)
- added J23: 430450228, ImportedV2:CONN_SD-43045-001_02_MOL, F.Cu at (195.8, 125.7)
- added J24: 430450228, ImportedV2:CONN_SD-43045-001_02_MOL, F.Cu at (204.7, 125.7)
- added J25: SBH11-PBPC-D10-ST-BK, ImportedV2:SULLINS_SBH11-PBPC-D10-ST-BK, F.Cu at (131.4, 77.9)
- added J26: 430450422, ImportedV2:CONN_SD-43045-008_04_MOL, F.Cu at (177.0, 125.7)
- added LED1: 1655, LED_SMD:LED_LiteOn_LTST-E563C_PLCC4_5.0x5.0mm_P3.2mm_HandSoldering, F.Cu at (79.2, 76.4)
- added LED10: 1655, LED_SMD:LED_LiteOn_LTST-E563C_PLCC4_5.0x5.0mm_P3.2mm_HandSoldering, F.Cu at (251.0, 77.9)
- added LED11: 1655, LED_SMD:LED_LiteOn_LTST-E563C_PLCC4_5.0x5.0mm_P3.2mm_HandSoldering, F.Cu at (251.0, 84.4)
- added LED12: 1655, LED_SMD:LED_LiteOn_LTST-E563C_PLCC4_5.0x5.0mm_P3.2mm_HandSoldering, F.Cu at (251.0, 91.0)
- added LED13: 1655, LED_SMD:LED_LiteOn_LTST-E563C_PLCC4_5.0x5.0mm_P3.2mm_HandSoldering, F.Cu at (251.0, 97.5)
- added LED14: 1655, LED_SMD:LED_LiteOn_LTST-E563C_PLCC4_5.0x5.0mm_P3.2mm_HandSoldering, F.Cu at (251.0, 104.0)
- added LED15: 1655, LED_SMD:LED_LiteOn_LTST-E563C_PLCC4_5.0x5.0mm_P3.2mm_HandSoldering, F.Cu at (251.0, 110.6)
- added LED16: 1655, LED_SMD:LED_LiteOn_LTST-E563C_PLCC4_5.0x5.0mm_P3.2mm_HandSoldering, F.Cu at (251.0, 117.1)
- added LED17: 1655, LED_SMD:LED_LiteOn_LTST-E563C_PLCC4_5.0x5.0mm_P3.2mm_HandSoldering, F.Cu at (251.0, 123.7)
- added LED18: 1655, LED_SMD:LED_LiteOn_LTST-E563C_PLCC4_5.0x5.0mm_P3.2mm_HandSoldering, F.Cu at (251.0, 130.2)
- added LED19: 1655, LED_SMD:LED_LiteOn_LTST-E563C_PLCC4_5.0x5.0mm_P3.2mm_HandSoldering, F.Cu at (251.0, 136.7)
- added LED2: 1655, LED_SMD:LED_LiteOn_LTST-E563C_PLCC4_5.0x5.0mm_P3.2mm_HandSoldering, F.Cu at (79.2, 83.0)
- added LED20: 1655, LED_SMD:LED_LiteOn_LTST-E563C_PLCC4_5.0x5.0mm_P3.2mm_HandSoldering, B.Cu at (251.1, 65.0)
- added LED21: 1655, LED_SMD:LED_LiteOn_LTST-E563C_PLCC4_5.0x5.0mm_P3.2mm_HandSoldering, B.Cu at (251.1, 71.5)
- added LED22: 1655, LED_SMD:LED_LiteOn_LTST-E563C_PLCC4_5.0x5.0mm_P3.2mm_HandSoldering, B.Cu at (251.1, 78.0)
- added LED23: 1655, LED_SMD:LED_LiteOn_LTST-E563C_PLCC4_5.0x5.0mm_P3.2mm_HandSoldering, B.Cu at (251.1, 84.5)
- added LED24: 1655, LED_SMD:LED_LiteOn_LTST-E563C_PLCC4_5.0x5.0mm_P3.2mm_HandSoldering, B.Cu at (251.1, 91.1)
- added LED25: 1655, LED_SMD:LED_LiteOn_LTST-E563C_PLCC4_5.0x5.0mm_P3.2mm_HandSoldering, B.Cu at (251.1, 97.6)
- added LED26: 1655, LED_SMD:LED_LiteOn_LTST-E563C_PLCC4_5.0x5.0mm_P3.2mm_HandSoldering, B.Cu at (251.1, 104.1)
- added LED27: 1655, LED_SMD:LED_LiteOn_LTST-E563C_PLCC4_5.0x5.0mm_P3.2mm_HandSoldering, B.Cu at (251.1, 110.6)
- added LED28: 1655, LED_SMD:LED_LiteOn_LTST-E563C_PLCC4_5.0x5.0mm_P3.2mm_HandSoldering, B.Cu at (251.1, 117.2)
- added LED29: 1655, LED_SMD:LED_LiteOn_LTST-E563C_PLCC4_5.0x5.0mm_P3.2mm_HandSoldering, B.Cu at (251.1, 123.7)
- added LED3: 1655, LED_SMD:LED_LiteOn_LTST-E563C_PLCC4_5.0x5.0mm_P3.2mm_HandSoldering, F.Cu at (79.2, 89.5)
- added LED30: 1655, LED_SMD:LED_LiteOn_LTST-E563C_PLCC4_5.0x5.0mm_P3.2mm_HandSoldering, B.Cu at (251.1, 130.2)
- added LED31: 1655, LED_SMD:LED_LiteOn_LTST-E563C_PLCC4_5.0x5.0mm_P3.2mm_HandSoldering, B.Cu at (251.1, 136.7)
- added LED32: 1655, LED_SMD:LED_LiteOn_LTST-E563C_PLCC4_5.0x5.0mm_P3.2mm_HandSoldering, B.Cu at (130.0, 116.3)
- added LED33: 1655, LED_SMD:LED_LiteOn_LTST-E563C_PLCC4_5.0x5.0mm_P3.2mm_HandSoldering, B.Cu at (130.0, 122.8)
- added LED34: 1655, LED_SMD:LED_LiteOn_LTST-E563C_PLCC4_5.0x5.0mm_P3.2mm_HandSoldering, B.Cu at (130.0, 129.4)
- added LED35: 1655, LED_SMD:LED_LiteOn_LTST-E563C_PLCC4_5.0x5.0mm_P3.2mm_HandSoldering, B.Cu at (130.0, 136.0)
- added LED36: 1655, LED_SMD:LED_LiteOn_LTST-E563C_PLCC4_5.0x5.0mm_P3.2mm_HandSoldering, F.Cu at (100.5, 132.7)
- added LED4: 1655, LED_SMD:LED_LiteOn_LTST-E563C_PLCC4_5.0x5.0mm_P3.2mm_HandSoldering, F.Cu at (130.1, 116.4)
- added LED5: 1655, LED_SMD:LED_LiteOn_LTST-E563C_PLCC4_5.0x5.0mm_P3.2mm_HandSoldering, F.Cu at (130.1, 122.9)
- added LED6: 1655, LED_SMD:LED_LiteOn_LTST-E563C_PLCC4_5.0x5.0mm_P3.2mm_HandSoldering, F.Cu at (130.1, 129.5)
- added LED7: 1655, LED_SMD:LED_LiteOn_LTST-E563C_PLCC4_5.0x5.0mm_P3.2mm_HandSoldering, F.Cu at (130.1, 136.0)
- added LED8: 1655, LED_SMD:LED_LiteOn_LTST-E563C_PLCC4_5.0x5.0mm_P3.2mm_HandSoldering, F.Cu at (251.0, 64.8)
- added LED9: 1655, LED_SMD:LED_LiteOn_LTST-E563C_PLCC4_5.0x5.0mm_P3.2mm_HandSoldering, F.Cu at (251.0, 71.4)
- added R8: 140, Resistor_SMD:R_0805_2012Metric_Pad1.20x1.40mm_HandSolder, F.Cu at (42.1, 142.0)
- added R9: 140, Resistor_SMD:R_0805_2012Metric_Pad1.20x1.40mm_HandSolder, F.Cu at (42.1, 145.0)
- added SW1: 09.03201.02, ImportedV2:09.03201_EAO, F.Cu at (59.3, 155.0)
- added U6: Teensy4.1, Module:Teensy41, F.Cu at (157.4, 104.3)
- added U8: BA033CC0FP-E2, ImportedV2:TO252-3_ROM, F.Cu at (43.9, 155.6)
- J12: value 430450228 -> J1B1211CCD; footprint ImportedV2:CONN_SD-43045-010_02_MOL -> ImportedV2:J1B1211CCD; moved to B.Cu
- J13: value 430450228 -> Conn_02x03_Odd_Even; footprint ImportedV2:CONN_SD-43045-010_02_MOL -> Connector_PinHeader_2.00mm:PinHeader_2x03_P2.00mm_Vertical
- J14: value 430450228 -> 430451027; footprint ImportedV2:CONN_SD-43045-010_02_MOL -> ImportedV2:CONN_SD-43045-010_10_MOL
- J17, J18, J19, J20: value Conn_02x03_Odd_Even -> 430450228; footprint Connector_PinHeader_2.54mm:PinHeader_2x03_P2.54mm_Vertical -> ImportedV2:CONN_SD-43045-001_02_MOL
- J3, J4, J8: moved to F.Cu
- J6: value Conn_01x02_Pin -> 430450422; footprint Connector_PinHeader_2.54mm:PinHeader_1x02_P2.54mm_Vertical -> ImportedV2:CONN_SD-43045-009_04_MOL; moved to F.Cu
- J7: value Conn_02x02_Odd_Even -> SBH11-PBPC-D10-ST-BK; footprint Connector_PinHeader_2.54mm:PinHeader_2x02_P2.54mm_Vertical -> ImportedV2:SULLINS_SBH11-PBPC-D10-ST-BK
- J9: value Conn_01x09_Pin -> 430450422; footprint Connector_PinHeader_2.54mm:PinHeader_1x09_P2.54mm_Vertical -> ImportedV2:CONN_SD-43045-009_04_MOL; moved to F.Cu
- U3: footprint Imported Footprints:BME280 -> ImportedV2:BME280
- moved J11 182.9 mm to (52.4, 171.1)
- moved C4 165.7 mm to (65.0, 177.7), turned to 0 degrees
- moved J4 159.2 mm to (50.4, 154.0)
- moved R4 157.7 mm to (42.1, 130.2), turned to 0 degrees
- moved R5 156.3 mm to (42.1, 133.2), turned to 0 degrees
- moved R3 154.6 mm to (42.1, 127.3)
- moved J9 151.2 mm to (52.0, 137.5), turned to 0 degrees
- moved J3 148.6 mm to (59.8, 122.2), turned to 0 degrees
- moved J6 141.9 mm to (52.0, 127.1), turned to 0 degrees
- moved J8 141.0 mm to (69.7, 175.5), turned to 0 degrees
- moved U4 137.6 mm to (42.8, 110.4), turned to 0 degrees
- moved R2 135.5 mm to (42.1, 124.3), turned to 0 degrees
- moved C3 134.6 mm to (65.0, 174.7)
- moved R1 133.3 mm to (42.1, 121.4), turned to 0 degrees
- moved R7 130.7 mm to (42.1, 139.1)
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Connections:
- J1 pad 1: GND -> unconnected-(J1-Pin_1-Pad1)
- J1 pad 11: +3.3V -> unconnected-(J1-Pin_11-Pad11)
- J1 pad 13: Dswitch2 -> unconnected-(J1-Pin_13-Pad13)
- J1 pad 15: +3.3V -> unconnected-(J1-Pin_15-Pad15)
- J1 pad 17: GND -> unconnected-(J1-Pin_17-Pad17)
- J1 pad 19: Net-(J1-Pin_19) -> unconnected-(J1-Pin_19-Pad19)
- J1 pad 21: Net-(J1-Pin_21) -> unconnected-(J1-Pin_21-Pad21)
- J1 pad 23: +3.3V -> unconnected-(J1-Pin_23-Pad23)
- J1 pad 3: Dled1 -> unconnected-(J1-Pin_3-Pad3)
- J1 pad 37: GND -> unconnected-(J1-Pin_37-Pad37)
- J1 pad 41: PWM9 -> unconnected-(J1-Pin_41-Pad41)
- J1 pad 43: GND -> unconnected-(J1-Pin_43-Pad43)
- J1 pad 47: PWM8 -> unconnected-(J1-Pin_47-Pad47)
- J1 pad 5: GND -> unconnected-(J1-Pin_5-Pad5)
- J1 pad 7: Dled2 -> unconnected-(J1-Pin_7-Pad7)
- J1 pad 9: Dswitch1 -> unconnected-(J1-Pin_9-Pad9)
- J11 pad 1: PWM0 -> unconnected-(J11-Pad1)
- J11 pad 2: GND -> unconnected-(J11-Pad2)
- J12 pad 1: PWM1 -> T+
- J12 pad 2: GND -> Net-(C6-Pad2)
- J13 pad 1: PWM2 -> R+
- J13 pad 2: GND -> R-
- J14 pad 1: PWM3 -> +5V
- J17 pad 1: GND -> +5V
- J17 pad 2: GND -> Net-(D2-A)
- J18 pad 1: GND -> Lumen_PWM
- J19 pad 1: GND -> Dswitch1
- J19 pad 2: GND -> +3.3V
- J20 pad 1: GND -> Dswitch2
- J20 pad 2: GND -> +3.3V
- J6 pad 1: BAR_SDA -> unconnected-(J6-Pad1)
- J6 pad 2: BAR_SCL -> unconnected-(J6-Pad2)
- J7 pad 1: +5V -> PWM0
- J7 pad 2: I2C2_SCL -> I2C1_SCL
- J7 pad 3: GND -> PWM1
- J7 pad 4: I2C2_SDA -> I2C1_SDA
- J9 pad 2: GND -> outNEO_CTRL_ESCs
- J9 pad 3: SPI_CS1 -> toNEO_CTRL_EXTs
- J9 pad 4: D5 -> GND
- J9 pad 5: D6 -> (no net)
- J9 pad 6: SPI_MOSI -> (no net)
Routing:
- net I2C1_SDA: track 208.9 -> 0.00 mm, vias 14 -> 0
- net I2C1_SCL: track 199.8 -> 0.00 mm, vias 16 -> 0
- net +5V: track 179.6 -> 0.00 mm, vias 2 -> 0
- net I2C2_SCL: track 104.4 -> 0.00 mm, vias 2 -> 0
- net +3.3V: track 100.8 -> 0.00 mm, vias 6 -> 0
- net I2C2_SDA: track 96.0 -> 0.00 mm, vias 2 -> 0
- net A3: track 91.6 -> 0.00 mm, vias 3 -> 0
- net A4: track 89.5 -> 0.00 mm, vias 3 -> 0
- net PWM0: track 79.9 -> 0.00 mm, vias 3 -> 0
- net PWM1: track 74.9 -> 0.00 mm, vias 3 -> 0
- net Dkill_out: track 71.0 -> 0.00 mm, vias 4 -> 0
- net xD6: track 70.1 -> 0.00 mm, vias 3 -> 0
- net PWM2: track 69.6 -> 0.00 mm, vias 3 -> 0
- net D3.3v_GE: track 67.4 -> 0.00 mm, vias 2 -> 0
- net PWM3: track 65.4 -> 0.00 mm, vias 3 -> 0
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Other:
- board size 65.6 x 74.8 mm -> 129.3 x 99 mm
- board text added: "ESC Board Interface"
- board text added: "Orin Board Interface"
- board text added: "Screen Connector"
- board text removed: "3.3V"
- board text removed: "5V"
- board text removed: "AnI"
- board text removed: "AnV"
- board text removed: "BAR30"
- board text removed: "CS"
- board text removed: "ESC Temperature (splits into two)"
- board text removed: "GND"
- board text removed: "Leak Detect"
- board text removed: "MISO"
- board text removed: "MOSI"
- board text removed: "Orin/IMU Temp"
- board text removed: "PWM1"
- board text removed: "RX1"
- board text removed: "SCK"
- board text removed: "SCL"
- board text removed: "SDA"
- board text removed: "TX1"

Commit message: [bugfix] depth via BME 0x76 removal, [add] MLUv2 progress
Parts:
- added H10: MountingHole, MountingHole:MountingHole_3.2mm_M3, F.Cu at (24.3, 86.7)
- added H11: MountingHole, MountingHole:MountingHole_3.2mm_M3, F.Cu at (24.3, 94.7)
- added H8: MountingHole, MountingHole:MountingHole_3.2mm_M3, F.Cu at (24.3, 70.8)
- added H9: MountingHole, MountingHole:MountingHole_3.2mm_M3, F.Cu at (24.3, 78.8)
- added J15: 430450228, ImportedV2:CONN_SD-43045-010_02_MOL, F.Cu at (75.5, 138.6)
- added J16: UART, Connector_PinSocket_2.54mm:PinSocket_1x02_P2.54mm_Vertical, F.Cu at (125.3, 182.1)
- added J21: 430450228, ImportedV2:CONN_SD-43045-001_02_MOL, F.Cu at (206.2, 128.7)
- added J22: 430450228, ImportedV2:CONN_SD-43045-001_02_MOL, F.Cu at (222.1, 128.6)
- added J27: ~, Connector_PinSocket_2.54mm:PinSocket_2x04_P2.54mm_Vertical, F.Cu at (199.1, 143.5)
- added JP1: Jumper_3_Bridged12, Jumper:SolderJumper-3_P1.3mm_Bridged2Bar12_RoundedPad1.0x1.5mm, F.Cu at (97.2, 74.4)
- added JP10: Jumper_3_Bridged12, Jumper:SolderJumper-3_P1.3mm_Bridged2Bar12_RoundedPad1.0x1.5mm, F.Cu at (121.5, 175.7)
- added JP11: Jumper_2_Small_Bridged, Jumper:SolderJumper-2_P1.3mm_Bridged2Bar_RoundedPad1.0x1.5mm, F.Cu at (101.4, 168.1)
- added JP12: Jumper_2_Small_Open, Jumper:SolderJumper-2_P1.3mm_Open_RoundedPad1.0x1.5mm, F.Cu at (101.4, 171.6)
- added JP13: Jumper_2_Small_Open, Jumper:SolderJumper-2_P1.3mm_Open_RoundedPad1.0x1.5mm, F.Cu at (101.4, 175.2)
- added JP14: Jumper_2_Small_Bridged, Jumper:SolderJumper-2_P1.3mm_Bridged2Bar_RoundedPad1.0x1.5mm, F.Cu at (105.8, 168.1)
- added JP15: Jumper_2_Small_Open, Jumper:SolderJumper-2_P1.3mm_Open_RoundedPad1.0x1.5mm, F.Cu at (105.8, 171.6)
- added JP16: Jumper_2_Small_Open, Jumper:SolderJumper-2_P1.3mm_Open_RoundedPad1.0x1.5mm, F.Cu at (105.8, 175.2)
- added JP17: Jumper_3_Bridged12, Jumper:SolderJumper-3_P1.3mm_Bridged2Bar12_RoundedPad1.0x1.5mm, F.Cu at (102.1, 178.7)
- added JP18: Jumper_2_Small_Bridged, Jumper:SolderJumper-2_P1.3mm_Bridged2Bar_RoundedPad1.0x1.5mm, F.Cu at (110.1, 168.1)
- added JP19: Jumper_2_Small_Open, Jumper:SolderJumper-2_P1.3mm_Open_RoundedPad1.0x1.5mm, F.Cu at (110.1, 171.6)
- added JP2: Jumper_3_Bridged12, Jumper:SolderJumper-3_P1.3mm_Bridged2Bar12_RoundedPad1.0x1.5mm, F.Cu at (125.8, 188.7)
- added JP20: Jumper_2_Small_Open, Jumper:SolderJumper-2_P1.3mm_Open_RoundedPad1.0x1.5mm, F.Cu at (110.1, 175.2)
- added JP21: Jumper_2_Small_Bridged, Jumper:SolderJumper-2_P1.3mm_Bridged2Bar_RoundedPad1.0x1.5mm, F.Cu at (114.5, 168.1)
- added JP22: Jumper_2_Small_Open, Jumper:SolderJumper-2_P1.3mm_Open_RoundedPad1.0x1.5mm, F.Cu at (114.5, 171.6)
- added JP23: Jumper_2_Small_Open, Jumper:SolderJumper-2_P1.3mm_Open_RoundedPad1.0x1.5mm, F.Cu at (114.5, 175.2)
- added JP24: Jumper_3_Bridged12, Jumper:SolderJumper-3_P1.3mm_Bridged2Bar12_RoundedPad1.0x1.5mm, F.Cu at (102.1, 182.5)
- added JP25: Jumper_2_Small_Open, Jumper:SolderJumper-2_P1.3mm_Open_RoundedPad1.0x1.5mm, F.Cu at (201.9, 148.0)
- added JP26: Jumper_2_Small_Open, Jumper:SolderJumper-2_P1.3mm_Open_RoundedPad1.0x1.5mm, F.Cu at (199.4, 148.0)
- added JP27: Jumper_2_Small_Open, Jumper:SolderJumper-2_P1.3mm_Open_RoundedPad1.0x1.5mm, F.Cu at (196.9, 148.0)
- added JP28: Jumper_2_Small_Open, Jumper:SolderJumper-2_P1.3mm_Open_RoundedPad1.0x1.5mm, F.Cu at (194.3, 148.0)
- added JP29: Jumper_2_Small_Open, Jumper:SolderJumper-2_P1.3mm_Open_RoundedPad1.0x1.5mm, F.Cu at (191.8, 147.9)
- added JP30: Jumper_2_Small_Open, Jumper:SolderJumper-2_P1.3mm_Open_RoundedPad1.0x1.5mm, F.Cu at (189.3, 147.9)
- added JP31: Jumper_2_Small_Open, Jumper:SolderJumper-2_P1.3mm_Open_RoundedPad1.0x1.5mm, F.Cu at (186.8, 147.9)
- added JP32: Jumper_2_Small_Bridged, Jumper:SolderJumper-2_P1.3mm_Bridged2Bar_RoundedPad1.0x1.5mm, F.Cu at (209.4, 150.1)
- added JP33: Jumper_2_Small_Bridged, Jumper:SolderJumper-2_P1.3mm_Bridged2Bar_RoundedPad1.0x1.5mm, F.Cu at (209.4, 153.7)
- added JP34: Jumper_2_Small_Bridged, Jumper:SolderJumper-2_P1.3mm_Bridged2Bar_RoundedPad1.0x1.5mm, F.Cu at (209.4, 157.2)
- added JP35: Jumper_2_Small_Bridged, Jumper:SolderJumper-2_P1.3mm_Bridged2Bar_RoundedPad1.0x1.5mm, F.Cu at (209.4, 160.8)
- added JP36: Jumper_2_Small_Bridged, Jumper:SolderJumper-2_P1.3mm_Bridged2Bar_RoundedPad1.0x1.5mm, F.Cu at (209.4, 164.3)
- added JP37: Jumper_2_Small_Bridged, Jumper:SolderJumper-2_P1.3mm_Bridged2Bar_RoundedPad1.0x1.5mm, F.Cu at (213.7, 150.0)
- added JP38: Jumper_2_Small_Bridged, Jumper:SolderJumper-2_P1.3mm_Bridged2Bar_RoundedPad1.0x1.5mm, F.Cu at (213.8, 153.7)
- added JP39: Jumper_2_Small_Bridged, Jumper:SolderJumper-2_P1.3mm_Bridged2Bar_RoundedPad1.0x1.5mm, F.Cu at (213.8, 157.2)
- added JP4: Jumper_2_Small_Open, Jumper:SolderJumper-2_P1.3mm_Open_RoundedPad1.0x1.5mm, F.Cu at (120.8, 181.6)
- added JP5: Jumper_2_Small_Bridged, Jumper:SolderJumper-2_P1.3mm_Bridged2Bar_RoundedPad1.0x1.5mm, F.Cu at (120.8, 185.1)
- added JP6: Jumper_2_Small_Bridged, Jumper:SolderJumper-2_P1.3mm_Bridged2Bar_RoundedPad1.0x1.5mm, F.Cu at (83.5, 138.9)
- added JP7: Jumper_2_Small_Open, Jumper:SolderJumper-2_P1.3mm_Open_RoundedPad1.0x1.5mm, F.Cu at (120.8, 188.7)
- added JP8: Jumper_3_Bridged12, Jumper:SolderJumper-3_P1.3mm_Bridged2Bar12_RoundedPad1.0x1.5mm, F.Cu at (121.5, 168.1)
- added JP9: Jumper_3_Bridged12, Jumper:SolderJumper-3_P1.3mm_Bridged2Bar12_RoundedPad1.0x1.5mm, F.Cu at (121.5, 171.9)
- added U1: Teensy4.1, Module:Teensy41, F.Cu at (52.6, 57.4)
- C1: value 135p -> 10uF; footprint Capacitor_SMD:C_0603_1608Metric_Pad1.08x0.95mm_HandSolder -> Capacitor_SMD:C_0805_2012Metric_Pad1.18x1.45mm_HandSolder
- C2: value 135p -> 0.1uF; footprint Capacitor_SMD:C_0603_1608Metric_Pad1.08x0.95mm_HandSolder -> ImportedV2:K104K15X7RF5TL2_VIS
- C4, C5: value 10uF -> 135p; footprint Capacitor_SMD:C_0805_2012Metric_Pad1.18x1.45mm_HandSolder -> Capacitor_SMD:C_0603_1608Metric_Pad1.08x0.95mm_HandSolder
- D1: value LED -> 1N5817; footprint LED_THT:LED_D3.0mm -> Diode_THT:D_5W_P12.70mm_Horizontal
- D3: value 1N5817 -> LED; footprint Diode_THT:D_5W_P12.70mm_Horizontal -> LED_THT:LED_D3.0mm
- J1: value Conn_02x24_Odd_Even -> 430450422; footprint Connector_PinSocket_2.54mm:PinSocket_2x24_P2.54mm_Horizontal -> ImportedV2:CONN_SD-43045-009_04_MOL
- J10: value Conn_01x17_Pin -> J1B1211CCD; footprint Connector_PinHeader_2.54mm:PinHeader_1x17_P2.54mm_Horizontal -> ImportedV2:J1B1211CCD
- J11: value 430450228 -> Conn_02x03_Odd_Even; footprint ImportedV2:CONN_SD-43045-010_02_MOL -> Connector_PinHeader_2.00mm:PinHeader_2x03_P2.00mm_Vertical
- J12: value J1B1211CCD -> PixHawk PM02; footprint ImportedV2:J1B1211CCD -> Connector_PinSocket_2.54mm:PinSocket_1x06_P2.54mm_Vertical
- J13: value Conn_02x03_Odd_Even -> SBH11-PBPC-D10-ST-BK; footprint Connector_PinHeader_2.00mm:PinHeader_2x03_P2.00mm_Vertical -> ImportedV2:SULLINS_SBH11-PBPC-D10-ST-BK
- J14: value 430451027 -> 430450422; footprint ImportedV2:CONN_SD-43045-010_10_MOL -> ImportedV2:CONN_SD-43045-009_04_MOL
- J17, J18, J19, J24: value 430450228 -> 430450422; footprint ImportedV2:CONN_SD-43045-001_02_MOL -> ImportedV2:CONN_SD-43045-008_04_MOL
- J2: value Conn_01x03_Pin -> 430450422; footprint Connector_PinHeader_2.54mm:PinHeader_1x03_P2.54mm_Vertical -> ImportedV2:CONN_SD-43045-009_04_MOL
- J25: value SBH11-PBPC-D10-ST-BK -> 430450228; footprint ImportedV2:SULLINS_SBH11-PBPC-D10-ST-BK -> ImportedV2:CONN_SD-43045-001_02_MOL
- J26: value 430450422 -> 430450821; footprint ImportedV2:CONN_SD-43045-008_04_MOL -> ImportedV2:CONN_SD-43045-008_08_MOL
- J3: value PixHawk PM02 -> Conn_01x03_Pin; footprint Connector_PinSocket_2.54mm:PinSocket_1x06_P2.54mm_Vertical -> Connector_PinHeader_2.54mm:PinHeader_1x03_P2.54mm_Vertical
- J4: value BUS1 -> 430450422; footprint Connector_PinSocket_2.54mm:PinSocket_1x04_P2.54mm_Vertical -> ImportedV2:CONN_SD-43045-009_04_MOL
- J5: value BUS2 -> 430451027; footprint Connector_PinSocket_2.54mm:PinSocket_1x04_P2.54mm_Vertical -> ImportedV2:CONN_SD-43045-010_10_MOL
- J6: value 430450422 -> 430450228; footprint ImportedV2:CONN_SD-43045-009_04_MOL -> ImportedV2:CONN_SD-43045-001_02_MOL
- J8: value UART -> Conn_02x20_Odd_Even; footprint Connector_PinSocket_2.54mm:PinSocket_1x02_P2.54mm_Vertical -> Connector_PinSocket_2.54mm:PinSocket_2x20_P2.54mm_Vertical
- J9: value 430450422 -> Conn_01x17_Pin; footprint ImportedV2:CONN_SD-43045-009_04_MOL -> Connector_PinHeader_2.54mm:PinHeader_1x17_P2.54mm_Horizontal
- JP3: value Jumper_3_Bridged12 -> Jumper_2_Small_Open; footprint Jumper:SolderJumper-3_P1.3mm_Bridged2Bar12_RoundedPad1.0x1.5mm -> Jumper:SolderJumper-2_P1.3mm_Open_RoundedPad1.0x1.5mm
- R6, R7: value 10k -> 140
- R8, R9: value 140 -> 10k
- U3: value BME280 -> MCP9808_MSOP; footprint ImportedV2:BME280 -> Package_SO:MSOP-8_3x3mm_P0.65mm
- U4: value Teensy4.1 -> BME280; footprint Module:Teensy41 -> ImportedV2:BME280
- U5: value MCP9808_MSOP -> BA033CC0FP-E2; footprint Package_SO:MSOP-8_3x3mm_P0.65mm -> ImportedV2:TO252-3_ROM
- moved J8 168.5 mm to (202.5, 71.7)
- moved J6 162.2 mm to (214.2, 128.7)
- moved JP3 156.2 mm to (204.5, 147.9), turned to -90 degrees
- moved J1 92.8 mm to (111.9, 152.1)
- moved J25 84.0 mm to (198.3, 128.7), turned to 0 degrees
- moved J24 47.8 mm to (157.0, 128.7)
- moved J5 43.7 mm to (98.6, 152.1)
- moved J26 36.8 mm to (200.0, 154.5)
- moved J23 34.3 mm to (230.0, 128.6)
- moved J18 33.3 mm to (179.2, 128.7)
- moved J20 9.90 mm to (146.0, 128.7)
- moved J17 4.87 mm to (190.3, 128.7)
- moved J19 4.41 mm to (168.1, 128.7)
Connections:
- C1 pad 1: I2C2_SDA -> Net-(D1-A)
- C2 pad 1: I2C2_SCL -> GND
- C2 pad 2: GND -> Net-(C2-Pad2)
- C4 pad 1: +5V -> Net-(JP8-C)
- C5 pad 1: Net-(D2-A) -> Net-(JP9-C)
- D1 pad 1: Net-(D1-K) -> Teensy_5V
- D3 pad 1: Teensy_5V -> Net-(D3-K)
- D3 pad 2: Net-(D2-A) -> Net-(D1-A)
- J1 pad 1: unconnected-(J1-Pin_1-Pad1) -> I2C1_SDA
- J1 pad 2: A3 -> GND
- J1 pad 3: unconnected-(J1-Pin_3-Pad3) -> I2C1_SCL
- J1 pad 4: GND -> Net-(JP1-C)
- J1 pad 5: unconnected-(J1-Pin_5-Pad5) -> (no net)
- J1 pad 6: A4 -> (no net)
- J10 pad 1: xD0 -> T+
- J10 pad 10: Ab_s -> LED
- J10 pad 11: Ai_s -> unconnected-(J10-Pad11)
- J10 pad 12: Dkill_out -> unconnected-(J10-Pad12)
- J10 pad 13: D3.3v_GE -> unconnected-(J10-Pad13)
- J10 pad 14: I2C1_SDA -> unconnected-(J10-Pad14)
- J10 pad 2: xD1 -> Net-(C2-Pad2)
- J10 pad 3: xD2 -> T-
- J10 pad 4: xD3 -> R+
- J10 pad 5: xD4 -> Net-(C2-Pad2)
- J10 pad 6: xD5 -> R-
- J10 pad 7: GND -> unconnected-(J10-Pad7)
- J10 pad 8: +3.3V -> GND
- J10 pad 9: +5V -> GND
- J11 pad 1: unconnected-(J11-Pad1) -> R+
- J11 pad 2: unconnected-(J11-Pad2) -> R-
- J12 pad 1: T+ -> +5V
- J12 pad 2: Net-(C6-Pad2) -> +5V
- J12 pad 3: T- -> Analog_Current
- J12 pad 4: R+ -> Analog_Voltage
- J12 pad 5: Net-(C6-Pad2) -> GND
- J12 pad 6: R- -> GND
- J13 pad 1: R+ -> +5V
- J13 pad 2: R- -> I2C1_SCL
- J13 pad 3: LED -> +5V
- J13 pad 4: GND -> I2C1_SDA
- J13 pad 5: T- -> +5V
- J13 pad 6: T+ -> Dswitch2
- J14 pad 1: +5V -> unconnected-(J14-Pad1)
- J14 pad 2: GND -> unconnected-(J14-Pad2)
- J14 pad 3: SPI_CS1 -> unconnected-(J14-Pad3)
- J14 pad 4: D5 -> unconnected-(J14-Pad4)
- J14 pad 5: D6 -> (no net)
- J14 pad 6: SPI_MOSI -> (no net)
- J17 pad 1: +5V -> I2C1_SDA
- J17 pad 2: Net-(D2-A) -> GND
- J18 pad 1: Lumen_PWM -> UART_RX2
- J19 pad 1: Dswitch1 -> Net-(JP11-B)
- J19 pad 2: +3.3V -> GND
- J2 pad 1: GND -> I2C1_SDA
- J2 pad 2: +3.3V -> GND
- J2 pad 3: Dleak -> I2C1_SCL
- J20 pad 1: Dswitch2 -> Lumen_PWM
- J20 pad 2: +3.3V -> GND
- J23 pad 1: Dled1 -> Dled2
- J24 pad 1: Dled2 -> Net-(JP18-B)
- J25 pad 1: unconnected-(J25-Pad1) -> Dswitch2
- J25 pad 2: I2C1_SCL -> +3.3V
- J26 pad 1: +3.3V -> Net-(JP3-B)
- J26 pad 2: I2C1_SDA -> Net-(JP25-B)
- J26 pad 3: I2C1_SCL -> Net-(JP26-B)
- J26 pad 4: GND -> Net-(JP27-B)
- J26 pad 5: (no net) -> Net-(JP28-B)
- J26 pad 6: (no net) -> Net-(JP29-B)
- J3 pad 1: +5V -> GND
- J3 pad 2: +5V -> +3.3V
- J3 pad 3: Analog_Current -> Dleak
- J4 pad 1: +3.3V -> outNEO_CTRL_ESCs
- J4 pad 3: I2C1_SCL -> toNEO_CTRL_EXTs
- J4 pad 4: I2C1_SDA -> +5V
- J5 pad 1: +3.3V -> +5V
- J5 pad 3: I2C1_SCL -> SPI_CS1
- J5 pad 4: I2C1_SDA -> D5
- J6 pad 1: unconnected-(J6-Pad1) -> +5V
- J6 pad 2: unconnected-(J6-Pad2) -> Net-(D1-A)
- J8 pad 1: UART_RX1 -> +5V
- J8 pad 2: UART_TX1 -> GND
- J9 pad 1: +5V -> xD0
- J9 pad 2: outNEO_CTRL_ESCs -> xD1
- J9 pad 3: toNEO_CTRL_EXTs -> xD2
- J9 pad 4: GND -> xD3
- J9 pad 5: (no net) -> xD4
- J9 pad 6: (no net) -> xD5
- JP3 pad 1: Net-(JP3-A) -> Net-(J27-Pin_8)
- JP3 pad 2: Net-(JP3-C) -> Net-(JP3-B)
- LED1 pad 2: NEO_PASS1 -> NEO_PASS7
- LED10 pad 4: NEO_PASS2 -> Net-(LED10-DOUT)
- LED11 pad 4: NEO_PASS1 -> Net-(LED11-DOUT)
- LED12 pad 4: NEO_PASS3 -> Net-(LED12-DOUT)
- LED13 pad 2: NEO_PASS4 -> Net-(LED13-DIN)
- LED14 pad 2: NEO_PASS3 -> Net-(LED14-DIN)
- LED15 pad 2: NEO_PASS5 -> Net-(LED15-DIN)
- LED16 pad 2: Net-(LED13-DOUT) -> Net-(LED10-DOUT)
- LED17 pad 2: Net-(LED14-DOUT) -> Net-(LED11-DOUT)
- LED18 pad 2: Net-(LED15-DOUT) -> Net-(LED12-DOUT)
- LED19 pad 2: Net-(LED16-DOUT) -> Net-(LED13-DOUT)
- LED19 pad 4: Net-(LED19-DOUT) -> NEO_PASS8
- LED2 pad 2: toNEO_CTRL_MLU -> NEO_PASS6
- LED20 pad 2: Net-(LED17-DOUT) -> Net-(LED14-DOUT)
- LED20 pad 4: Net-(LED20-DOUT) -> NEO_PASS7
- LED21 pad 2: Net-(LED18-DOUT) -> Net-(LED15-DOUT)
- LED21 pad 4: Net-(LED21-DOUT) -> outNEO_CTRL_MLU
- LED22 pad 2: Net-(LED19-DOUT) -> Net-(LED16-DOUT)
- LED22 pad 4: NEO_PASS5 -> NEO_PASS2
- LED23 pad 2: Net-(LED20-DOUT) -> Net-(LED17-DOUT)
- LED23 pad 4: NEO_PASS4 -> NEO_PASS1
- LED24 pad 2: Net-(LED21-DOUT) -> Net-(LED18-DOUT)
- LED24 pad 4: NEO_PASS6 -> NEO_PASS3
- LED25 pad 2: NEO_PASS7 -> NEO_PASS4
- LED26 pad 2: NEO_PASS6 -> NEO_PASS3
- LED27 pad 2: NEO_PASS8 -> NEO_PASS5
- LED3 pad 2: NEO_PASS2 -> NEO_PASS8
- LED34 pad 4: NEO_PASS8 -> NEO_PASS5
- LED35 pad 4: NEO_PASS7 -> NEO_PASS4
- LED36 pad 4: outNEO_CTRL_MLU -> NEO_PASS6
- LED4 pad 2: Net-(LED1-DOUT) -> NEO_PASS1
- LED4 pad 4: Net-(LED4-DOUT) -> Net-(LED10-DIN)
- LED5 pad 2: Net-(LED2-DOUT) -> toNEO_CTRL_MLU
- LED5 pad 4: Net-(LED5-DOUT) -> Net-(LED11-DIN)
- LED6 pad 2: Net-(LED3-DOUT) -> NEO_PASS2
- LED6 pad 4: Net-(LED6-DOUT) -> Net-(LED12-DIN)
- LED7 pad 2: Net-(LED4-DOUT) -> Net-(LED1-DOUT)
- LED7 pad 4: Net-(LED10-DIN) -> Net-(LED13-DIN)
- LED8 pad 2: Net-(LED5-DOUT) -> Net-(LED2-DOUT)
- LED8 pad 4: Net-(LED11-DIN) -> Net-(LED14-DIN)
- LED9 pad 2: Net-(LED6-DOUT) -> Net-(LED3-DOUT)
- LED9 pad 4: Net-(LED12-DIN) -> Net-(LED15-DIN)
- R1 pad 2: UART_TX2 -> Net-(U4-SDO)
- R2 pad 2: UART_RX2 -> Net-(U4-CSB)
- R6 pad 1: +3.3V -> Net-(D2-K)
- R6 pad 2: Net-(U3-SDO) -> GND
- R7 pad 1: +3.3V -> Net-(D3-K)
- R7 pad 2: Net-(U3-CSB) -> GND
- R8 pad 1: Net-(D1-K) -> UART_TX2
- R8 pad 2: GND -> +3.3V
- R9 pad 1: Net-(D2-K) -> UART_RX2
- R9 pad 2: GND -> +3.3V
- RN1 pad 1: Net-(JP3-A) -> Net-(JP10-A)
- RN1 pad 2: Dint -> GPIOExp_INT
- RN1 pad 3: I2C2_SCL -> Net-(JP8-C)
- RN1 pad 4: I2C2_SDA -> Net-(JP9-C)
- SW1 pad 2: Net-(D1-A) -> Net-(D2-A)
- SW1 pad 3: Net-(D2-A) -> Net-(D1-A)
- U3 pad 1: GND -> I2C1_SDA
- U3 pad 2: Net-(U3-CSB) -> I2C1_SCL
- U3 pad 3: I2C1_SDA -> unconnected-(U3-Alert-Pad3)
- U3 pad 4: I2C1_SCL -> GND
- U3 pad 5: Net-(U3-SDO) -> GND
- U3 pad 6: +3.3V -> GND
- U3 pad 7: GND -> +3.3V
- U4 pad 2: PWM0 -> Net-(U4-CSB)
- U4 pad 3: PWM1 -> I2C1_SDA
- U4 pad 4: PWM2 -> I2C1_SCL
- U4 pad 5: PWM3 -> Net-(U4-SDO)
- U4 pad 6: PWM4 -> +3.3V
- U4 pad 7: PWM5 -> GND
- U4 pad 8: PWM6 -> +3.3V
- U5 pad 1: I2C1_SDA -> +5V
- U5 pad 2: I2C1_SCL -> GND
- U5 pad 3: unconnected-(U5-Alert-Pad3) -> +3.3V
- U6 pad 11: toNEO_CTRL_ESCs_M -> unconnected-(U6-9_OUT1C-Pad11)
- U6 pad 12: toNEO_CTRL_ESCs_S -> SPI_CS1
- U6 pad 13: toNEO_CTRL_EXTs -> SPI_MOSI
- U6 pad 14: unconnected-(U6-12_MISO_MQSL-Pad14) -> SPI_MISO
- U6 pad 16: unconnected-(U6-24_A10_TX6_SCL2-Pad16) -> UART_TX3
- U6 pad 17: unconnected-(U6-25_A11_RX6_SDA2-Pad17) -> UART_RX3
- U6 pad 20: unconnected-(U6-28_RX7-Pad20) -> UART_RX2
- U6 pad 21: unconnected-(U6-29_TX7-Pad21) -> UART_TX2
- U6 pad 32: unconnected-(U6-40_A16-Pad32) -> Analog_Voltage
- U6 pad 33: unconnected-(U6-41_A17-Pad33) -> Analog_Current
- U6 pad 35: unconnected-(U6-13_SCK_LED-Pad35) -> SPI_SCK
- U6 pad 36: unconnected-(U6-14_A0_TX3_SPDIF_OUT-Pad36) -> D/A14
- U6 pad 37: unconnected-(U6-15_A1_RX3_SPDIF_IN-Pad37) -> GPIOExp_INT
- U6 pad 38: unconnected-(U6-16_A2_RX4_SCL1-Pad38) -> I2C2_SCL
- U6 pad 39: unconnected-(U6-17_A3_TX4_SDA1-Pad39) -> I2C2_SDA
- U6 pad 42: unconnected-(U6-20_A6_TX5_LRCLK1-Pad42) -> D/A20
- U6 pad 43: unconnected-(U6-21_A7_RX5_BCLK1-Pad43) -> D/A21
- U6 pad 44: unconnected-(U6-22_A8_CTX1-Pad44) -> D/A22
- U6 pad 45: unconnected-(U6-23_A9_CRX1_MCLK1-Pad45) -> D/A23
- U6 pad 56: unconnected-(U6-D--Pad56) -> Host_D-
- U6 pad 57: unconnected-(U6-D+-Pad57) -> Host_D+

Commit message: [changes] MLUv2
Parts:
- removed J11: Conn_02x03_Odd_Even, Connector_PinHeader_2.00mm:PinHeader_2x03_P2.00mm_Vertical
- removed J15: 430450228, ImportedV2:CONN_SD-43045-010_02_MOL
- removed J16: UART, Connector_PinSocket_2.54mm:PinSocket_1x02_P2.54mm_Vertical
- removed U8: BA033CC0FP-E2, ImportedV2:TO252-3_ROM
- added JP40: Jumper_3_Bridged12, Jumper:SolderJumper-3_P1.3mm_Bridged2Bar12_RoundedPad1.0x1.5mm, F.Cu at (69.7, 86.6)
- added JP41: Jumper_2_Small_Bridged, Jumper:SolderJumper-2_P1.3mm_Bridged2Bar_RoundedPad1.0x1.5mm, F.Cu at (43.0, 78.4)
- added JP42: Jumper_2_Small_Open, Jumper:SolderJumper-2_P1.3mm_Open_RoundedPad1.0x1.5mm, F.Cu at (43.0, 81.9)
- added JP43: Jumper_2_Small_Open, Jumper:SolderJumper-2_P1.3mm_Open_RoundedPad1.0x1.5mm, F.Cu at (43.0, 85.5)
- added JP44: Jumper_2_Small_Open, Jumper:SolderJumper-2_P1.3mm_Open_RoundedPad1.0x1.5mm, F.Cu at (43.0, 89.0)
- added JP45: Jumper_2_Small_Open, Jumper:SolderJumper-2_P1.3mm_Open_RoundedPad1.0x1.5mm, F.Cu at (43.0, 92.6)
- added JP46: Jumper_2_Small_Bridged, Jumper:SolderJumper-2_P1.3mm_Bridged2Bar_RoundedPad1.0x1.5mm, F.Cu at (43.0, 96.1)
- added JP47: Jumper_2_Small_Bridged, Jumper:SolderJumper-2_P1.3mm_Bridged2Bar_RoundedPad1.0x1.5mm, F.Cu at (43.0, 99.7)
- added JP48: Jumper_2_Small_Bridged, Jumper:SolderJumper-2_P1.3mm_Bridged2Bar_RoundedPad1.0x1.5mm, F.Cu at (47.4, 71.3)
- added JP49: Jumper_2_Small_Bridged, Jumper:SolderJumper-2_P1.3mm_Bridged2Bar_RoundedPad1.0x1.5mm, F.Cu at (47.4, 74.8)
- added JP50: Jumper_2_Small_Bridged, Jumper:SolderJumper-2_P1.3mm_Bridged2Bar_RoundedPad1.0x1.5mm, F.Cu at (47.4, 78.4)
- added JP51: Jumper_2_Small_Bridged, Jumper:SolderJumper-2_P1.3mm_Bridged2Bar_RoundedPad1.0x1.5mm, F.Cu at (47.4, 81.9)
- added JP52: Jumper_2_Small_Bridged, Jumper:SolderJumper-2_P1.3mm_Bridged2Bar_RoundedPad1.0x1.5mm, F.Cu at (47.4, 85.5)
- added JP53: Jumper_2_Small_Open, Jumper:SolderJumper-2_P1.3mm_Open_RoundedPad1.0x1.5mm, F.Cu at (47.4, 89.0)
- added JP54: Jumper_2_Small_Open, Jumper:SolderJumper-2_P1.3mm_Open_RoundedPad1.0x1.5mm, F.Cu at (47.4, 92.6)
- added JP55: Jumper_2_Small_Open, Jumper:SolderJumper-2_P1.3mm_Open_RoundedPad1.0x1.5mm, F.Cu at (47.4, 96.1)
- added JP56: Jumper_2_Small_Open, Jumper:SolderJumper-2_P1.3mm_Open_RoundedPad1.0x1.5mm, F.Cu at (47.4, 99.7)
- added JP57: Jumper_2_Small_Open, Jumper:SolderJumper-2_P1.3mm_Open_RoundedPad1.0x1.5mm, F.Cu at (51.7, 71.3)
- added JP58: Jumper_2_Small_Open, Jumper:SolderJumper-2_P1.3mm_Open_RoundedPad1.0x1.5mm, F.Cu at (51.7, 74.8)
- added JP59: Jumper_2_Small_Open, Jumper:SolderJumper-2_P1.3mm_Open_RoundedPad1.0x1.5mm, F.Cu at (51.7, 78.4)
- added JP60: Jumper_2_Small_Open, Jumper:SolderJumper-2_P1.3mm_Open_RoundedPad1.0x1.5mm, F.Cu at (51.7, 81.9)
- added JP61: Jumper_2_Small_Open, Jumper:SolderJumper-2_P1.3mm_Open_RoundedPad1.0x1.5mm, F.Cu at (90.3, 85.5)
- added JP62: Jumper_2_Small_Open, Jumper:SolderJumper-2_P1.3mm_Open_RoundedPad1.0x1.5mm, F.Cu at (94.6, 71.3)
- added JP63: Jumper_2_Small_Open, Jumper:SolderJumper-2_P1.3mm_Open_RoundedPad1.0x1.5mm, F.Cu at (94.6, 74.8)
- added JP64: Jumper_2_Small_Open, Jumper:SolderJumper-2_P1.3mm_Open_RoundedPad1.0x1.5mm, F.Cu at (94.6, 78.4)
- added JP65: Jumper_2_Small_Open, Jumper:SolderJumper-2_P1.3mm_Open_RoundedPad1.0x1.5mm, F.Cu at (94.6, 81.9)
- added JP66: Jumper_2_Small_Open, Jumper:SolderJumper-2_P1.3mm_Open_RoundedPad1.0x1.5mm, F.Cu at (94.6, 85.5)
- J10: value J1B1211CCD -> Conn_02x03_Odd_Even; footprint ImportedV2:J1B1211CCD -> Connector_PinHeader_2.00mm:PinHeader_2x03_P2.00mm_Vertical
- J8: value Conn_02x20_Odd_Even -> Conn_02x22_Odd_Even; footprint Connector_PinSocket_2.54mm:PinSocket_2x20_P2.54mm_Vertical -> Connector_PinSocket_2.54mm:PinSocket_2x22_P2.54mm_Vertical
- J9: value Conn_01x17_Pin -> J1B1211CCD; footprint Connector_PinHeader_2.54mm:PinHeader_1x17_P2.54mm_Horizontal -> ImportedV2:J1B1211CCD
- U1: value Teensy4.1 -> BA033CC0FP-E2; footprint Module:Teensy41 -> ImportedV2:TO252-3_ROM
- moved JP38 189.5 mm to (43.0, 71.3)
- moved JP39 189.5 mm to (43.0, 74.8)
- moved JP32 183.8 mm to (38.7, 81.9)
- moved JP33 183.8 mm to (38.7, 85.5)
- moved JP34 183.8 mm to (38.7, 89.0)
- moved JP35 183.8 mm to (38.7, 92.6)
- moved JP36 183.8 mm to (38.7, 96.1)
- moved JP37 182.1 mm to (38.7, 99.7), turned to 0 degrees
- moved JP2 126.7 mm to (69.7, 75.1)
- moved JP22 122.9 mm to (38.7, 74.8)
- moved JP21 122.9 mm to (38.7, 71.3)
- moved JP23 122.9 mm to (38.7, 78.4)
- moved JP12 117.8 mm to (34.3, 74.8)
- moved JP11 117.8 mm to (34.3, 71.3)
- moved JP13 117.8 mm to (34.3, 78.4)
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Connections:
- J1 pad 1: I2C1_SDA -> Net-(JP52-A)
- J1 pad 2: GND -> Net-(JP51-A)
- J1 pad 3: I2C1_SCL -> Net-(JP50-A)
- J1 pad 4: Net-(JP1-C) -> Net-(JP41-A)
- J10 pad 1: T+ -> R+
- J10 pad 2: Net-(C2-Pad2) -> R-
- J10 pad 3: T- -> LED
- J10 pad 4: R+ -> GND
- J10 pad 5: Net-(C2-Pad2) -> T-
- J10 pad 6: R- -> T+
- J13 pad 11: unconnected-(J13-Pad11) -> Net-(JP65-B)
- J13 pad 12: unconnected-(J13-Pad12) -> Net-(JP61-A)
- J13 pad 14: unconnected-(J13-Pad14) -> Net-(JP62-A)
- J13 pad 16: unconnected-(J13-Pad16) -> Net-(JP63-A)
- J13 pad 18: unconnected-(J13-Pad18) -> Net-(JP64-A)
- J13 pad 20: unconnected-(J13-Pad20) -> toNEO_CTRL_Orin
- J13 pad 7: +3.3V -> +5V
- J13 pad 9: unconnected-(J13-Pad9) -> Net-(JP66-B)
- J2 pad 1: I2C1_SDA -> Net-(JP45-B)
- J2 pad 2: GND -> Net-(JP44-B)
- J2 pad 3: I2C1_SCL -> Net-(JP43-B)
- J2 pad 4: Net-(JP2-C) -> Net-(JP42-B)
- J3 pad 3: Dleak -> xDleak
- J4 pad 1: outNEO_CTRL_ESCs -> toNEO_CTRL_EXTs
- J4 pad 3: toNEO_CTRL_EXTs -> outNEO_CTRL_EXTs
- J5 pad 4: D5 -> DISP_RST
- J5 pad 5: D6 -> DISP_DC
- J5 pad 8: D7 -> Net-(JP40-C)
- J7 pad 17: toNEO_CTRL_ESCs_S -> unconnected-(J7-Pad17)
- J7 pad 19: outNEO_CTRL_ESCs_S -> unconnected-(J7-Pad19)
- J7 pad 6: toNEO_CTRL_ESCs_M -> toNEO_CTRL_ESCs
- J7 pad 8: outNEO_CTRL_ESCs_M -> outNEO_CTRL_ESCs
- J8 pad 12: unconnected-(J8-Pin_12-Pad12) -> DISP_LED
- J8 pad 14: unconnected-(J8-Pin_14-Pad14) -> xD0
- J8 pad 16: unconnected-(J8-Pin_16-Pad16) -> xD1
- J8 pad 22: unconnected-(J8-Pin_22-Pad22) -> UART_TX1
- J8 pad 24: unconnected-(J8-Pin_24-Pad24) -> UART_RX1
- J8 pad 25: unconnected-(J8-Pin_25-Pad25) -> Device_D-
- J8 pad 27: unconnected-(J8-Pin_27-Pad27) -> Device_D+
- J8 pad 29: unconnected-(J8-Pin_29-Pad29) -> toNEO_CTRL_ESCs
- J8 pad 31: unconnected-(J8-Pin_31-Pad31) -> outNEO_CTRL_ESCs
- J8 pad 33: unconnected-(J8-Pin_33-Pad33) -> toNEO_CTRL_EXTs
- J8 pad 35: unconnected-(J8-Pin_35-Pad35) -> outNEO_CTRL_EXTs
- J8 pad 36: GND -> xD2
- J8 pad 37: unconnected-(J8-Pin_37-Pad37) -> toNEO_CTRL_MLU
- J8 pad 38: unconnected-(J8-Pin_38-Pad38) -> xD3
- J8 pad 39: unconnected-(J8-Pin_39-Pad39) -> outNEO_CTRL_MLU
- J8 pad 40: unconnected-(J8-Pin_40-Pad40) -> xD4
- J9 pad 1: xD0 -> T+
- J9 pad 10: Ab_s -> LED
- J9 pad 11: Ai_s -> unconnected-(J9-Pad11)
- J9 pad 12: Dkill_out -> unconnected-(J9-Pad12)
- J9 pad 13: D3.3v_GE -> unconnected-(J9-Pad13)
- J9 pad 14: I2C1_SDA -> unconnected-(J9-Pad14)
- J9 pad 2: xD1 -> Net-(C2-Pad2)
- J9 pad 3: xD2 -> T-
- J9 pad 4: xD3 -> R+
- J9 pad 5: xD4 -> Net-(C2-Pad2)
- J9 pad 6: xD5 -> R-
- J9 pad 7: GND -> unconnected-(J9-Pad7)
- J9 pad 8: +3.3V -> GND
- J9 pad 9: +5V -> GND
- U1 pad 1: unconnected-(U1-GND-Pad1) -> +5V
- U1 pad 2: unconnected-(U1-0_RX1_CRX2_CS1-Pad2) -> GND
- U1 pad 3: unconnected-(U1-1_TX1_CTX2_MISO1-Pad3) -> +3.3V
- U6 pad 11: unconnected-(U6-9_OUT1C-Pad11) -> toNEO_CTRL_ESCs
- U6 pad 22: unconnected-(U6-30_CRX3-Pad22) -> DISP_RST
- U6 pad 23: unconnected-(U6-31_CTX3-Pad23) -> DISP_DC
- U6 pad 24: unconnected-(U6-32_OUT1B-Pad24) -> DISP_LED
- U6 pad 25: Dleak -> toNEO_CTRL_Orin
- U6 pad 26: unconnected-(U6-34_RX8-Pad26) -> UART_RX1
- U6 pad 27: unconnected-(U6-35_TX8-Pad27) -> UART_TX1
- U6 pad 30: unconnected-(U6-38_CS1_IN1-Pad30) -> toNEO_CTRL_EXTs
- U6 pad 31: unconnected-(U6-39_MISO1_OUT1A-Pad31) -> toNEO_CTRL_MLU
- U6 pad 66: unconnected-(U6-D--Pad66) -> Device_D-
- U6 pad 67: unconnected-(U6-D+-Pad67) -> Device_D+

Commit message: quick save
Parts:
- moved JP37 178.4 mm to (211.3, 144.8), turned to 90 degrees
- moved JP36 175.4 mm to (207.2, 144.8), turned to 90 degrees
- moved JP35 172.6 mm to (203.2, 144.8), turned to 90 degrees
- moved JP34 169.8 mm to (199.1, 144.8), turned to 90 degrees
- moved JP39 169.3 mm to (206.5, 118.8), turned to 90 degrees
- moved JP33 167.2 mm to (195.1, 144.8), turned to 90 degrees
- moved JP32 164.8 mm to (191.0, 144.8), turned to 90 degrees
- moved JP38 153.3 mm to (188.8, 118.8), turned to -90 degrees
- moved J25 83.5 mm to (233.5, 129.0)
- moved J21 83.4 mm to (241.4, 128.9)
- moved J6 48.3 mm to (209.9, 128.9)
- moved J27 28.8 mm to (201.4, 114.8)
- moved J26 25.6 mm to (202.0, 128.9)
- moved JP25 25.6 mm to (203.9, 122.4)
- moved JP26 25.6 mm to (201.4, 122.4)
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Other:
- outline, holes or cut-outs redrawn
