File: 0-Gen2/1-PCBs/MLU_BreakoutV2/MLU_BreakoutV2.kicad_pcb (KiCad board)
At the start: 4 copper layers, 129.3 x 99 mm, 160 parts, among them J1 430450422, J10 Conn_02x03_Odd_Even, J12 PixHawk PM02, J13 SBH11-PBPC-D10-ST-BK, J14 430450422, J17 430450422, J18 430450422, J19 430450422, J2 430450422, J20 430450228, J21 430450228, J22 430450228, J23 430450228, J24 430450422, J25 430450228, J26 430450821, J3 Conn_01x03_Pin, J4 430450422, J5 430451027, J6 430450228, J7 SBH11-PBPC-D10-ST-BK, J8 Conn_02x22_Odd_Even, J9 J1B1211CCD, SW1 09.03201.02, U1 BA033CC0FP-E2, U2 MCP9808_MSOP, U3 MCP9808_MSOP, U4 BME280, U5 BA033CC0FP-E2, U6 Teensy4.1

Commit message: [add] major layout updates
Parts:
- removed J24: 430450422, ImportedV2:CONN_SD-43045-008_04_MOL
- removed U5: BA033CC0FP-E2, ImportedV2:TO252-3_ROM
- added C7: 1uF, Capacitor_SMD:C_0805_2012Metric_Pad1.18x1.45mm_HandSolder, F.Cu at (237.8, 107.0)
- added J11: 430450422, ImportedV2:CONN_SD-43045-008_04_MOL, F.Cu at (151.7, 128.9)
- added J31: Conn_01x02_Socket, Connector_PinSocket_2.54mm:PinSocket_1x02_P2.54mm_Vertical, F.Cu at (171.2, 108.5)
- C6: value 0.1uF -> 10uF; footprint ImportedV2:K104K15X7RF5TL2_VIS -> Capacitor_SMD:C_0805_2012Metric_Pad1.18x1.45mm_HandSolder
- J14: value 430450422 -> Conn_01x02_Socket; footprint ImportedV2:CONN_SD-43045-009_04_MOL -> Connector_PinSocket_2.54mm:PinSocket_1x02_P2.54mm_Vertical
- JP11, JP14, JP18, JP21: value Jumper_2_Small_Bridged -> Jumper_2_Small_Open; footprint Jumper:SolderJumper-2_P1.3mm_Bridged2Bar_RoundedPad1.0x1.5mm -> Connector_PinHeader_1.27mm:PinHeader_1x02_P1.27mm_Vertical
- JP12, JP13, JP15, JP16, JP19, JP20, JP22, JP23, JP25, JP26, JP27, JP28, JP29, JP3, JP30, JP31, JP57, JP59, JP60: footprint Jumper:SolderJumper-2_P1.3mm_Open_RoundedPad1.0x1.5mm -> Connector_PinHeader_1.27mm:PinHeader_1x02_P1.27mm_Vertical
- JP17: footprint Jumper:SolderJumper-3_P1.3mm_Bridged2Bar12_RoundedPad1.0x1.5mm -> Connector_PinHeader_1.27mm:PinHeader_1x03_P1.27mm_Vertical
- JP24: value Jumper_3_Bridged12 -> Jumper_2_Small_Open; footprint Jumper:SolderJumper-3_P1.3mm_Bridged2Bar12_RoundedPad1.0x1.5mm -> Connector_PinHeader_1.27mm:PinHeader_1x02_P1.27mm_Vertical
- JP32, JP33, JP34, JP35, JP36, JP37, JP38, JP39: footprint Jumper:SolderJumper-2_P1.3mm_Bridged2Bar_RoundedPad1.0x1.5mm -> Connector_PinHeader_1.27mm:PinHeader_1x02_P1.27mm_Vertical
- JP58: value Jumper_2_Small_Open -> Jumper_3_Bridged12; footprint Jumper:SolderJumper-2_P1.3mm_Open_RoundedPad1.0x1.5mm -> Connector_PinHeader_1.27mm:PinHeader_1x03_P1.27mm_Vertical
- moved U1 154.8 mm to (239.1, 116.5), turned to 180 degrees
- moved D1 147.6 mm to (229.9, 106.9), turned to -90 degrees
- moved JP13 145.0 mm to (175.3, 112.1), turned to -90 degrees
- moved JP14 144.9 mm to (175.3, 115.3), turned to -90 degrees
- moved JP15 144.8 mm to (175.3, 118.5), turned to -90 degrees
- moved JP16 144.7 mm to (175.3, 121.7), turned to -90 degrees
- moved C1 143.4 mm to (225.4, 110.0), turned to -90 degrees
- moved JP11 143.3 mm to (170.7, 115.3), turned to -90 degrees
- moved JP12 140.1 mm to (169.4, 112.1), turned to 90 degrees
- moved JP59 125.5 mm to (170.7, 118.5), turned to -90 degrees
- moved JP60 125.4 mm to (170.7, 121.7), turned to -90 degrees
- moved SW1 125.3 mm to (215.7, 108.9), turned to 90 degrees
- moved D2 122.9 mm to (217.0, 114.7)
- moved D3 122.8 mm to (217.0, 119.5)
- moved JP21 121.4 mm to (153.1, 112.1), turned to -90 degrees
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Connections:
- C6 pad 1: GND -> +3.3V
- C6 pad 2: Net-(C6-Pad2) -> GND
- J14 pad 1: unconnected-(J14-Pad1) -> Net-(J14-Pin_1)
- J14 pad 2: unconnected-(J14-Pad2) -> Net-(J14-Pin_2)
- J19 pad 1: Net-(JP11-B) -> Net-(JP13-B)
- J19 pad 3: Net-(JP14-A) -> Net-(JP11-A)
- JP11 pad 1: I2C1_SDA -> Net-(JP11-A)
- JP11 pad 2: Net-(JP11-B) -> I2C1_SCL
- JP12 pad 1: Net-(JP11-B) -> Net-(J31-Pin_1)
- JP12 pad 2: D/A20 -> Net-(JP11-A)
- JP13 pad 1: Net-(JP11-B) -> Net-(J31-Pin_2)
- JP13 pad 2: D/A22 -> Net-(JP13-B)
- JP14 pad 1: Net-(JP14-A) -> I2C1_SDA
- JP14 pad 2: I2C1_SDA -> Net-(JP13-B)
- JP15 pad 1: D/A21 -> D/A22
- JP15 pad 2: Net-(JP14-A) -> Net-(JP13-B)
- JP16 pad 1: D/A23 -> D/A20
- JP16 pad 2: Net-(JP14-A) -> Net-(JP13-B)
- JP19 pad 1: Net-(JP18-B) -> D/A20
- JP19 pad 2: D/A20 -> Net-(JP18-B)
- JP20 pad 1: Net-(JP18-B) -> D/A22
- JP20 pad 2: D/A22 -> Net-(JP18-B)
- JP21 pad 1: Net-(JP21-A) -> Net-(J14-Pin_2)
- JP21 pad 2: I2C1_SDA -> Net-(JP18-B)
- JP22 pad 1: D/A21 -> Net-(J14-Pin_1)
- JP22 pad 2: Net-(JP21-A) -> Net-(JP22-B)
- JP23 pad 1: D/A23 -> Net-(JP22-B)
- JP23 pad 2: Net-(JP21-A) -> I2C1_SCL
- JP24 pad 1: +3.3V -> Net-(JP22-B)
- JP24 pad 2: Net-(JP24-C) -> D/A21
- JP32 pad 1: Net-(JP28-B) -> UART_RX3
- JP32 pad 2: Host_D+ -> Net-(JP30-B)
- JP33 pad 1: Net-(JP27-B) -> UART_TX3
- JP33 pad 2: Host_D- -> Net-(JP29-B)
- JP34 pad 1: Net-(JP26-B) -> Net-(JP3-B)
- JP34 pad 2: I2C1_SCL -> +5V
- JP36 pad 1: UART_TX3 -> Net-(JP26-B)
- JP36 pad 2: Net-(JP29-B) -> I2C1_SCL
- JP37 pad 1: UART_RX3 -> Net-(JP27-B)
- JP37 pad 2: Net-(JP30-B) -> Host_D-
- JP39 pad 1: Net-(JP3-B) -> Net-(JP28-B)
- JP39 pad 2: +5V -> Host_D+
- JP57 pad 1: Net-(JP18-B) -> Net-(JP22-B)
- JP57 pad 2: unconnected-(JP57-B-Pad2) -> D/A23
- JP58 pad 1: Net-(JP21-A) -> +3.3V
- JP58 pad 2: unconnected-(JP58-B-Pad2) -> Net-(JP58-C)
- JP59 pad 1: Net-(JP11-B) -> Net-(JP11-A)
- JP59 pad 2: Net-(J31-Pin_2) -> D/A23
- JP60 pad 1: Net-(JP14-A) -> Net-(JP11-A)
- JP60 pad 2: Net-(J31-Pin_1) -> D/A21
Other:
- board text added: "+3.3V"
- board text added: "+5V"
- board text added: "Arm Enclosure Interconnect"
- board text added: "Blank Bus (I2C Nominal)"
- board text added: "BlueRobotics Depth"
- board text added: "D/A20"
- board text added: "D/A21"
- board text added: "D/A22"
- board text added: "D/A23"
- board text added: "Data Log Switch"
- board text added: "GND"
- board text added: "Host_D+"
- board text added: "Host_D-"
- board text added: "I2C1 SCL"
- board text added: "I2C1 SDA"
- board text added: "I2C1_SCL"
- board text added: "I2C1_SDA"
- board text added: "Kill Switch"
- board text added: "LED1"
- board text added: "LED2"
- board text added: "Lumen PWM"
- board text added: "Pin1"
- board text added: "Pin2"
- board text added: "Pin7"
- board text added: "Pin8"
- board text added: "StarOddi CTD"
- board text added: "Teensy Off"
- board text added: "Teensy On"
- board text added: "Teensy PWR Off"
- board text added: "Teensy PWR On"
- board text added: "Teensy Reset"
- board text added: "UART_RX3"
- board text added: "UART_TX3"
- board text removed: "Screen Connector"

Commit message: [final pass] MLU breakout
Parts:
- removed H10, H11: MountingHole, MountingHole:MountingHole_3.2mm_M3
- removed J1: 430450422, ImportedV2:CONN_SD-43045-009_04_MOL
- removed JP1: Jumper_3_Bridged12, Jumper:SolderJumper-3_P1.3mm_Bridged2Bar12_RoundedPad1.0x1.5mm
- removed JP54, JP55, JP56, JP61, JP62, JP63, JP64, JP65, JP66: Jumper_2_Small_Open, Jumper:SolderJumper-2_P1.3mm_Open_RoundedPad1.0x1.5mm
- added J28: Conn_01x04_Socket, Connector_PinSocket_2.54mm:PinSocket_1x04_P2.54mm_Vertical, F.Cu at (192.8, 71.0)
- added JP67: Jumper_2_Small_Open, Connector_PinHeader_1.27mm:PinHeader_1x02_P1.27mm_Vertical, F.Cu at (191.9, 74.7)
- added U7: MCP23008-E_P, ImportedV2:MCP3008, F.Cu at (235.3, 71.9)
- H8, H9: value MountingHole -> ~
- J12: moved to F.Cu
- JP10, JP2, JP40, JP8, JP9: footprint Jumper:SolderJumper-3_P1.3mm_Bridged2Bar12_RoundedPad1.0x1.5mm -> Connector_PinHeader_1.27mm:PinHeader_1x03_P1.27mm_Vertical
- JP41, JP49, JP50, JP51, JP52: value Jumper_2_Small_Bridged -> Jumper_2_Small_Open; footprint Jumper:SolderJumper-2_P1.3mm_Bridged2Bar_RoundedPad1.0x1.5mm -> Connector_PinHeader_1.27mm:PinHeader_1x02_P1.27mm_Vertical
- JP42, JP43, JP44, JP53: footprint Jumper:SolderJumper-2_P1.3mm_Open_RoundedPad1.0x1.5mm -> Connector_PinHeader_1.27mm:PinHeader_1x02_P1.27mm_Vertical
- JP45: value Jumper_2_Small_Open -> Jumper_2_Small_Bridged; footprint Jumper:SolderJumper-2_P1.3mm_Open_RoundedPad1.0x1.5mm -> Connector_PinHeader_1.27mm:PinHeader_1x02_P1.27mm_Vertical
- JP46, JP47, JP48: footprint Jumper:SolderJumper-2_P1.3mm_Bridged2Bar_RoundedPad1.0x1.5mm -> Connector_PinHeader_1.27mm:PinHeader_1x02_P1.27mm_Vertical
- LED1, LED2: moved to B.Cu
- moved J3 210.7 mm to (242.8, 58.7), turned to 180 degrees
- moved C3 180.1 mm to (245.5, 72.8), turned to -90 degrees
- moved H8 178.5 mm to (222.8, 74.4)
- moved H9 175.9 mm to (222.8, 89.4)
- moved JP40 174.8 mm to (206.3, 87.3)
- moved JP8 169.6 mm to (230.3, 71.4)
- moved JP9 168.9 mm to (230.3, 76.8)
- moved JP2 167.4 mm to (198.1, 81.5), turned to -90 degrees
- moved C4 166.5 mm to (233.1, 73.5), turned to -90 degrees
- moved JP10 166.4 mm to (230.2, 87.2)
- moved JP44 165.7 mm to (203.1, 74.7), turned to -90 degrees
- moved C5 165.6 mm to (233.1, 78.3), turned to -90 degrees
- moved RN1 164.0 mm to (230.2, 83.2), turned to 180 degrees
- moved JP43 161.0 mm to (199.4, 74.7), turned to -90 degrees
- moved J2 160.0 mm to (194.9, 61.3), turned to 180 degrees
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Connections:
- C2 pad 1: GND -> ETH_GND
- J10 pad 4: GND -> ETH_GND
- J13 pad 11: Net-(JP65-B) -> Net-(JP41-B)
- J13 pad 12: Net-(JP61-A) -> Net-(JP50-B)
- J13 pad 14: Net-(JP62-A) -> Net-(JP51-B)
- J13 pad 16: Net-(JP63-A) -> Net-(JP52-B)
- J13 pad 18: Net-(JP64-A) -> Net-(JP53-B)
- J13 pad 9: Net-(JP66-B) -> Net-(JP49-B)
- J2 pad 1: Net-(JP45-B) -> Net-(JP45-A)
- J2 pad 2: Net-(JP44-B) -> Net-(JP42-B)
- J2 pad 4: Net-(JP42-B) -> Net-(JP44-B)
- J9 pad 8: GND -> ETH_GND
- J9 pad 9: GND -> ETH_GND
- JP41 pad 1: Net-(JP41-A) -> Device_D+
- JP41 pad 2: Net-(JP1-C) -> Net-(JP41-B)
- JP42 pad 1: unconnected-(JP42-A-Pad1) -> Net-(J28-Pin_3)
- JP43 pad 1: unconnected-(JP43-A-Pad1) -> Net-(J28-Pin_2)
- JP44 pad 1: unconnected-(JP44-A-Pad1) -> Net-(J28-Pin_1)
- JP45 pad 1: unconnected-(JP45-A-Pad1) -> Net-(JP45-A)
- JP45 pad 2: Net-(JP45-B) -> I2C1_SDA
- JP46 pad 1: Net-(JP44-B) -> Net-(JP42-B)
- JP48 pad 1: Net-(JP45-B) -> Net-(JP44-B)
- JP48 pad 2: I2C1_SDA -> Net-(JP2-C)
- JP49 pad 1: Net-(JP42-B) -> Device_D-
- JP49 pad 2: Net-(JP2-C) -> Net-(JP49-B)
- JP50 pad 1: Net-(JP50-A) -> D/A23
- JP50 pad 2: I2C1_SCL -> Net-(JP50-B)
- JP51 pad 1: Net-(JP51-A) -> D/A22
- JP51 pad 2: GND -> Net-(JP51-B)
- JP52 pad 1: Net-(JP52-A) -> D/A21
- JP52 pad 2: I2C1_SDA -> Net-(JP52-B)
- JP53 pad 1: Net-(J29-Pin_4) -> D/A20
- JP53 pad 2: Net-(JP52-A) -> Net-(JP53-B)
- U6 pad 64: GND -> ETH_GND
Routing:
- removed copper zone on In1.Cu, net +3.3V
- removed copper zone on In2.Cu, net GND
Other:
- board text added: "+5V_Pullup"
- board text added: "15mm (screen mount)"
- board text added: "3.3V Regulator"
- board text added: "A_I"
- board text added: "A_V"
- board text added: "Backup Power In"
- board text added: "Configureable Blank"
- board text added: "DISP_DC"
- board text added: "DISP_LED"
- board text added: "DISP_RST"
- board text added: "Display Interface"
- board text added: "ESC Interface"
- board text added: "Ethernet Jumper"
- board text added: "External Neo Interface"
- board text added: "GPIO Expander"
- board text added: "Humidity Sensor"
- board text added: "I2C1 Pullup"
- board text added: "I2C2_SCL"
- board text added: "I2C2_SDA"
- board text added: "Leak"
- board text added: "Orin Interface"
- board text added: "Pin1 (R+)"
- board text added: "Pin19"
- board text added: "Pin20"
- board text added: "Pin6 (T+)"
- board text added: "RX_Pullup"
- board text added: "SPI_CS1"
- board text added: "SPI_MISO"
- board text added: "SPI_MOSI"
- board text added: "SPI_SCK"
- board text added: "TX_Pullup"
- board text added: "xDleak"
- board text removed: "ESC Board Interface"
- board text removed: "Orin Board Interface"

Commit message: [add] beginning routing
Parts:
- moved LED36 121.7 mm to (251.1, 84.6)
- moved LED11 121.6 mm to (130.2, 70.3)
- moved LED5 59.2 mm to (130.1, 63.8)
- moved LED3 59.1 mm to (130.0, 122.8)
- moved J8 2.54 mm to (169.3, 100.6)
- moved U6 0.70 mm to (157.1, 83.4)
Connections:
- J8 pad 22: UART_TX1 -> UART_RX1
- J8 pad 24: UART_RX1 -> UART_TX1
Routing:
- net GND: track 0.00 -> 845.7 mm, vias 0 -> 18
- net +5V: track 0.00 -> 807.3 mm, vias 0 -> 7
- net +3.3V: track 0.00 -> 248.8 mm, vias 0 -> 1
- net Teensy_5V: track 0.00 -> 118.7 mm, vias 0 -> 1
- net D/A22: track 0.00 -> 88.1 mm, vias 0 -> 5
- net D/A23: track 0.00 -> 81.6 mm, vias 0 -> 3
- net D/A21: track 0.00 -> 79.3 mm, vias 0 -> 2
- net I2C1_SDA: track 0.00 -> 76.0 mm, vias 0 -> 2
- net D/A20: track 0.00 -> 69.1 mm, vias 0 -> 2
- net UART_RX2: track 0.00 -> 65.8 mm, vias 0 -> 3
- net I2C1_SCL: track 0.00 -> 65.4 mm, vias 0 -> 4
- net UART_TX2: track 0.00 -> 64.6 mm, vias 0 -> 3
- net Lumen_PWM: track 0.00 -> 43.8 mm
- net R-: track 0.00 -> 43.5 mm
- net R+: track 0.00 -> 42.3 mm
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Other:
- board text added: "D/A14"
- board text added: "Device_D+"
- board text added: "Device_D-"
- board text added: "UART_RX1"
- board text added: "UART_RX2"
- board text added: "UART_TX1"
- board text added: "UART_TX2"
- board text added: "oNeo_ESCs"
- board text added: "oNeo_EXTs"
- board text added: "oNeo_MLU"
- board text added: "tNeo_ESCs"
- board text added: "tNeo_EXTs"
- board text added: "tNeo_MLU"
- board text added: "xD0"
- board text added: "xD1"
- board text added: "xD2"
- board text added: "xD3"
- board text added: "xD4"
- board text added: "xD5"
- board text added: "xD6"

Commit message: before restructure
Parts:
- renumbered J9 to J3, J10 to J4, U6 to U1, U1 to U17
