File: 0-Gen2/1-PCBs/MLU_BreakoutV2/NEOs.kicad_sch (KiCad schematic)
At the start: 36 parts

Commit message: [bugfix] depth via BME 0x76 removal, [add] MLUv2 progress
Parts:
- renumbered LED25 to LED1, LED4 to LED10, LED5 to LED11, LED6 to LED12, LED31 to LED13, LED32 to LED14, LED33 to LED15, LED7 to LED16, LED8 to LED17, LED9 to LED18, LED34 to LED19, LED26 to LED2, LED35 to LED20, LED36 to LED21, LED10 to LED22, LED11 to LED23, LED12 to LED24, LED13 to LED25, LED14 to LED26, LED15 to LED27, LED16 to LED28, LED17 to LED29, LED27 to LED3, LED18 to LED30, LED19 to LED31, LED20 to LED32, LED21 to LED33, LED22 to LED34, LED23 to LED35, LED24 to LED36, LED1 to LED4, LED2 to LED5, LED3 to LED6, LED28 to LED7, LED29 to LED8, LED30 to LED9
Connections:
- net outNEO_CTRL_MLU renamed outNEO_MLU
- net toNEO_CTRL_MLU renamed toNEO_MLU

Commit message: routing
Parts:
- renumbered LED5 to LED1, LED12 to LED10, LED18 to LED11, LED24 to LED12, LED26 to LED13, LED29 to LED14, LED32 to LED15, LED35 to LED16, LED25 to LED17, LED28 to LED18, LED31 to LED19, LED11 to LED2, LED34 to LED20, LED27 to LED21, LED30 to LED22, LED33 to LED23, LED36 to LED24, LED2 to LED25, LED8 to LED26, LED14 to LED27, LED20 to LED28, LED1 to LED29, LED17 to LED3, LED7 to LED30, LED13 to LED31, LED19 to LED32, LED3 to LED33, LED9 to LED34, LED15 to LED35, LED21 to LED36, LED23 to LED4, LED4 to LED5, LED10 to LED6, LED16 to LED7, LED22 to LED8, LED6 to LED9
