File: 0-Gen2/1-PCBs/MLU_BreakoutV2/sensors.kicad_sch (KiCad schematic)
At the start: 6 parts, among them U2 MCP9808_MSOP, U3 MCP9808_MSOP, U4 BME280

Commit message: [changes] MLUv2
Changed lines of the file:
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@@
 		)
 	)
-	(global_label "I2C1_SCL"
+	(hierarchical_label "I2C1_SDA"
+		(shape bidirectional)
+		(at 33.02 32.258 180)
+		(fields_autoplaced yes)
+		(effects
+			(font
+				(size 1.27 1.27)
+			)
+			(justify right)
+		)
+	)
+	(hierarchical_label "I2C1_SDA"
+		(shape bidirectional)
+		(at 83.312 32.512 180)
+		(fields_autoplaced yes)
+		(effects
+			(font
+				(size 1.27 1.27)
+			)
+			(justify right)
+		)
+	)
+	(hierarchical_label "I2C1_SCL"
+		(shape input)
+		(at 144.526 37.592 180)
+		(fields_autoplaced yes)
+		(effects
+			(font
+				(size 1.27 1.27)
+			)
+			(justify right)
+		)
+	)
+	(hierarchical_label "I2C1_SCL"
 		(shape input)
 		(at 33.02 34.798 180)
@@
 			(justify right)
 		)
-		(property "Intersheetrefs" "${INTERSHEET_REFS}"
-			(at 21.2658 34.798 0)
-			(effects
-				(font
-					(size 1.27 1.27)
-				)
-				(justify right)
-				(hide yes)
-			)
-		)
 	)
-	(global_label "I2C1_SDA"
-		(shape bidirectional)
-		(at 33.02 32.258 180)
-		(fields_autoplaced yes)
-		(effects
-			(font
-				(size 1.27 1.27)
-			)
-			(justify right)
-		)
-		(property "Intersheetrefs" "${INTERSHEET_REFS}"
-			(at 20.094 32.258 0)
-			(effects
-				(font
-					(size 1.27 1.27)
-				)
-				(justify right)
-				(hide yes)
-			)
-		)
-	)
-	(global_label "I2C1_SDA"
+	(hierarchical_label "I2C1_SDA"
 		(shape bidirectional)
 		(at 144.272 42.672 180)
@@
 			(justify right)
 		)
-		(property "Intersheetrefs" "${INTERSHEET_REFS}"
-			(at 131.346 42.672 0)
-			(effects
-				(font
-					(size 1.27 1.27)
-				)
-				(justify right)
-				(hide yes)
-			)
-		)
 	)
-	(global_label "I2C1_SCL"
-		(shape input)
-		(at 144.526 37.592 180)
-		(fields_autoplaced yes)
-		(effects
-			(font
-				(size 1.27 1.27)
-			)
-			(justify right)
-		)
-		(property "Intersheetrefs" "${INTERSHEET_REFS}"
-			(at 132.7718 37.592 0)
-			(effects
-				(font
-					(size 1.27 1.27)
-				)
-				(justify right)
-				(hide yes)
-			)
-		)
-	)
-	(global_label "I2C1_SDA"
-		(shape bidirectional)
-		(at 83.312 32.512 180)
-		(fields_autoplaced yes)
-		(effects
-			(font
-				(size 1.27 1.27)
-			)
-			(justify right)
-		)
-		(property "Intersheetrefs" "${INTERSHEET_REFS}"
-			(at 70.386 32.512 0)
-			(effects
-				(font
-					(size 1.27 1.27)
-				)
-				(justify right)
-				(hide yes)
-			)
-		)
-	)
-	(global_label "I2C1_SCL"
+	(hierarchical_label "I2C1_SCL"
 		(shape input)
 		(at 83.312 35.052 180)
@@
 			(justify right)
 		)
-		(property "Intersheetrefs" "${INTERSHEET_REFS}"
-			(at 71.5578 35.052 0)
-			(effects
-				(font
-					(size 1.27 1.27)
-				)
-				(justify right)
-				(hide yes)
-			)
-		)
 	)

Commit message: [add] comp modifications
Other:
- note added: "I2C @ 0x76 when SDO low *I2C @ 0x77 when SDO high"
- note removed: "I2C @ 0x76 when SDO low I2C @ 0x77 when SDO high"
Changed lines of the file:
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@@
 		)
 	)
-	(text "I2C @ 0x76 when SDO low\nI2C @ 0x77 when SDO high"
+	(text "I2C @ 0x76 when SDO low\n*I2C @ 0x77 when SDO high"
 		(exclude_from_sim no)
 		(at 125.476 54.102 0)
