File: 0-Gen2/1-PCBs/Battery_hot_swap/Battery_hot_swap.kicad_sch (KiCad schematic)
At the start: 16 parts, among them J1 1190297, J2 1190297, J3 1190297, J4 Conn_01x02_Pin, J5 Conn_01x02_Pin, J6 Conn_01x02_Pin, J7 Conn_01x02_Pin

Commit message: management2 updates
Parts:
- added PS1: URB2405YMD-20WR3, Imported_Footprints:CONV_URB2405YMD-20WR3, symbol Imported_Symbols:URB2405YMD-20WR3
- added TP1, TP2: TestPoint, TestPoint:TestPoint_Keystone_5019_Minature, symbol Connector:TestPoint
Connections:
- new net: PS1.5 (TRIM), TP2.1
- new net: PS1.1 (CTRL), TP1.1
- new net 5V_GND: PS1.6 (0V)
- new net GND: PS1.2 (GND)
Other:
- note added: "leave open"
