File: 0-Gen2/1-PCBs/Power_ManagementV2/Power_ManagementV2.kicad_sch (KiCad schematic)
At the start: 16 parts, among them J1 Conn_01x02_Pin, J10 Conn_01x02_Pin, J11 SBH11-PBPC-D10-ST-BK, J12 1986660-2, J13 1986660-2, J2 Conn_01x02_Pin, J6 Conn_01x02_Pin, J9 Conn_01x03_Pin, U7 BA033CC0FP-E2

Commit message: management2 updates
Other:
- removed sheet V_I_sample
Changed lines of the file:
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@@
-	)
-	(sheet
-		(at 109.22 55.88)
-		(size 31.242 21.844)
-		(fields_autoplaced yes)
-		(stroke
-			(width 0.1524)
-			(type solid)
-		)
-		(fill
-			(color 255 229 191 1.0000)
-		)
-		(property "Sheetname" "V_I_sample"
-			(at 109.22 55.1684 0)
-			(effects
-				(font
-					(size 1.27 1.27)
-				)
-				(justify left bottom)
-			)
-		)
-		(property "Sheetfile" "V_I_sample.kicad_sch"
-			(at 109.22 78.3086 0)
-			(effects
-				(font
-					(size 1.27 1.27)
-				)
-				(justify left top)
-			)
-		)
-		(pin "ISENSE_ANALOG" output
-			(at 140.462 75.946 0)
-			(effects
-				(font
-					(size 1.27 1.27)
-				)
-				(justify right)
-			)
-		)
-		(pin "BATT_SAMPLE" output
-			(at 140.462 73.66 0)
-			(effects
-				(font
-					(size 1.27 1.27)
-				)
-				(justify right)
-			)
-		)
-		(pin "-BATT" output
-			(at 109.22 67.564 180)
-			(effects
-				(font
-					(size 1.27 1.27)
-				)
-				(justify left)
-			)
-		)
-		(pin "+BATT_HALL" input
-			(at 109.22 65.532 180)
-			(effects
-				(font
-					(size 1.27 1.27)
-				)
-				(justify left)
-			)
-		)
-		(pin "+Batt" output
-			(at 140.462 66.04 0)
-			(effects
-				(font
-					(size 1.27 1.27)
-				)
-				(justify right)
-			)
-		)
-		(instances
-			(project "Power_ManagementV2"
-				(path "/1c59de6a-87fe-4223-8898-4b0383164a31"
-					(page "4")
-				)
-			)
-		)
 	)
 	(sheet
