File: 0-Gen2/1-PCBs/Power_ManagementV2/BatteryHotSwap.kicad_sch (KiCad schematic)
At the start: 43 parts, among them J3 Conn_01x04_Pin, K1 G5V-1 DC3, Q5 MCTL160N15Y-TP, Q6 MCTL160N15Y-TP, Q7 MCTL160N15Y-TP, U10 74LVC1G08, U11 74LVC1G08, U12 74LVC1G08, U13 74LVC1G08, U15 74AHC1G04, U16 74LVC1G08, U8 LM393DT, U9 LTC1255CS8-PBF

Commit message: progress distribution
Parts:
- added TP2: DiodeRegSupply, TestPoint:TestPoint_Keystone_5019_Minature, symbol Connector:TestPoint
- added U14, U17: STPS5045SG-TR, Imported_Footprints:D2PAK_STM, symbol Imported_Symbols:STPS5045SG-TR
Connections:
- net -BATT2 is gone; now on net -BATT1: R5.2
- net GND is gone; now on net -BATT1: D10.1 (K), D11.1 (K), D12.1 (K), D13.1 (K), D14.1 (K), D15.1 (K), K1.9, U10.3 (GND), U11.3 (GND), U12.3 (GND), U13.3 (GND), U16.3 (GND), U8.4 (VCC-)
- net +BATT1: now also U17.1 (Input), U17.3 (Input)
- net +BATT2: now also U14.1 (Input), U14.3 (Input)
- net +Batt: no longer C12.1, JP12.2 (B), JP14.2 (B), TH3.1, TH4.1, U9.6 (VS)
- net -BATT1: now also C12.2, R18.1, R19.1, U9.3 (GND)
- net -Batt: no longer C12.2, R18.1, R19.1, U9.3 (GND)
- net GATE_DRIVER_EN: no longer U9.4 (IN1), U9.5 (IN2)
- net V_THRUST: no longer D1.2 (A), D9.2 (A)
- net GATE1_DRIVE renamed Gate1Drive
- net GATE2_DRIVE renamed Gate2Drive
- new net +VregDiode: C12.1, JP12.2 (B), JP14.2 (B), TH3.1, TH4.1, U14.2 (Output), U17.2 (Output), U9.6 (VS)
- new net +VregFET: D1.2 (A), D9.2 (A)
- new net Batt1Enable: U9.4 (IN1)
- new net Batt2Enable: U9.5 (IN2)
Other:
- note added: "50A, 0.55Vf Minimal Pw at high current"
- note added: "Always live: 12.0V - 16V diode-regulated supply"
- note added: "Common Ground Reference"
- note added: "Diode Regulated Supply"
- note added: "High-side gate driver. V_g - V_s = 12V Input: 9-24V (12.1 - 16.1V from diode-regulated batt works) V_g Output: 24.1V to 28.1V (+12V relative to V_s)"
- note added: "can use 3.3V enable"
- moved on the sheet: C12, D1, D9, JP12, JP13, JP14, JP15, JP16, K1, R18, R19, TH3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

Commit message: management2 updates
Parts:
- removed R13, R16: 100k, Resistor_SMD:R_0805_2012Metric_Pad1.20x1.40mm_HandSolder, symbol Device:R_US
- removed R6: 500k, Resistor_SMD:R_0805_2012Metric_Pad1.20x1.40mm_HandSolder, symbol Device:R_US
- removed U8: LM393DT, Imported_Footprints:LM393DT, symbol Imported_Symbols:LM393DT
- added C1: 0.1u, Capacitor_SMD:C_0805_2012Metric_Pad1.18x1.45mm_HandSolder, symbol Device:C
- added C100: 100nF, Capacitor_SMD:C_0805_2012Metric_Pad1.18x1.45mm_HandSolder, symbol Device:C
- added C102: 1µF, Capacitor_SMD:C_0805_2012Metric_Pad1.18x1.45mm_HandSolder, symbol Device:C
- added C13, C15, C16, C17: 10uF, Capacitor_SMD:C_0805_2012Metric_Pad1.18x1.45mm_HandSolder, symbol Device:C
- added C14: 1uF, Capacitor_SMD:C_0805_2012Metric_Pad1.18x1.45mm_HandSolder, symbol Device:C
- added J14, J15: Conn_01x08, Connector_PinHeader_2.54mm:PinHeader_1x08_P2.54mm_Vertical, symbol Connector_Generic:Conn_01x08
- added JP19: Jumper_3_Bridged12, Jumper:SolderJumper-3_P1.3mm_Bridged2Bar12_RoundedPad1.0x1.5mm, symbol Jumper:Jumper_3_Bridged12
- added JP20, JP21: Jumper_2_Bridged, Jumper:SolderJumper-2_P1.3mm_Bridged2Bar_RoundedPad1.0x1.5mm, symbol Jumper:Jumper_2_Bridged
- added PM1, PM2: LMS78, Imported_Footprints:LMS78, symbol Connector:Conn_01x03_Pin
- added Q4, Q8, Q9: MCTL160N15Y-TP, Imported_Footprints:TOLL-8L_MCC, symbol Imported_Symbols:MCTL160N15Y-TP
- added R1, R2: 100, Resistor_SMD:R_0805_2012Metric_Pad1.20x1.40mm_HandSolder, symbol Device:R_US
- added R20: 50k, Resistor_SMD:R_0805_2012Metric_Pad1.20x1.40mm_HandSolder, symbol Device:R_US
- added R21, R22, R23: 10k, Resistor_SMD:R_0805_2012Metric_Pad1.20x1.40mm_HandSolder, symbol Device:R_US
- added R3: 2.2k, Resistor_SMD:R_0805_2012Metric_Pad1.20x1.40mm_HandSolder, symbol Device:R_US
- added U1: ACS758LCB-100U-PFF-T, Imported_Footprints:Allegro_MicroSystems,_LLC-CB-5-PFF-0-0-MFG, symbol Imported_Symbols:ACS758ECB-200U-PFF-T
- added U18: BA033CC0FP-E2, Imported_Footprints:TO252-3_ROM, symbol Imported:BA033CC0FP-E2
- added U19, U8: LMV982MM, Imported_Footprints:LMV982MM_NOPB, symbol Imported_Symbols:LMV982MM_NOPB
- added U20: SN74LVC1G373DCKR, Imported_Footprints:SN74LVC, symbol Imported_Symbols:SN74LVC1G373DCKR
- added VR1, VR2: 3296W-1-103RLF, Imported_Footprints:TRIM_3296W-1-103RLF, symbol Imported_Symbols:3296W-1-103RLF
- D13, D15: value LED -> GreenLED; footprint LED_SMD:LED_0805_2012Metric_Pad1.15x1.40mm_HandSolder -> LED_SMD:LED_0603_1608Metric_Pad1.05x0.95mm_HandSolder; MFR Würth Elektronik -> (none); MFR S/N 150080BS75000 -> (none); Supplier 1 https://www.digikey.com/en/products/detail/w%C3%BCrth-elekt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 -> https://www.digikey.com/en/products/detail/rohm-semiconduct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; Supplier 1 S/N 732-4982-1-ND -> 846-SML-D12P8WT86CT-ND
- R17: value 500k -> 10k; MFR Stackpole Electronics Inc -> (none); MFR S/N RNCF0805BTE500K -> (none); Supplier 1 https://www.digikey.com/en/products/detail/stackpole-electr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 -> https://www.digikey.com/en/products/detail/susumu/RR1220P-1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; Supplier 1 S/N 738-RNCF0805BTE500KCT-ND -> RR12P10.0KDCT-ND
- R4: value 100k -> 50k; MFR YAGEO -> (none); MFR S/N RC0805FR-07100KL -> (none); Supplier 1 https://www.digikey.com/en/products/detail/yageo/RC0805FR-0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 -> https://www.digikey.com/en/products/detail/vishay-dale-thin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; Supplier 1 S/N 311-100KCRCT-ND -> 764-1535-1-ND
- R5: value 100k -> 3.9k; MFR YAGEO -> (none); MFR S/N RC0805FR-07100KL -> (none); Supplier 1 https://www.digikey.com/en/products/detail/yageo/RC0805FR-0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 -> https://www.digikey.com/en/products/detail/te-connectivity-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; Supplier 1 S/N 311-100KCRCT-ND -> A126369CT-ND
Connections:
- net +3.3V: now also C13.1, C14.1, JP19.2 (C), JP20.2 (B), U18.3 (OUT), U19.10 (Vcc), U19.5 (SD1), U20.5 (VCC), U8.10 (Vcc), U8.5 (SD1), U8.6 (SD2), VR1.1, VR2.1
- net +BATT1: now also R4.2
- net +BATT2: now also Q4.9 (D), Q8.9 (D), Q9.9 (D), R20.1; no longer R17.1
- net +VregDiode: now also TP2.1, C15.1, C16.1, PM1.1 (Pin_1), PM2.1 (Pin_1)
- net -BATT1: now also C1.1, C100.2, C102.2, C13.2, C14.2, C15.2, C16.2, C17.2, J14.2 (Pin_2), JP21.2 (B), PM1.2 (Pin_2), PM2.2 (Pin_2), R1.2, R2.2, R21.1, R23.1, U1.2 (GND), U18.2 (GND), U19.4 (GND), U19.6 (SD2), U20.2 (GND), U8.4 (GND), VR1.3, VR2.3; no longer D13.1 (K), D15.1 (K)
- net Kill_Switch: no longer D13.2 (A)
- net OCP_COMP: now also U20.3 (D)
- net OCP_LATCH: now also U20.4 (Q)
- net +BATTHall: now reaches Q5.2 (S), Q5.3 (S), Q5.4 (S), Q5.5 (S), Q5.6 (S), Q5.7 (S), Q5.8 (S), Q6.2 (S), Q6.3 (S), Q6.4 (S), Q6.5 (S), Q6.6 (S), Q6.7 (S), Q6.8 (S), Q7.2 (S), Q7.3 (S), Q7.4 (S), Q7.5 (S), Q7.6 (S), Q7.7 (S), Q7.8 (S)
- net +BATTHall: now also Q4.2 (S), Q4.3 (S), Q4.4 (S), Q4.5 (S), Q4.6 (S), Q4.7 (S), Q4.8 (S), Q8.2 (S), Q8.3 (S), Q8.4 (S), Q8.5 (S), Q8.6 (S), Q8.7 (S), Q8.8 (S), Q9.2 (S), Q9.3 (S), Q9.4 (S), Q9.5 (S), Q9.6 (S), Q9.7 (S), Q9.8 (S), U1.4 (IP+)
- net at R4.1: now also R17.1; no longer R17.2
- net Batt1>UVP: now reaches D15.2 (A)
- net Batt1>UVP: now also U8.1 (OUT1)
- net B1_D renamed Batt1Gate
- net BATT1>BATT2: no longer names the net of U13.2
- net BATT2_SAMPLE renamed ISample3.3V
- net ISample3.3V: now also R3.2, U19.3 (IN1+); no longer R4.2
- new net: D15.1 (K), R2.1
- new net: R20.2, R22.2
- new net: D13.1 (K), R1.1
- new net: J14.1 (Pin_1), JP19.1 (A)
- new net +5V: C1.2, C17.1, JP19.3 (B), PM1.3 (Pin_3), PM2.3 (Pin_3), U1.1 (VCC), U18.1 (Vcc)
- new net +BATT: U1.5 (IP-)
- new net AD0: J14.7 (Pin_7)
- new net AD1: J14.8 (Pin_8)
- new net Batt2>UVP: D13.2 (A), U8.9 (OUT2)
- new net Batt2Gate: Q4.1 (G), Q8.1 (G), Q9.1 (G)
- new net COM: J14.6 (Pin_6), JP21.1 (A)
- new net ISample5V: C100.1, C102.1, R3.1, U1.3 (VIOUT)
- new net LE_Teensy: U20.1 (LE)
- new net OCPReference: U19.2 (IN1-), VR2.2
- new net OE_Teensy: U20.6 (*OE)
- new net REF: J14.5 (Pin_5), JP20.1 (A)
- new net SCL: J14.3 (Pin_3)
- new net SDA: J14.4 (Pin_4)
- new net UVPReference: U8.2 (IN1-), U8.8 (IN2-), VR1.2
- new net VIout1Div: J15.8 (Pin_8)
- new net VIout2Div: J15.7 (Pin_7)
- new net VIout3Div: J15.6 (Pin_6)
- new net VIout4Div: J15.5 (Pin_5)
- new net VIout5Div: J15.4 (Pin_4)
- new net VIout6Div: J15.3 (Pin_3)
- new net VIout7Div: J15.2 (Pin_2)
- new net VIout8Div: J15.1 (Pin_1)
- new net VSampleBatt1: R17.2, R21.2, U8.3 (IN1+)
- new net VSampleBatt2: R22.1, R23.2, U8.7 (IN2+)
- new net ~{OCP}: U19.1 (OUT1)
- no-connect marks 0 -> 5
Other:
- note added: "1.82V to 2.4V"
- note added: "3.3V reference -> 12.9mV resolution"
- note added: "3.3V, 1A output"
- note added: "5V --> 3.3V Reg"
- note added: "5V or 3.3V, sets I2C output and Vanalog range"
- note added: "5V regulator"
- note added: "Adafruit ADS7830 Interconnect"
- note added: "Assuming Rdiv = 0.64 40 mV/A at 25C (5V ref) or 25.6mV/A (3.3V ref) 20A = .8V (5V ref) or 0.512V (3.3V ref) 100A = 4V (5V ref) or 2.56V (3.3V ref)"
- note added: "Determines the OCP threshold"
- note added: "Determines the UVP threshold"
- note added: "Hall Effect Current Sensor"
- note added: "High while Batt1>UVP Low when Batt1<UVP or Batt1 disconnected"
- note added: "High while Batt2>UVP Low when Batt2<UVP or Batt2 disconnected"
- note added: "I2C @ 0x48"
- note added: "Latch for OCP"
- note added: "Let R2 = 10k, R1 = 60k, Vdiv = 0.142 Meaning that V_batt,max = 2.4V and V_batt,min = 1.82V P = V^2 / R, with R_eff = 70k = 3.12mW"
- note added: "Make sure to put IP+ and IP- contacts as close to the power trace as possible"
- note added: "TODO: Voltage divide down the drive signal to be within 25? Swap to x150B (max 3.3V output)"
- note added: "Vf=2.2 1.1V/100ohm = 11mA"
- note added: "https://learn.adafruit.com/adafruit-ads7830-8-channel-8-bit-adc/pinouts"
- note added: "input: 9V to 36V. non-isolated output (per supply): 5V, 2A (expect 300mA for Teensy, 1A max for Neopixels) each Oak-D draws more (600mA * 2 = 1.2A). 2x supplies = 4A out this supply won't be able to drive motors"
- note added: "low while nominal high if OCP"
- note added: "other diode option: https://www.digikey.com/en/products/detail/vishay-general-semiconductor-diodes-division/V20PWM63-M3-I/16683192"
- note added: "slap a heat sink on it"
- note added: "start with one, add second if necessary"
- note removed: "If BATT1>BATT2 --> 3.3V If BATT2>BATT1 --> 0V prioritize charging via BATT1 before switching"
- note removed: "Teensy 4.1 Analog Pin Range is 0-3.3V -- 10 bit ADC, 1023 levels Need Vdiv at least = ~0.19 and on the order of kohm Let R2 = 100k, R1 = 600k, Vdiv = 0.142 Meaning that V_batt,max = 2.38V and V_batt,min = 1.91V P = V^2 / R, with R_eff = 700k = 403uW"
- note removed: "Voltage Sampling"
- moved on the sheet: C12, D1, D9, JP12, JP13, JP14, JP15, JP16, K1, Q5, Q6, Q7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

Commit message: hotswap modifications
Parts:
- removed D11, D12, D14: LED, LED_SMD:LED_0805_2012Metric_Pad1.15x1.40mm_HandSolder, symbol Device:LED
- removed J3: Conn_01x04_Pin, Connector_PinHeader_2.54mm:PinHeader_1x04_P2.54mm_Vertical, symbol Connector:Conn_01x04_Pin
- removed JP17: SolderJumper_2_Bridged, Jumper:SolderJumper-2_P1.3mm_Bridged_RoundedPad1.0x1.5mm, symbol Jumper:SolderJumper_2_Bridged
- removed JP18: SolderJumper_3_Bridged12, Jumper:SolderJumper-3_P1.3mm_Bridged2Bar12_RoundedPad1.0x1.5mm, symbol Jumper:SolderJumper_3_Bridged12
- removed U10, U11, U12, U13: 74LVC1G08, Package_TO_SOT_SMD:SOT-353_SC-70-5_Handsoldering, symbol 74xGxx:74LVC1G08
- removed U15: 74AHC1G04, symbol 74xGxx:74AHC1G04
- added D16, D17: GreenLED, LED_SMD:LED_0603_1608Metric_Pad1.05x0.95mm_HandSolder, symbol Device:LED
- added JP22: Jumper_2_Bridged, Jumper:SolderJumper-2_P1.3mm_Bridged2Bar_RoundedPad1.0x1.5mm, symbol Jumper:Jumper_2_Bridged
- added JP23: Jumper_2_Open, Jumper:SolderJumper-2_P1.3mm_Open_RoundedPad1.0x1.5mm, symbol Jumper:Jumper_2_Open
- added R13, R16, R6: 100, Resistor_SMD:R_0805_2012Metric_Pad1.20x1.40mm_HandSolder, symbol Device:R_US
- added S1: 100SP1T1B4M2QE, Imported_Footprints:SW_100SP1T1B4M2QE, symbol Imported_Symbols:100SP1T1B4M2QE
- added U15: 74AHC1G32, Package_TO_SOT_SMD:SOT-23-5, symbol 74xGxx:74AHC1G32
- added U21, U22, U23, U24: 74LVC1G08, Package_TO_SOT_SMD:SOT-353_SC-70-5_Handsoldering, symbol 74xGxx:74LVC1G08
- added U25, U26: 74AHC1G04, symbol 74xGxx:74AHC1G04
- D10: value LED -> GreenLED; footprint LED_SMD:LED_0805_2012Metric_Pad1.15x1.40mm_HandSolder -> LED_SMD:LED_0603_1608Metric_Pad1.05x0.95mm_HandSolder; MFR Würth Elektronik -> (none); MFR S/N 150080BS75000 -> (none); Supplier 1 https://www.digikey.com/en/products/detail/w%C3%BCrth-elekt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 -> https://www.digikey.com/en/products/detail/rohm-semiconduct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; Supplier 1 S/N 732-4982-1-ND -> 846-SML-D12P8WT86CT-ND
Connections:
- net BATT2_EN is gone; now on net ~{SystemKill}: U16.4
- net OCP_COMP is gone; now on net ~{OCP}: U20.3 (D)
- net +3.3V: now also U19.6 (SD2), S1.3, U15.5 (VCC), U21.5 (VCC), U22.5 (VCC), U23.5 (VCC), U24.5 (VCC), U25.5 (VCC)
- net -BATT1: now also JP22.1 (A), R13.2, R16.2, R6.2, S1.1, U15.3 (GND), U21.3 (GND), U22.3 (GND), U23.3 (GND), U24.3 (GND), U25.3 (GND); no longer D10.1 (K), U19.6 (SD2)
- net Batt1>UVP: now also U22.1
- net Batt1Enable: now also U23.4, U26.2
- net Batt2>UVP: now also U24.1
- net VSampleBatt1: now also U19.8 (IN2-)
- net VSampleBatt2: now also U19.7 (IN2+)
- net ~{OCP}: now also D16.2 (A)
- net at U16.1: now also S1.2
- net KillSwitch: now reaches U16.2
- net ~{SystemKill}: now reaches D10.2 (A)
- net ~{SystemKill}: now also U21.2
- net VBatt1>VBatt2: now reaches U19.9 (OUT2)
- net LE_Teensy renamed LETeensy
- net LETeensy: now also JP23.1 (A)
- net OCP_LATCH renamed ~{OCPLatch}
- net ~{OCPLatch}: now also D17.2 (A), JP23.2 (B), U21.1
- net OE_Teensy: no longer names the net of U20.6 (*OE)
- net OE_Teensy: now also JP22.2 (B)
- new net: D17.1 (K), R13.1
- new net: D16.1 (K), R6.1
- new net: U22.4, U23.1
- new net: D10.1 (K), R16.1
- new net VBatt1<VBatt2: U23.2, U25.2
- new net ~{GateDisable}: U21.4, U22.2, U24.2
- no-connect marks 5 -> 2
Other:
- note added: ""If Batt1 is available and system is nominal""
- note added: ""If Batt2 is available and system is nominal""
- note added: ""Turn Batt1 On""
- note added: ""and Batt1 is off""
- note added: ""and Batt1<Batt2""
- note added: ""and Batt2<Batt1""
- note added: "TODO: Voltage divide down the drive signal to be within 25?"
- note added: "Want to prioritize lower voltage battery"
- note added: "from MLU"
- note added: "high when Batt1<Batt2 low when Batt1>Batt2"
- note added: "high while nominal latched low if OCP"
- note added: "high while nominal low if OCP"
- note added: "high while nominal low if killed"
- note added: "high while nominal low if problem"
- note added: "onboard kill switch"
- note removed: "TODO: Voltage divide down the drive signal to be within 25? Swap to x150B (max 3.3V output)"
- note removed: "low while nominal high if OCP"
- moved on the sheet: U20
