File: 0-Gen2/1-PCBs/Power_ManagementV2/BatteryControlLogic.kicad_sch (KiCad schematic)
At the start: 34 parts, among them U19 LMV982MM, U20 74VHC21FT, U21 74AHC1G04, U22 LMV982MM, U23 SN74LVC1G373DCKR, U24 74AHC1G04, U25 74LVC1G08, U26 74LVC1G08

Commit message: cleaned up circuit
Connections:
- net VBatt1>VBatt2 is gone; now on net VBatt1<VBatt2: U22.9 (OUT2)
Changed lines of the file:
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@@
 	(hierarchical_label "~{GateDisable}"
 		(shape input)
-		(at 177.673 58.674 180)
+		(at 177.546 58.674 180)
 		(fields_autoplaced yes)
 		(effects
@@
 		)
 	)
-	(hierarchical_label "VBatt1>VBatt2"
+	(hierarchical_label "VBatt1<VBatt2"
 		(shape output)
 		(at 76.2 147.447 0)

Commit message: almost done with layout
Parts:
- removed D19: GreenLED, LED_SMD:LED_0603_1608Metric_Pad1.05x0.95mm_HandSolder, symbol Device:LED
- removed R30, R31, R32, R34, R35, R36, R37: 100, Resistor_SMD:R_0805_2012Metric_Pad1.20x1.40mm_HandSolder, symbol Device:R_US
- added D12, D13: GreenLED, LED_SMD:LED_0603_1608Metric_Pad1.05x0.95mm_HandSolder, symbol Device:LED
- added R21: 100 Ohm, Imported_Footprints:RES_EXB2HV_1506x8, symbol Imported_Symbols:EXB-2HV222JV
- U8: renamed from U21; footprint (none) -> Package_TO_SOT_SMD:SOT-353_SC-70-5_Handsoldering
- U9: renamed from U24; footprint (none) -> Package_TO_SOT_SMD:SOT-353_SC-70-5_Handsoldering
- renumbered D21 to D10, D20 to D11, D14 to D4, D15 to D5, D16 to D6, D17 to D7, D18 to D8, JP19 to JP21, JP20 to JP22, JP21 to JP23, JP22 to JP24, JP23 to JP25, JP24 to JP26, JP25 to JP27, R33 to R19, S2 to S1, U22 to U10, U23 to U11, U25 to U12, U26 to U13, U19 to U6, U20 to U7, VR3 to VR1, VR4 to VR2
Connections:
- net GND: now also R21.10, R21.11, R21.12, R21.13, R21.14, R21.15, R21.16, R21.9
- net KillSwitch: now also D12.2 (A)
- net at S1.2, U13.1: now also D13.2 (A)
- net RArray6: now reaches D4.1 (K)
- net RArray6: now also R21.6
- net RArray4: now reaches D10.1 (K)
- net RArray4: now also R21.4
- net RArray7: now reaches D6.1 (K)
- net RArray7: now also R21.7
- net RArray3: now reaches D11.1 (K)
- net RArray3: now also R21.3
- net RArray8: now reaches D5.1 (K)
- net RArray8: now also R21.8
- net RArray5: now reaches D8.1 (K)
- net RArray5: now also R21.5
- new net RArray1: D12.1 (K), R21.1
- new net RArray2: D13.1 (K), R21.2

Commit message: ready for fab
Parts:
- R21: footprint Imported_Footprints:RES_EXB2HV_1506x8 -> Imported_Footprints:2506_8x_Resistor_Array; Supplier 1 https://www.digikey.com/en/products/detail/panasonic-electr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 -> https://www.digikey.com/en/products/detail/cts-resistor-pro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; Supplier 1 S/N Y1101CT-ND -> 60-742C163101JPCT-ND
Changed lines of the file:
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@@
 			)
 		)
-		(property "Footprint" "Imported_Footprints:RES_EXB2HV_1506x8"
+		(property "Footprint" "Imported_Footprints:2506_8x_Resistor_Array"
 			(at 261.112 112.014 0)
 			(effects
@@
 			)
 		)
-		(property "Datasheet" "EXB-2HV222JV"
+		(property "Datasheet" ""
 			(at 261.112 112.014 0)
 			(effects
@@
 			)
 		)
-		(property "Supplier 1" "https://www.digikey.com/en/products/detail/panasonic-electronic-components/EXB-2HV101JV/285307"
+		(property "Supplier 1" "https://www.digikey.com/en/products/detail/cts-resistor-products/742C163101JP/1124353"
 			(at 261.112 112.014 0)
 			(effects
@@
 			)
 		)
-		(property "Supplier 1 S/N" "Y1101CT-ND"
+		(property "Supplier 1 S/N" "60-742C163101JPCT-ND"
 			(at 261.112 112.014 0)
 			(effects

Commit message: some updates
Parts:
- removed U10, U6: LMV982MM, Imported_Footprints:LMV982MM_NOPB, symbol Imported_Symbols:LMV982MM_NOPB
- added U15: TSX634AIPT, Imported_Footprints:TSSOP14_STM, symbol Imported_Symbols:TSX634AIPT
Connections:
- net +3.3V: now also U15.4 (VCC+)
- net Batt1>UVP: now also U15.1 (OUT1)
- net Batt2>UVP: now also U15.7 (OUT2)
- net GND: now also U15.11 (VCC-)
- net ISample3.3V: now also U15.10 (IN3+)
- net OCPReference: now also U15.9 (IN3-)
- net UVPReference: now also U15.2 (IN1-), U15.6 (IN2-)
- net VBatt1<VBatt2: now also U15.14 (OUT4)
- net VSampleBatt1: now also U15.13 (IN4-), U15.3 (IN1+)
- net VSampleBatt2: now also U15.12 (IN4+), U15.5 (IN2+)
- net ~{OCP}: now also U15.8 (OUT3)
Other:
- moved on the sheet: VR1
