File: 0-Gen2/1-PCBs/Power_ManagementV2/Power_ManagementV2.kicad_pcb (KiCad board)
At the start: 2 copper layers, 70 x 94 mm, 59 parts, among them J1 Conn_01x02_Pin, J10 Conn_01x02_Pin, J2 Conn_01x02_Pin, J3 1986660-2, J4 1986660-2, J5 Conn_01x02_Pin, J6 Conn_01x02_Pin, J7 Conn_01x02_Pin, J8 Conn_01x04_Pin, J9 Conn_01x03_Pin, K2 G5V-1 DC3, Q1 MCTL160N15Y-TP, Q2 MCTL160N15Y-TP, Q3 MCTL160N15Y-TP, U1 ACS758ECB-200U-PFF-T, U2 LM393DT, U3 SN74LVC1G373DCKR, U4 74LVC1G08, U5 74LVC1G08, U6 LTC1255CS8-PBF

Commit message: almost ready to fab
Parts:
- removed C1: 0.1u, Capacitor_SMD:C_0805_2012Metric_Pad1.18x1.45mm_HandSolder
- removed C2: 10uF, Imported_Footprints:CAP_EEE-1CA100SR_PAN
- removed C6: 10uF, Capacitor_SMD:C_0805_2012Metric_Pad1.18x1.45mm_HandSolder
- removed C7, C8, C9: 1u, Imported_Footprints:U2-D_NCH
- removed CR1: SBRT15U50SP5-13, Imported_Footprints:POWERDI5_DIO
- removed D2, D3, D4, D5, D7: LED, LED_SMD:LED_0805_2012Metric_Pad1.15x1.40mm_HandSolder
- removed D6, D8: D_Zener, Imported_Footprints:1N5242B
- removed H1, H3, H4: MountingHole, MountingHole:MountingHole_3.2mm_M3
- removed J1, J10, J2, J5, J6, J7: Conn_01x02_Pin, Connector_PinHeader_2.54mm:PinHeader_1x02_P2.54mm_Vertical
- removed J3, J4: 1986660-2, Imported_Footprints:CONN2_1986660-2_TEC
- removed J8: Conn_01x04_Pin, Connector_PinHeader_2.54mm:PinHeader_1x04_P2.54mm_Vertical
- removed J9: Conn_01x03_Pin, Connector_PinHeader_2.54mm:PinHeader_1x03_P2.54mm_Vertical
- removed JP1, JP4, JP7, JP9: SolderJumper_3_Bridged12, Jumper:SolderJumper-3_P1.3mm_Bridged2Bar12_RoundedPad1.0x1.5mm
- removed JP2, JP3: SolderJumper_2_Open, Jumper:SolderJumper-2_P1.3mm_Open_RoundedPad1.0x1.5mm
- removed JP5, JP6, JP8: SolderJumper_2_Bridged, Jumper:SolderJumper-2_P1.3mm_Bridged_RoundedPad1.0x1.5mm
- removed K2: G5V-1 DC3, Imported_Footprints:RELAY_G5V-1_OMR
- removed Q1, Q2, Q3: MCTL160N15Y-TP, Imported_Footprints:TOLL-8L_MCC
- removed R10: 200k, Resistor_SMD:R_0805_2012Metric_Pad1.20x1.40mm_HandSolder
- removed R11, R12, R8, R9: ~, Resistor_SMD:R_0805_2012Metric_Pad1.20x1.40mm_HandSolder
- removed R13: 500k, Resistor_SMD:R_0805_2012Metric_Pad1.20x1.40mm_HandSolder
- removed R14, R15: 100k, Resistor_SMD:R_0805_2012Metric
- removed R5, R6: 100k, Resistor_SMD:R_0805_2012Metric_Pad1.20x1.40mm_HandSolder
- removed R7: 150k, Resistor_SMD:R_0805_2012Metric_Pad1.20x1.40mm_HandSolder
- removed TH1, TH2: Thermistor_US, Resistor_SMD:R_0805_2012Metric
- removed U1: ACS758ECB-200U-PFF-T, Imported_Footprints:Allegro_MicroSystems,_LLC-CB-5-PFF-0-0-MFG
- removed U2: LM393DT, Imported_Footprints:LM393DT
- removed U3: SN74LVC1G373DCKR, Imported_Footprints:SN74LVC
- removed U4, U5: 74LVC1G08, Package_TO_SOT_SMD:SOT-353_SC-70-5_Handsoldering
- removed U6: LTC1255CS8-PBF, Imported_Footprints:LTC1255
Routing:
- net /Battery_input/-Batt: track 238.5 -> 0.00 mm, vias 9 -> 0
- net GND: track 214.0 -> 0.00 mm, vias 7 -> 0
- net /FETs/V_THRUST: track 203.8 -> 0.00 mm, vias 2 -> 0
- net /FETs/+Batt: track 133.8 -> 0.00 mm, vias 2 -> 0
- net +3.3V: track 98.5 -> 0.00 mm, vias 6 -> 0
- net /FET_control_logic/Kill_Switch: track 65.7 -> 0.00 mm, vias 11 -> 0
- net Net-(J8-Pin_4): track 64.1 -> 0.00 mm, vias 9 -> 0
- net /FET_control_logic/OCP_LATCH: track 63.2 -> 0.00 mm, vias 2 -> 0
- net /FETs/GATE2_DRIVE: track 63.1 -> 0.00 mm, vias 4 -> 0
- net /FETs/GATE1_DRIVE: track 63.0 -> 0.00 mm, vias 5 -> 0
- net /FET_control_logic/OCP_COMP: track 61.4 -> 0.00 mm, vias 4 -> 0
- net /FET_control_logic/UVP_COMP: track 61.4 -> 0.00 mm, vias 11 -> 0
- net /FET_control_logic/3.3V_GATE_EN: track 58.5 -> 0.00 mm, vias 9 -> 0
- net VREF2: track 54.9 -> 0.00 mm, vias 6 -> 0
- net VREF1: track 50.7 -> 0.00 mm, vias 8 -> 0
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- removed copper zone on F.Cu, net /Battery_input/+BATT_HALL
- removed copper zone on F.Cu, net /FETs/+Batt
Other:
- board outline removed
- board text removed: "3.3V"
- board text removed: "BATT_S"
- board text removed: "GATE_EN"
- board text removed: "Kill"
- board text removed: "Kill In"
- board text removed: "LE"
- board text removed: "OE"
- board text removed: "UVP"
- board text removed: "VREF1/2"

Commit message: almost done with layout
Parts:
- added C1: 10uF, Imported_Footprints:CAP_EEE-1CA100SR_PAN, F.Cu at (240.5, 67.3)
- added C10: 10,000uF, Capacitor_THT:CP_Radial_D16.0mm_P7.50mm, F.Cu at (180.1, 140.6)
- added C11: 10,000uF, Capacitor_THT:CP_Radial_D16.0mm_P7.50mm, F.Cu at (163.0, 140.6)
- added C2: 10uF, Capacitor_SMD:C_0805_2012Metric_Pad1.18x1.45mm_HandSolder, F.Cu at (127.0, 91.6)
- added C3: 10uF, Capacitor_SMD:C_0805_2012Metric_Pad1.18x1.45mm_HandSolder, F.Cu at (127.0, 94.6)
- added C4: 10uF, Capacitor_SMD:C_0805_2012Metric_Pad1.18x1.45mm_HandSolder, F.Cu at (262.5, 138.1)
- added C5: 10uF, Capacitor_SMD:C_0805_2012Metric_Pad1.18x1.45mm_HandSolder, F.Cu at (257.8, 138.2)
- added C6: 1uF, Capacitor_SMD:C_0805_2012Metric_Pad1.18x1.45mm_HandSolder, F.Cu at (260.1, 138.2)
- added C7: 0.1u, Capacitor_SMD:C_0805_2012Metric_Pad1.18x1.45mm_HandSolder, F.Cu at (127.0, 97.6)
- added C8: 100nF, Capacitor_SMD:C_0805_2012Metric_Pad1.18x1.45mm_HandSolder, F.Cu at (187.6, 126.6)
- added C9: 1µF, Capacitor_SMD:C_0805_2012Metric_Pad1.18x1.45mm_HandSolder, F.Cu at (190.0, 126.6)
- added CR1: SBRT15U50SP5-13, Imported_Footprints:POWERDI5_DIO, F.Cu at (125.5, 114.2)
- added D1: D_Zener, Imported_Footprints:1N5242B, F.Cu at (245.6, 73.9)
- added D10: GreenLED, LED_SMD:LED_0603_1608Metric_Pad1.05x0.95mm_HandSolder, F.Cu at (252.6, 146.6)
- added D11: GreenLED, LED_SMD:LED_0603_1608Metric_Pad1.05x0.95mm_HandSolder, F.Cu at (252.6, 148.3)
- added D12: GreenLED, LED_SMD:LED_0603_1608Metric_Pad1.05x0.95mm_HandSolder, F.Cu at (252.6, 151.8)
- added D13: GreenLED, LED_SMD:LED_0603_1608Metric_Pad1.05x0.95mm_HandSolder, F.Cu at (252.6, 150.0)
- added D2: D_Zener, Imported_Footprints:1N5242B, F.Cu at (245.7, 60.5)
- added D3: TVS, Diode_SMD:D_SMA, F.Cu at (175.9, 113.4)
- added D4: GreenLED, LED_SMD:LED_0603_1608Metric_Pad1.05x0.95mm_HandSolder, F.Cu at (252.7, 143.2)
- added D5: GreenLED, LED_SMD:LED_0603_1608Metric_Pad1.05x0.95mm_HandSolder, F.Cu at (252.7, 139.8)
- added D6: GreenLED, LED_SMD:LED_0603_1608Metric_Pad1.05x0.95mm_HandSolder, F.Cu at (252.7, 141.5)
- added D7: GreenLED, LED_SMD:LED_0603_1608Metric_Pad1.05x0.95mm_HandSolder, F.Cu at (252.7, 138.2)
- added D8: GreenLED, LED_SMD:LED_0603_1608Metric_Pad1.05x0.95mm_HandSolder, F.Cu at (252.7, 144.9)
- added H1: MountingHole, MountingHole:MountingHole_3.2mm_M3, F.Cu at (189.7, 72.8)
- added H2: MountingHole, MountingHole:MountingHole_3.2mm_M3, F.Cu at (189.7, 136.8)
- added H3: MountingHole, MountingHole:MountingHole_3.2mm_M3, F.Cu at (237.7, 136.8)
- added H4: MountingHole, MountingHole:MountingHole_3.2mm_M3, F.Cu at (237.7, 72.8)
- added J1: Conn_01x02_Pin, Connector_AMASS:AMASS_XT60-M_1x02_P7.20mm_Vertical, F.Cu at (257.4, 93.5)
- added J2: Conn_01x02_Pin, Connector_AMASS:AMASS_XT60-M_1x02_P7.20mm_Vertical, F.Cu at (257.3, 105.6)
- added J3: Conn_01x08, Connector_PinHeader_2.54mm:PinHeader_1x08_P2.54mm_Vertical, F.Cu at (194.1, 78.5)
- added J4: Conn_01x08, Connector_PinHeader_2.54mm:PinHeader_1x08_P2.54mm_Vertical, F.Cu at (194.1, 91.2)
- added J5: Conn_01x02_Pin, Connector_AMASS:AMASS_XT60PW-F_1x02_P7.20mm_Horizontal, F.Cu at (162.1, 102.6)
- added J6: Conn_01x02_Pin, Connector_AMASS:AMASS_XT30PW-F_1x02_P2.50mm_Horizontal, F.Cu at (162.8, 128.7)
- added J7: USB_A_Stacked, Connector_USB:USB_A_Wuerth_61400826021_Horizontal_Stacked, F.Cu at (170.4, 67.5)
- added J8: SBH11-PBPC-D10-ST-BK, Imported_Footprints:SULLINS_SBH11-PBPC-D10-ST-BK, F.Cu at (170.9, 56.0)
- added JP1: SolderJumper_2_Bridged, Jumper:SolderJumper-2_P1.3mm_Bridged2Bar_RoundedPad1.0x1.5mm, F.Cu at (262.3, 68.3)
- added JP10: Jumper_2_Bridged, Jumper:SolderJumper-2_P1.3mm_Bridged2Bar_RoundedPad1.0x1.5mm, F.Cu at (177.2, 86.8)
- added JP11: Jumper_2_Bridged, Jumper:SolderJumper-2_P1.3mm_Bridged2Bar_RoundedPad1.0x1.5mm, F.Cu at (177.2, 82.8)
- added JP12: Jumper_2_Open, Imported_Footprints:KEYSTONE_5102, F.Cu at (168.7, 127.8)
- added JP13: Jumper_2_Bridged, Jumper:SolderJumper-2_P1.3mm_Bridged2Bar_RoundedPad1.0x1.5mm, F.Cu at (175.6, 63.1)
- added JP14: Jumper_2_Bridged, Jumper:SolderJumper-2_P1.3mm_Bridged2Bar_RoundedPad1.0x1.5mm, F.Cu at (187.4, 131.5)
- added JP15: Jumper_2_Bridged, Jumper:SolderJumper-2_P1.3mm_Bridged2Bar_RoundedPad1.0x1.5mm, F.Cu at (184.3, 87.0)
- added JP16: Jumper_2_Bridged, Jumper:SolderJumper-2_P1.3mm_Bridged2Bar_RoundedPad1.0x1.5mm, F.Cu at (188.1, 87.0)
- added JP17: Jumper_2_Bridged, Jumper:SolderJumper-2_P1.3mm_Bridged2Bar_RoundedPad1.0x1.5mm, F.Cu at (119.3, 91.9)
- added JP18: Jumper_2_Bridged, Jumper:SolderJumper-2_P1.3mm_Bridged2Bar_RoundedPad1.0x1.5mm, F.Cu at (167.8, 80.8)
- added JP19: Jumper_2_Bridged, Jumper:SolderJumper-2_P1.3mm_Bridged2Bar_RoundedPad1.0x1.5mm, F.Cu at (119.3, 99.0)
- added JP2: SolderJumper_2_Open, Jumper:SolderJumper-2_P1.3mm_Open_RoundedPad1.0x1.5mm, F.Cu at (247.0, 69.6)
- added JP20: Jumper_2_Bridged, Jumper:SolderJumper-2_P1.3mm_Bridged2Bar_RoundedPad1.0x1.5mm, F.Cu at (119.3, 102.5)
- added JP21: Jumper_2_Open, Jumper:SolderJumper-2_P1.3mm_Open_RoundedPad1.0x1.5mm, F.Cu at (198.6, 151.7)
- added JP22: Jumper_2_Bridged, Jumper:SolderJumper-2_P1.3mm_Bridged2Bar_RoundedPad1.0x1.5mm, F.Cu at (202.0, 151.7)
- added JP23: Jumper_2_Open, Jumper:SolderJumper-2_P1.3mm_Open_RoundedPad1.0x1.5mm, F.Cu at (210.9, 151.7)
- added JP24: Jumper_2_Bridged, Jumper:SolderJumper-2_P1.3mm_Bridged2Bar_RoundedPad1.0x1.5mm, F.Cu at (207.5, 151.7)
- added JP25: Jumper_2_Bridged, Jumper:SolderJumper-2_P1.3mm_Bridged2Bar_RoundedPad1.0x1.5mm, F.Cu at (204.6, 132.0)
- added JP26: Jumper_2_Open, Jumper:SolderJumper-2_P1.3mm_Open_RoundedPad1.0x1.5mm, F.Cu at (201.4, 133.6)
- added JP27: Jumper_2_Bridged, Jumper:SolderJumper-2_P1.3mm_Bridged2Bar_RoundedPad1.0x1.5mm, F.Cu at (212.3, 138.2)
- added JP3: SolderJumper_2_Bridged, Jumper:SolderJumper-2_P1.3mm_Bridged2Bar_RoundedPad1.0x1.5mm, F.Cu at (247.0, 65.7)
- added JP4: Jumper_2_Open, Jumper:SolderJumper-2_P1.3mm_Open_RoundedPad1.0x1.5mm, F.Cu at (262.6, 60.8)
- added JP5: Jumper_2_Open, Jumper:SolderJumper-2_P1.3mm_Open_RoundedPad1.0x1.5mm, F.Cu at (263.1, 75.5)
- added JP6: Jumper_2_Bridged, Jumper:SolderJumper-2_P1.3mm_Bridged_RoundedPad1.0x1.5mm, F.Cu at (262.6, 64.2)
- added JP7: Jumper_2_Bridged, Jumper:SolderJumper-2_P1.3mm_Bridged_RoundedPad1.0x1.5mm, F.Cu at (263.1, 79.0)
- added JP8: Jumper_3_Bridged12, Jumper:SolderJumper-3_P1.3mm_Bridged2Bar12_RoundedPad1.0x1.5mm, F.Cu at (171.9, 90.4)
- added JP9: Jumper_3_Bridged12, Jumper:SolderJumper-3_P1.3mm_Bridged2Bar12_RoundedPad1.0x1.5mm, F.Cu at (192.9, 84.2)
- added LED1: 1655, LED_SMD:LED_LiteOn_LTST-E563C_PLCC4_5.0x5.0mm_P3.2mm_HandSoldering, F.Cu at (157.4, 157.2)
- added LED10: 1655, LED_SMD:LED_LiteOn_LTST-E563C_PLCC4_5.0x5.0mm_P3.2mm_HandSoldering, F.Cu at (216.0, 157.2)
- added LED11: 1655, LED_SMD:LED_LiteOn_LTST-E563C_PLCC4_5.0x5.0mm_P3.2mm_HandSoldering, F.Cu at (222.5, 157.2)
- added LED12: 1655, LED_SMD:LED_LiteOn_LTST-E563C_PLCC4_5.0x5.0mm_P3.2mm_HandSoldering, F.Cu at (229.0, 157.2)
- added LED13: 1655, LED_SMD:LED_LiteOn_LTST-E563C_PLCC4_5.0x5.0mm_P3.2mm_HandSoldering, F.Cu at (235.5, 157.2)
- added LED14: 1655, LED_SMD:LED_LiteOn_LTST-E563C_PLCC4_5.0x5.0mm_P3.2mm_HandSoldering, F.Cu at (242.0, 157.2)
- added LED15: 1655, LED_SMD:LED_LiteOn_LTST-E563C_PLCC4_5.0x5.0mm_P3.2mm_HandSoldering, F.Cu at (248.5, 157.2)
- added LED16: 1655, LED_SMD:LED_LiteOn_LTST-E563C_PLCC4_5.0x5.0mm_P3.2mm_HandSoldering, F.Cu at (255.0, 157.2)
- added LED17: 1655, LED_SMD:LED_LiteOn_LTST-E563C_PLCC4_5.0x5.0mm_P3.2mm_HandSoldering, F.Cu at (261.5, 157.2)
- added LED18: 1655, LED_SMD:LED_LiteOn_LTST-E563C_PLCC4_5.0x5.0mm_P3.2mm_HandSoldering, F.Cu at (261.5, 54.7)
- added LED19: 1655, LED_SMD:LED_LiteOn_LTST-E563C_PLCC4_5.0x5.0mm_P3.2mm_HandSoldering, F.Cu at (255.1, 54.7)
- added LED2: 1655, LED_SMD:LED_LiteOn_LTST-E563C_PLCC4_5.0x5.0mm_P3.2mm_HandSoldering, F.Cu at (163.9, 157.2)
- added LED20: 1655, LED_SMD:LED_LiteOn_LTST-E563C_PLCC4_5.0x5.0mm_P3.2mm_HandSoldering, F.Cu at (248.6, 54.7)
- added LED21: 1655, LED_SMD:LED_LiteOn_LTST-E563C_PLCC4_5.0x5.0mm_P3.2mm_HandSoldering, F.Cu at (242.2, 54.7)
- added LED22: 1655, LED_SMD:LED_LiteOn_LTST-E563C_PLCC4_5.0x5.0mm_P3.2mm_HandSoldering, F.Cu at (235.8, 54.7)
- added LED23: 1655, LED_SMD:LED_LiteOn_LTST-E563C_PLCC4_5.0x5.0mm_P3.2mm_HandSoldering, F.Cu at (229.4, 54.7)
- added LED24: 1655, LED_SMD:LED_LiteOn_LTST-E563C_PLCC4_5.0x5.0mm_P3.2mm_HandSoldering, F.Cu at (223.0, 54.7)
- added LED25: 1655, LED_SMD:LED_LiteOn_LTST-E563C_PLCC4_5.0x5.0mm_P3.2mm_HandSoldering, F.Cu at (216.5, 54.7)
- added LED26: 1655, LED_SMD:LED_LiteOn_LTST-E563C_PLCC4_5.0x5.0mm_P3.2mm_HandSoldering, F.Cu at (210.1, 54.7)
- added LED27: 1655, LED_SMD:LED_LiteOn_LTST-E563C_PLCC4_5.0x5.0mm_P3.2mm_HandSoldering, F.Cu at (203.7, 54.7)
- added LED28: 1655, LED_SMD:LED_LiteOn_LTST-E563C_PLCC4_5.0x5.0mm_P3.2mm_HandSoldering, F.Cu at (197.3, 54.7)
- added LED29: 1655, LED_SMD:LED_LiteOn_LTST-E563C_PLCC4_5.0x5.0mm_P3.2mm_HandSoldering, F.Cu at (190.9, 54.7)
- added LED3: 1655, LED_SMD:LED_LiteOn_LTST-E563C_PLCC4_5.0x5.0mm_P3.2mm_HandSoldering, F.Cu at (170.4, 157.2)
- added LED30: 1655, LED_SMD:LED_LiteOn_LTST-E563C_PLCC4_5.0x5.0mm_P3.2mm_HandSoldering, F.Cu at (153.6, 22.6)
- added LED31: 1655, LED_SMD:LED_LiteOn_LTST-E563C_PLCC4_5.0x5.0mm_P3.2mm_HandSoldering, F.Cu at (147.4, 22.7)
- added LED32: 1655, LED_SMD:LED_LiteOn_LTST-E563C_PLCC4_5.0x5.0mm_P3.2mm_HandSoldering, F.Cu at (141.3, 22.7)
- added LED33: 1655, LED_SMD:LED_LiteOn_LTST-E563C_PLCC4_5.0x5.0mm_P3.2mm_HandSoldering, F.Cu at (134.8, 22.7)
- added LED34: 1655, LED_SMD:LED_LiteOn_LTST-E563C_PLCC4_5.0x5.0mm_P3.2mm_HandSoldering, F.Cu at (128.2, 22.7)
- added LED35: 1655, LED_SMD:LED_LiteOn_LTST-E563C_PLCC4_5.0x5.0mm_P3.2mm_HandSoldering, F.Cu at (122.1, 22.6)
- added LED36: 1655, LED_SMD:LED_LiteOn_LTST-E563C_PLCC4_5.0x5.0mm_P3.2mm_HandSoldering, F.Cu at (115.6, 22.6)
- added LED4: 1655, LED_SMD:LED_LiteOn_LTST-E563C_PLCC4_5.0x5.0mm_P3.2mm_HandSoldering, F.Cu at (176.9, 157.2)
- added LED5: 1655, LED_SMD:LED_LiteOn_LTST-E563C_PLCC4_5.0x5.0mm_P3.2mm_HandSoldering, F.Cu at (183.4, 157.2)
- added LED6: 1655, LED_SMD:LED_LiteOn_LTST-E563C_PLCC4_5.0x5.0mm_P3.2mm_HandSoldering, F.Cu at (189.9, 157.2)
- added LED7: 1655, LED_SMD:LED_LiteOn_LTST-E563C_PLCC4_5.0x5.0mm_P3.2mm_HandSoldering, F.Cu at (196.5, 157.2)
- added LED8: 1655, LED_SMD:LED_LiteOn_LTST-E563C_PLCC4_5.0x5.0mm_P3.2mm_HandSoldering, F.Cu at (203.0, 157.2)
- added LED9: 1655, LED_SMD:LED_LiteOn_LTST-E563C_PLCC4_5.0x5.0mm_P3.2mm_HandSoldering, F.Cu at (209.5, 157.2)
- added PM1: LMS78, Imported_Footprints:LMS78, F.Cu at (237.5, 132.1)
- added PM2: LMS78, Imported_Footprints:LMS78, F.Cu at (250.9, 132.0)
- added Q1: MCTL160N15Y-TP, Imported_Footprints:TOLL-8L_MCC, F.Cu at (227.7, 70.2)
- added Q2: MCTL160N15Y-TP, Imported_Footprints:TOLL-8L_MCC, F.Cu at (222.8, 81.3)
- added Q3: MCTL160N15Y-TP, Imported_Footprints:TOLL-8L_MCC, F.Cu at (228.1, 92.7)
- added Q4: MCTL160N15Y-TP, Imported_Footprints:TOLL-8L_MCC, F.Cu at (228.1, 106.7)
- added Q5: MCTL160N15Y-TP, Imported_Footprints:TOLL-8L_MCC, F.Cu at (222.8, 118.3)
- added Q6: MCTL160N15Y-TP, Imported_Footprints:TOLL-8L_MCC, F.Cu at (228.1, 130.1)
- added R1: 50k, Resistor_SMD:R_0805_2012Metric_Pad1.20x1.40mm_HandSolder, F.Cu at (110.8, 109.3)
- added R10: 12k, Resistor_SMD:R_0805_2012Metric_Pad1.20x1.40mm_HandSolder, F.Cu at (258.0, 75.8)
- added R11: 86.6k, Resistor_SMD:R_0805_2012Metric_Pad1.20x1.40mm_HandSolder, F.Cu at (258.9, 63.4)
- added R12: 86.6k, Resistor_SMD:R_0805_2012Metric_Pad1.20x1.40mm_HandSolder, F.Cu at (259.0, 78.8)
- added R13: 2.2k, Resistor_SMD:R_0805_2012Metric_Pad1.20x1.40mm_HandSolder, F.Cu at (192.3, 126.6)
- added R14: 0.5 Ohm 25W, Imported_Footprints:TO508P1229X317-3N, F.Cu at (178.1, 127.8)
- added R15: 3.9k, Resistor_SMD:R_0805_2012Metric_Pad1.20x1.40mm_HandSolder, F.Cu at (192.3, 130.6)
- added R16: 10k, Resistor_SMD:R_0805_2012Metric_Pad1.20x1.40mm_HandSolder, F.Cu at (214.4, 101.1)
- added R19: 100, Resistor_SMD:R_0805_2012Metric_Pad1.20x1.40mm_HandSolder, F.Cu at (241.4, 143.5)
- added R2: 10k, Resistor_SMD:R_0805_2012Metric_Pad1.20x1.40mm_HandSolder, F.Cu at (110.8, 112.3)
- added R21: 100 Ohm, Imported_Footprints:RES_EXB2HV_1506x8, F.Cu at (241.2, 148.0)
- added R3: 10k, Resistor_SMD:R_0805_2012Metric_Pad1.20x1.40mm_HandSolder, F.Cu at (110.8, 115.2)
- added R4: 100k, Resistor_SMD:R_0805_2012Metric, F.Cu at (250.4, 69.5)
- added R5: 100k, Resistor_SMD:R_0805_2012Metric, F.Cu at (250.4, 67.0)
- added R6: 50k, Resistor_SMD:R_0805_2012Metric_Pad1.20x1.40mm_HandSolder, F.Cu at (110.8, 118.2)
- added R7: 10k, Resistor_SMD:R_0805_2012Metric_Pad1.20x1.40mm_HandSolder, F.Cu at (115.6, 109.3)
- added R8: 10k, Resistor_SMD:R_0805_2012Metric_Pad1.20x1.40mm_HandSolder, F.Cu at (115.6, 112.3)
- added R9: 12k, Resistor_SMD:R_0805_2012Metric_Pad1.20x1.40mm_HandSolder, F.Cu at (257.9, 60.5)
- added S1: 100SP1T1B4M2QE, Imported_Footprints:SW_100SP1T1B4M2QE, F.Cu at (234.1, 145.9)
- added TH1: Thermistor_US, Resistor_SMD:R_0805_2012Metric, F.Cu at (259.5, 68.3)
- added TH2: Thermistor_US, Resistor_SMD:R_0805_2012Metric, F.Cu at (254.5, 63.1)
- added TP1: DiodeRegSupply, TestPoint:TestPoint_Keystone_5019_Minature, F.Cu at (244.7, 99.5)
- added TP2: TestPoint, TestPoint:TestPoint_Pad_1.0x1.0mm, F.Cu at (123.0, 91.6)
- added TP3: TestPoint, TestPoint:TestPoint_Pad_1.0x1.0mm, F.Cu at (123.0, 94.7)
- added TP4: TestPoint, TestPoint:TestPoint_Pad_1.0x1.0mm, F.Cu at (123.0, 97.7)
- added TP5: TestPoint, TestPoint:TestPoint_Pad_1.0x1.0mm, F.Cu at (123.0, 100.8)
- added TP6: TestPoint, TestPoint:TestPoint_Pad_1.0x1.0mm, F.Cu at (123.0, 103.8)
- added U1: STPS5045SG-TR, Imported_Footprints:D2PAK_STM, F.Cu at (244.7, 90.2)
- added U10: LMV982MM, Imported_Footprints:LMV982MM_NOPB, F.Cu at (197.3, 129.3)
- added U11: SN74LVC1G373DCKR, Imported_Footprints:SN74LVC, F.Cu at (201.2, 130.0)
- added U12: 74LVC1G08, Package_TO_SOT_SMD:SOT-353_SC-70-5_Handsoldering, F.Cu at (208.3, 135.3)
- added U13: 74LVC1G08, Package_TO_SOT_SMD:SOT-353_SC-70-5_Handsoldering, F.Cu at (208.3, 138.4)
- added U14: MCP9808_MSOP, Package_SO:MSOP-8_3x3mm_P0.65mm, F.Cu at (209.7, 101.1)
- added U2: STPS5045SG-TR, Imported_Footprints:D2PAK_STM, F.Cu at (244.6, 109.2)
- added U3: LTC1255CS8-PBF, Imported_Footprints:LTC1255, F.Cu at (255.2, 68.3)
- added U4: BA033CC0FP-E2, Imported_Footprints:TO252-3_ROM, F.Cu at (260.1, 149.3)
- added U5: ACS758LCB-100U-PFF-T, Imported_Footprints:Allegro_MicroSystems,_LLC-CB-5-PFF-0-0-MFG, F.Cu at (188.7, 112.5)
- added U6: LMV982MM, Imported_Footprints:LMV982MM_NOPB, F.Cu at (200.6, 137.3)
- added U7: 74VHC21FT, Imported_Footprints:TSSOP14B, F.Cu at (201.1, 147.6)
- added U8: 74AHC1G04, Package_TO_SOT_SMD:SOT-353_SC-70-5_Handsoldering, F.Cu at (199.8, 140.8)
- added U9: 74AHC1G04, Package_TO_SOT_SMD:SOT-353_SC-70-5_Handsoldering, F.Cu at (204.7, 142.8)
- added VR1: 3296W-1-103RLF, Imported_Footprints:TRIM_3296W-1-103RLF, F.Cu at (223.2, 143.8)
- added VR2: 3296W-1-103RLF, Imported_Footprints:TRIM_3296W-1-103RLF, F.Cu at (223.2, 149.6)
Routing:
- net +5V: track 0.00 -> 570.6 mm, vias 0 -> 1
- net +BATTHall: track 0.00 -> 304.7 mm
- net +3.3V: track 0.00 -> 258.4 mm, vias 0 -> 14
- net /Battery Control Logic/~{GateDisable}: track 0.00 -> 186.5 mm, vias 0 -> 21
- net +BATT: track 0.00 -> 173.9 mm, vias 0 -> 5
- net KillSwitch: track 0.00 -> 164.5 mm, vias 0 -> 12
- net Analog_Current: track 0.00 -> 110.1 mm, vias 0 -> 2
- net +VregDiode: track 0.00 -> 104.2 mm, vias 0 -> 2
- net Batt2Gate: track 0.00 -> 102.4 mm, vias 0 -> 4
- net /Battery Control Logic/~{OCP}: track 0.00 -> 101.7 mm, vias 0 -> 6
- net /Battery Control Logic/OCPReference: track 0.00 -> 99.7 mm, vias 0 -> 3
- net ISample3.3V: track 0.00 -> 93.3 mm, vias 0 -> 8
- net /Battery Control Logic/Batt1>UVP: track 0.00 -> 91.5 mm, vias 0 -> 8
- net /Battery Control Logic/UVPReference: track 0.00 -> 89.3 mm, vias 0 -> 12
- net Batt1Gate: track 0.00 -> 80.9 mm, vias 0 -> 6
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- added copper zone on B.Cu, net -BATT1
Other:
- board outline added: 110.5 x 110.5 mm
- board text added: "ADC Splitter"
- board text added: "Batt1En"
- board text added: "Batt1UVP"
- board text added: "Batt2En"
- board text added: "Batt2UVP"
- board text added: "Enable"
- board text added: "ExtKill"
- board text added: "KillStatus"
- board text added: "OCPCtrl"
- board text added: "OCPLatch"
- board text added: "On/Off"
- board text added: "Orin Output"
- board text added: "Switch"
- board text added: "Teensy Passthrough"
- board text added: "Thruster Output"
- board text added: "UVPCtrl"

Commit message: done with dist
Parts:
- removed LED30, LED31, LED32, LED33, LED34, LED35, LED36: 1655, LED_SMD:LED_LiteOn_LTST-E563C_PLCC4_5.0x5.0mm_P3.2mm_HandSoldering
- added J9: Conn_01x04_Pin, Imported_Footprints:CONN_SD-43045-008_04_MOL, F.Cu at (160.3, 89.2)
- added JP28: Jumper_3_Bridged12, Jumper:SolderJumper-3_P1.3mm_Bridged2Bar12_RoundedPad1.0x1.5mm, F.Cu at (166.6, 86.1)
- moved TP5 143.2 mm to (263.2, 71.7)
- moved C2 139.9 mm to (260.6, 133.1)
- moved TP6 136.1 mm to (256.6, 78.1)
- moved R3 129.8 mm to (239.5, 98.2), turned to 180 degrees
- moved R1 126.5 mm to (236.2, 92.4), turned to 90 degrees
- moved R2 126.4 mm to (236.2, 96.2), turned to -90 degrees
- moved R6 126.0 mm to (236.4, 107.1), turned to 90 degrees
- moved R8 124.4 mm to (239.4, 101.1), turned to 180 degrees
- moved R7 121.0 mm to (236.4, 103.2), turned to -90 degrees
- moved C3 115.1 mm to (236.3, 130.5), turned to -90 degrees
- moved TP4 99.0 mm to (208.6, 147.4)
- moved TP2 90.0 mm to (196.4, 143.7)
- moved TP3 85.4 mm to (193.4, 143.1)
- moved JP20 69.6 mm to (182.5, 73.4)
- moved JP19 69.2 mm to (182.5, 70.6)
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Connections:
- LED1 pad 2: NEO_PASS1 -> toNEO_CTRL_Orin
- LED10 pad 4: NEO_PASS2 -> NeoPass2
- LED11 pad 2: Net-(LED11-DIN) -> NeoPass2
- LED11 pad 4: NEO_PASS1 -> Net-(LED11-DOUT)
- LED12 pad 2: Net-(LED12-DIN) -> Net-(LED11-DOUT)
- LED12 pad 4: NEO_PASS3 -> Net-(LED12-DOUT)
- LED13 pad 2: NEO_PASS4 -> Net-(LED12-DOUT)
- LED14 pad 2: NEO_PASS3 -> Net-(LED13-DOUT)
- LED15 pad 2: NEO_PASS5 -> Net-(LED14-DOUT)
- LED15 pad 4: Net-(LED15-DOUT) -> NeoPass3
- LED16 pad 2: Net-(LED13-DOUT) -> NeoPass3
- LED17 pad 2: Net-(LED14-DOUT) -> Net-(LED16-DOUT)
- LED18 pad 2: Net-(LED15-DOUT) -> Net-(LED17-DOUT)
- LED19 pad 2: Net-(LED16-DOUT) -> Net-(LED18-DOUT)
- LED2 pad 2: toNEO_CTRL_Orin -> Net-(LED1-DOUT)
- LED20 pad 2: Net-(LED17-DOUT) -> Net-(LED19-DOUT)
- LED20 pad 4: Net-(LED20-DOUT) -> NeoPass4
- LED21 pad 2: Net-(LED18-DOUT) -> NeoPass4
- LED22 pad 2: Net-(LED19-DOUT) -> Net-(LED21-DOUT)
- LED22 pad 4: NEO_PASS5 -> Net-(LED22-DOUT)
- LED23 pad 2: Net-(LED20-DOUT) -> Net-(LED22-DOUT)
- LED23 pad 4: NEO_PASS4 -> Net-(LED23-DOUT)
- LED24 pad 2: Net-(LED21-DOUT) -> Net-(LED23-DOUT)
- LED24 pad 4: NEO_PASS6 -> Net-(LED24-DOUT)
- LED25 pad 2: NEO_PASS7 -> Net-(LED24-DOUT)
- LED25 pad 4: Net-(LED25-DOUT) -> NeoPass5
- LED26 pad 2: NEO_PASS6 -> NeoPass5
- LED27 pad 2: NEO_PASS8 -> Net-(LED26-DOUT)
- LED28 pad 2: Net-(LED25-DOUT) -> Net-(LED27-DOUT)
- LED29 pad 2: Net-(LED26-DOUT) -> Net-(LED28-DOUT)
- LED29 pad 4: Net-(LED29-DOUT) -> /Neopixels/outNEO_Orin
- LED3 pad 2: NEO_PASS2 -> Net-(LED2-DOUT)
- LED4 pad 2: Net-(LED1-DOUT) -> Net-(LED3-DOUT)
- LED5 pad 2: Net-(LED2-DOUT) -> Net-(LED4-DOUT)
- LED5 pad 4: Net-(LED5-DOUT) -> NeoPass1
- LED6 pad 2: Net-(LED3-DOUT) -> NeoPass1
- LED7 pad 2: Net-(LED4-DOUT) -> Net-(LED6-DOUT)
- LED7 pad 4: Net-(LED10-DIN) -> Net-(LED7-DOUT)
- LED8 pad 2: Net-(LED5-DOUT) -> Net-(LED7-DOUT)
- LED8 pad 4: Net-(LED11-DIN) -> Net-(LED8-DOUT)
- LED9 pad 2: Net-(LED6-DOUT) -> Net-(LED8-DOUT)
- LED9 pad 4: Net-(LED12-DIN) -> Net-(LED10-DIN)
Routing:
- net toNEO_CTRL_Orin: track 0.00 -> 123.7 mm, vias 0 -> 8
- net ~{SystemKill}: track 60.6 -> 177.7 mm, vias 2 -> 18
- net Net-(LED17-DOUT): track 0.00 -> 107.0 mm, vias 0 -> 2
- net ~{OCPLatch}: track 80.5 -> 178.9 mm, vias 8 -> 22
- net LETeensy: track 5.45 -> 102.1 mm, vias 2 -> 12
- net Batt2Enable: track 53.8 -> 142.7 mm, vias 12 -> 20
- net I2C1_SCL: track 38.7 -> 122.2 mm, vias 2 -> 13
- net Batt1Enable: track 74.3 -> 157.8 mm, vias 17 -> 23
- net I2C1_SDA: track 36.2 -> 115.0 mm, vias 2 -> 9
- net D/A20: track 0.00 -> 66.6 mm, vias 0 -> 7
- net -BATT1: track 62.6 -> 117.6 mm, vias 22 -> 36
- net +VregDiode: track 104.2 -> 157.1 mm
- net +5V: track 570.6 -> 613.9 mm, vias 1 -> 2
- net VSampleBatt1: track 74.3 -> 114.2 mm, vias 6 -> 12
- net VSampleBatt2: track 78.5 -> 113.6 mm, vias 11 -> 15
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Other:
- board text added: "Batt1 Input"
- board text added: "Batt2 Input"
- board text added: "Blame: Vassili"
- board text added: "Stanford Robosub Power Management"
- board text removed: "Stanford Robosub 2024-2025"

Commit message: almost done with all orders
Parts:
- J1, J2: footprint Connector_AMASS:AMASS_XT60-M_1x02_P7.20mm_Vertical -> Connector_AMASS:AMASS_XT60IPW-M_1x03_P7.20mm_Horizontal
- moved J1 5.65 mm to (257.5, 87.8), turned to -90 degrees
- moved C1 3.26 mm to (240.8, 64.1)
- moved J2 3.14 mm to (254.3, 104.8)
- moved U1 1.93 mm to (242.8, 90.2)
- moved H1 1.69 mm to (191.3, 73.0)
- moved H4 1.69 mm to (239.3, 73.0)
- moved H2 1.69 mm to (191.3, 137.0)
- moved H3 1.69 mm to (239.3, 137.0)
- moved U2 1.65 mm to (242.9, 109.2)
- moved S1 1.49 mm to (232.7, 145.7)
Routing:
- net -BATT1: track 117.6 -> 163.4 mm, vias 36 -> 53
- net +VregDiode: track 157.1 -> 189.2 mm, vias 2 -> 6
- net Batt2Gate: track 105.4 -> 116.6 mm, vias 4 -> 2
- net /Battery Control Logic/UVPReference: track 90.1 -> 100.7 mm, vias 12 -> 13
- net +3.3V: track 276.3 -> 285.3 mm
- net +BATT1: track 71.1 -> 78.5 mm
- net Net-(LED17-DOUT): track 107.0 -> 112.4 mm, vias 2 -> 6
- net +5V: track 613.9 -> 609.6 mm
- net +BATT2: track 70.7 -> 68.0 mm
- net Batt1Enable: track 157.8 -> 155.2 mm, vias 23 -> 25
- net Batt2Enable: track 142.7 -> 144.7 mm, vias 20 -> 24
- net ~{OCPLatch}: track 178.9 -> 180.3 mm
- net Batt1Gate: track 80.9 -> 79.6 mm
- net +BATT: track 181.7 -> 182.6 mm
- net VSampleBatt1: track 114.2 -> 114.8 mm
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
Commit message: ready for fab
Parts:
- R21: footprint Imported_Footprints:RES_EXB2HV_1506x8 -> Imported_Footprints:2506_8x_Resistor_Array
- moved R21 0.37 mm to (241.2, 148.4)
Routing:
- net -BATT1: track 163.4 -> 169.8 mm

Commit message: some updates
Parts:
- removed U10, U6: LMV982MM, Imported_Footprints:LMV982MM_NOPB
- added U15: TSX634AIPT, Imported_Footprints:TSSOP14_STM, F.Cu at (199.3, 136.0)
- moved JP26 5.09 mm to (197.9, 129.9), turned to -90 degrees
- moved JP25 0.44 mm to (204.7, 131.6)
Routing:
- net ISample3.3V: track 93.4 -> 106.5 mm, vias 8 -> 10
- net -BATT1: track 169.8 -> 180.8 mm
- net /Battery Control Logic/OCPReference: track 100.9 -> 108.9 mm, vias 3 -> 4
- net /Battery Control Logic/~{OCP}: track 101.8 -> 109.0 mm, vias 6 -> 7
- net ~{OCPLatch}: track 180.7 -> 186.8 mm, vias 22 -> 24
- net +3.3V: track 285.3 -> 281.1 mm, vias 16 -> 15
- net /Battery Control Logic/Batt1>UVP: track 97.5 -> 101.5 mm
- net VSampleBatt2: track 113.7 -> 111.6 mm, vias 15 -> 13
- net /Battery Control Logic/Batt2>UVP: track 73.3 -> 74.9 mm, vias 16 -> 18
- net Net-(LED17-DOUT): track 112.4 -> 111.1 mm, vias 6 -> 4
- net VSampleBatt1: track 114.8 -> 116.1 mm, vias 12 -> 14
- net LETeensy: track 102.5 -> 103.8 mm, vias 12 -> 11
- net ~{SystemKill}: track 177.7 -> 178.7 mm
- net /Battery Control Logic/UVPReference: track 100.7 -> 101.3 mm, vias 13 -> 11
- net /Battery Control Logic/VBatt1<VBatt2: track 25.0 -> 24.7 mm, vias 4 -> 2
Other:
- board size 110.5 x 110.5 mm -> 110.9 x 110.5 mm

Commit message: board updates
Parts:
- removed TP2: TestPoint, TestPoint:TestPoint_Pad_1.0x1.0mm
- moved TP3 23.6 mm to (215.6, 151.1)
- moved U7 8.36 mm to (192.7, 147.6)
- moved TP4 7.06 mm to (215.7, 147.4)
- moved U11 7.03 mm to (200.6, 137.0)
- moved U8 6.69 mm to (200.4, 147.5)
- moved U15 6.41 mm to (200.4, 142.3), turned to 180 degrees
- moved JP16 6.05 mm to (182.1, 87.6)
- moved U9 4.96 mm to (206.6, 147.4)
- moved JP26 3.85 mm to (200.7, 132.6), turned to 180 degrees
- moved U13 3.25 mm to (209.6, 141.4)
- moved JP15 3.06 mm to (182.1, 84.9)
- moved JP27 3.00 mm to (209.3, 138.1), turned to 180 degrees
- moved JP25 2.23 mm to (203.8, 133.6), turned to -90 degrees
- moved JP23 1.48 mm to (209.6, 151.1)
- moved JP24 1.48 mm to (206.2, 151.1)
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Routing:
- net D/A20: track 66.6 -> 32.1 mm, vias 7 -> 3
- net VSampleBatt1: track 116.1 -> 146.2 mm, vias 14 -> 15
- net Analog_Voltage1: track 39.1 -> 68.5 mm, vias 3 -> 8
- net Batt2Enable: track 144.7 -> 171.0 mm
- net -BATT1: track 180.8 -> 205.2 mm, vias 53 -> 55
- net VSampleBatt2: track 111.6 -> 132.7 mm, vias 13 -> 15
- net /Battery Control Logic/~{GateDisable}: track 187.2 -> 203.9 mm, vias 21 -> 19
- net Net-(U7-2D): track 5.71 -> 22.3 mm
- net Net-(JP22-A): track 7.24 -> 20.7 mm
- net /Battery Control Logic/VBatt1<VBatt2: track 24.7 -> 13.0 mm
- net +5V: track 609.7 -> 621.2 mm
- net /Battery Control Logic/Batt1>UVP: track 101.5 -> 90.3 mm, vias 10 -> 8
- net Net-(JP24-A): track 3.77 -> 11.8 mm
- net +3.3V: track 281.1 -> 273.2 mm, vias 15 -> 14
- net toNEO_CTRL_Orin: track 123.7 -> 131.0 mm, vias 8 -> 6
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